File: FixtureDevKit-ADS.sch (KiCad schematic (older format))
At the start: 41 parts

Commit message: adding the dummy load circuit
Other:
- note added: "NC"
Changed lines of the file:
@@
 $Descr A4 11693 8268
 encoding utf-8
-Sheet 5 5
+Sheet 5 6
 Title ""
 Date ""
@@
 Text Notes 650  800  0    157  ~ 0
 ADS Voltage Read Circuit
+Text Notes 8650 3000 1    60   ~ 0
+NC
+Text Notes 8900 3000 1    60   ~ 0
+NC
+Text Notes 9200 3000 1    60   ~ 0
+NC
+Text Notes 9500 3000 1    60   ~ 0
+NC
 $EndSCHEMATC
