File: FixtureDevKit_Switches.sch (KiCad schematic (older format))
At the start: 0 parts

Commit message: adding LED and Button circuit
Parts:
- added D? (x8): LED_Dual_AACC, symbol LED_Dual_AACC
- added J?: LED_0, symbol Conn_01x03
- added J?: LED_7, symbol Conn_01x03
- added J?: LED_1, symbol Conn_01x03
- added J?: LED_2, symbol Conn_01x03
- added J?: LED_3, symbol Conn_01x03
- added J?: LED_4, symbol Conn_01x03
- added J?: LED_5, symbol Conn_01x03
- added J?: LED_6, symbol Conn_01x03
- added J?: SW_0, symbol Conn_01x04
- added J?: SW_1, symbol Conn_01x04
- added J?: SW_2, symbol Conn_01x04
- added J?: SW_3, symbol Conn_01x04
- added J?: SW_4, symbol Conn_01x04
- added J?: SW_5, symbol Conn_01x04
- added J?: SW_6, symbol Conn_01x04
- added J?: SW_7, symbol Conn_01x04
- added R? (x16): 1K, symbol R
- added SW? (x8): SW_Push_Dual, symbol SW_Push_Dual
Connections:
- new net: D?.1 (A1), J?.1 (Pin_1) (x8)
- new net: D?.2 (A2), R?.1 (x8)
- new net: D?.3 (K1), R?.1 (x8)
- new net: D?.4 (K2), J?.3 (Pin_3) (x8)
- new net: J?.2 (Pin_2), R?.2, R?.2 (x8)
- new net: J?.1 (Pin_1), SW?.1 (x8)
- new net: J?.2 (Pin_2), SW?.2 (x8)
- new net: J?.3 (Pin_3), SW?.3 (x8)
- new net: J?.4 (Pin_4), SW?.4 (x8)
Other:
- note added: "BUTTONS :)"
- note added: "GND\n"
- note added: "LED_Status_Indicators\n"
- note added: "SIG"
- note added: "VS"
