File: HARDWARE/v0.01/FixtureDevKit-Functional-Computer.sch (KiCad schematic (older format))
At the start: 15 parts, among them J5? CHIP4LH, J6? CHIP4RH, J8? CHIP4B2B

Commit message: addin more circuits!
Parts:
- added C? (x4): 1uf, symbol C
- added J?: VBUS, symbol Conn_01x02
- added J?: Audio-Jack-3, symbol Audio-Jack-3
- added R? (x2): 0R, symbol R
Connections:
- net GND: now also C?.2, C?.2, J?.3
- net LOLN: now also C?.1
- net LOLP: now also R?.1
- net LORN: now also C?.1
- net LORP: now also R?.1
- net at J?.1 (VBUS): now also J?.1 (Pin_1), J?.2 (Pin_2)
- new net: C?.2, J?.1
- new net: C?.2, J?.2
- new net: C?.1, R?.2 (x2)
Other:
- note added: "B2B Audio\n"
- note added: "TODO:\n- verify all pinouts\n- test points"
- note removed: "TODO:\nHEADERS\n - Audio\nB2B\n - Audio"
- moved on the sheet: J5?, J6?, J8?, J?

Commit message: adding netlist and design rules check
Parts:
- gave numbers to parts that had none: 22
- renumbered 10K to 10K1
Changed lines of the file:
@@
 $EndDescr
 $Comp
-L CHIP4LH J5?
+L CHIP4LH J57
 U 1 1 59EE680F
 P 8800 5700
-F 0 "J5?" H 8250 7900 60  0000 C CNN
+F 0 "J57" H 8250 7900 60  0000 C CNN
 F 1 "CHIP4LH" H 8600 5550 60  0000 C CNN
 F 2 "" H 8900 5700 60  0001 C CNN
@@
 $EndComp
 $Comp
-L CHIP4RH J6?
+L CHIP4RH J51
 U 1 1 59EE6892
 P 8850 2900
-F 0 "J6?" H 8350 4950 60  0000 C CNN
+F 0 "J51" H 8350 4950 60  0000 C CNN
 F 1 "CHIP4RH" H 8600 2800 60  0000 C CNN
 F 2 "" H 8900 2900 60  0001 C CNN
@@
 $EndComp
 $Comp
-L Conn_01x20 J?
+L Conn_01x20 J50
 U 1 1 59EE69C7
 P 9700 1850
-F 0 "J?" H 9700 2850 50  0000 C CNN
+F 0 "J50" H 9700 2850 50  0000 C CNN
 F 1 "Conn_01x20" H 9700 750 50  0000 C CNN
 F 2 "" H 9700 1850 50  0001 C CNN
@@
 $EndComp
 $Comp
-L Conn_01x20 J?
+L Conn_01x20 J49
 U 1 1 59EE6A17
 P 7950 1850
-F 0 "J?" H 7950 2850 50  0000 C CNN
+F 0 "J49" H 7950 2850 50  0000 C CNN
 F 1 "Conn_01x20" H 7950 750 50  0000 C CNN
 F 2 "" H 7950 1850 50  0001 C CNN
@@
 $EndComp
 $Comp
-L Conn_01x20 J?
+L Conn_01x20 J54
 U 1 1 59EE6A7B
 P 7950 4550
-F 0 "J?" H 7950 5550 50  0000 C CNN
+F 0 "J54" H 7950 5550 50  0000 C CNN
 F 1 "Conn_01x20" H 7950 3450 50  0000 C CNN
 F 2 "" H 7950 4550 50  0001 C CNN
@@
 $EndComp
 $Comp
-L Conn_01x20 J?
+L Conn_01x20 J55
 U 1 1 59EE6B51
 P 9700 4550
-F 0 "J?" H 9700 5550 50  0000 C CNN
+F 0 "J55" H 9700 5550 50  0000 C CNN
 F 1 "Conn_01x20" H 9700 3450 50  0000 C CNN
 F 2 "" H 9700 4550 50  0001 C CNN
@@
 $EndComp
 $Comp
-L GND #PWR?
+L GND #PWR048
 U 1 1 59EE7DE0
 P 7650 900
-F 0 "#PWR?" H 7650 650 50  0001 C CNN
+F 0 "#PWR048" H 7650 650 50  0001 C CNN
 F 1 "GND" H 7650 750 50  0000 C CNN
 F 2 "" H 7650 900 50  0001 C CNN
@@
 $EndComp
 $Comp
-L GND #PWR?
+L GND #PWR049
 U 1 1 59EE7F13
 P 10000 900
-F 0 "#PWR?" H 10000 650 50  0001 C CNN
+F 0 "#PWR049" H 10000 650 50  0001 C CNN
 F 1 "GND" H 10000 750 50  0000 C CNN
 F 2 "" H 10000 900 50  0001 C CNN
@@
 $EndComp
 $Comp
-L GND #PWR?
+L GND #PWR050
 U 1 1 59EE8282
 P 7650 3600
-F 0 "#PWR?" H 7650 3350 50  0001 C CNN
+F 0 "#PWR050" H 7650 3350 50  0001 C CNN
 F 1 "GND" H 7650 3450 50  0000 C CNN
 F 2 "" H 7650 3600 50  0001 C CNN
@@
 $EndComp
 $Comp
-L GND #PWR?
+L GND #PWR051
 U 1 1 59EE829F
 P 10000 3600
-F 0 "#PWR?" H 10000 3350 50  0001 C CNN
+F 0 "#PWR051" H 10000 3350 50  0001 C CNN
 F 1 "GND" H 10000 3450 50  0000 C CNN
 F 2 "" H 10000 3600 50  0001 C CNN
@@
 STATUSLED
 $Comp
-L LED D?
+L LED D10
 U 1 1 59EE94F2
 P 1900 7200
-F 0 "D?" H 1900 7300 50  0000 C CNN
+F 0 "D10" H 1900 7300 50  0000 C CNN
 F 1 "LED" H 1900 7100 50  0000 C CNN
 F 2 "" H 1900 7200 50  0001 C CNN
@@
 $EndComp
 $Comp
-L GND #PWR?
+L GND #PWR052
 U 1 1 59EE95A1
 P 1900 7450
-F 0 "#PWR?" H 1900 7200 50  0001 C CNN
+F 0 "#PWR052" H 1900 7200 50  0001 C CNN
 F 1 "GND" H 1900 7300 50  0000 C CNN
 F 2 "" H 1900 7450 50  0001 C CNN
@@
 PWRON
 $Comp
-L SW_Push SW?
+L SW_Push SW9
 U 1 1 59EEA13E
 P 900 7100
-F 0 "SW?" H 950 7200 50  0000 L CNN
+F 0 "SW9" H 950 7200 50  0000 L CNN
 F 1 "SW_Push" H 900 7040 50  0000 C CNN
 F 2 "" H 900 7300 50  0001 C CNN
@@
 $EndComp
 $Comp
-L GND #PWR?
+L GND #PWR053
 U 1 1 59EEA1C1
 P 900 7450
-F 0 "#PWR?" H 900 7200 50  0001 C CNN
+F 0 "#PWR053" H 900 7200 50  0001 C CNN
 F 1 "GND" H 900 7300 50  0000 C CNN
 F 2 "" H 900 7450 50  0001 C CNN
@@
 TS
 $Comp
-L R 10K
+L R 10K1
 U 1 1 59EEAD6D
 P 2650 6950
-F 0 "10K" V 2730 6950 50  0000 C CNN
+F 0 "10K1" V 2730 6950 50  0000 C CNN
 F 1 "R" V 2650 6950 50  0000 C CNN
 F 2 "" V 2580 6950 50  0001 C CNN
@@
 $EndComp
 $Comp
-L GND #PWR?
+L GND #PWR054
 U 1 1 59EEADAD
 P 2650 7250
-F 0 "#PWR?" H 2650 7000 50  0001 C CNN
+F 0 "#PWR054" H 2650 7000 50  0001 C CNN
 F 1 "GND" H 2650 7100 50  0000 C CNN
 F 2 "" H 2650 7250 50  0001 C CNN
@@
 BAT
 $Comp
-L GND #PWR?
+L GND #PWR055
 U 1 1 59EEB6E8
 P 3150 6650
-F 0 "#PWR?" H 3150 6400 50  0001 C CNN
+F 0 "#PWR055" H 3150 6400 50  0001 C CNN
 F 1 "GND" H 3150 6500 50  0000 C CNN
 F 2 "" H 3150 6650 50  0001 C CNN
@@
 $EndComp
 $Comp
-L Conn_01x02 J?
+L Conn_01x02 J60
 U 1 1 59EEB707
 P 3150 7050
-F 0 "J?" H 3150 7150 50  0000 C CNN
+F 0 "J60" H 3150 7150 50  0000 C CNN
 F 1 "JST-2P" H 3150 6850 50  0000 C CNN
 F 2 "" H 3150 7050 50  0001 C CNN
@@
 TODO:\n- verify all pinouts\n- test points
 $Comp
-L CHIP4B2B J8?
+L CHIP4B2B J56
 U 1 1 59EEDA12
 P 2600 5700
-F 0 "J8?" H 2100 9400 60  0000 C CNN
+F 0 "J56" H 2100 9400 60  0000 C CNN
 F 1 "CHIP4B2B" H 2300 5450 60  0000 C CNN
 F 2 "" H 2700 7250 60  0001 C CNN
@@
 $EndComp
 $Comp
-L Conn_01x35 J?
+L Conn_01x35 J52
 U 1 1 59EEDDE2
 P 1700 3900
-F 0 "J?" H 1700 5700 50  0000 C CNN
+F 0 "J52" H 1700 5700 50  0000 C CNN
 F 1 "Conn_01x35" H 1700 2100 50  0000 C CNN
 F 2 "" H 1700 3900 50  0001 C CNN
@@
 $EndComp
 $Comp
-L Conn_01x35 J?
+L Conn_01x35 J53
 U 1 1 59EEDE6B
 P 3550 3900
-F 0 "J?" H 3550 5700 50  0000 C CNN
+F 0 "J53" H 3550 5700 50  0000 C CNN
 F 1 "Conn_01x35" H 3550 2100 50  0000 C CNN
 F 2 "" H 3550 3900 50  0001 C CNN
@@
 USBOTG_B_ID
 $Comp
-L GND #PWR?
+L GND #PWR056
 U 1 1 59EF55B6
 P 3600 7300
-F 0 "#PWR?" H 3600 7050 50  0001 C CNN
+F 0 "#PWR056" H 3600 7050 50  0001 C CNN
 F 1 "GND" H 3600 7150 50  0000 C CNN
 F 2 "" H 3600 7300 50  0001 C CNN
@@
 $EndComp
 $Comp
-L Jumper_NC_Small JP?
+L Jumper_NC_Small JP5
 U 1 1 59EF5E24
 P 4200 7600
-F 0 "JP?" H 4200 7680 50  0000 C CNN
+F 0 "JP5" H 4200 7680 50  0000 C CNN
 F 1 "Jumper_NC" H 4210 7540 50  0000 C CNN
 F 2 "" H 4200 7600 50  0001 C CNN
@@
 $EndComp
 $Comp
-L GND #PWR?
+L GND #PWR057
 U 1 1 59EF61DC
 P 4450 7600
-F 0 "#PWR?" H 4450 7350 50  0001 C CNN
+F 0 "#PWR057" H 4450 7350 50  0001 C CNN
 F 1 "GND" H 4450 7450 50  0000 C CNN
 F 2 "" H 4450 7600 50  0001 C CNN
@@
 	3300 6100 4700 6100
 $Comp
-L USB_A J?
+L USB_A J59
 U 1 1 59EF4A5C
 P 3600 6800
-F 0 "J?" H 3400 7250 50  0000 L CNN
+F 0 "J59" H 3400 7250 50  0000 L CNN
 F 1 "USB_A" H 3400 7150 50  0000 L CNN
 F 2 "" H 3750 6750 50  0001 C CNN
@@
 $EndComp
 $Comp
-L Conn_01x02 J?
+L Conn_01x02 J58
 U 1 1 59F0CB92
 P 4250 6500
-F 0 "J?" H 4250 6600 50  0000 C CNN
+F 0 "J58" H 4250 6600 50  0000 C CNN
 F 1 "VBUS" V 4350 6450 50  0000 C CNN
 F 2 "" H 4250 6500 50  0001 C CNN
@@
 	4050 6600 4050 6500
 $Comp
-L Audio-Jack-3 J?
+L Audio-Jack-3 J61
 U 1 1 59F0D2AB
 P 5250 7450
-F 0 "J?" H 5200 7625 50  0000 C CNN
+F 0 "J61" H 5200 7625 50  0000 C CNN
 F 1 "Audio-Jack-3" H 5350 7380 50  0000 C CNN
 F 2 "" H 5500 7550 50  0001 C CNN
@@
 LORN
 $Comp
-L R R?
+L R R61
 U 1 1 59F0D645
 P 4850 6750
-F 0 "R?" V 4930 6750 50  0000 C CNN
+F 0 "R61" V 4930 6750 50  0000 C CNN
 F 1 "0R" V 4850 6750 50  0000 C CNN
 F 2 "" V 4780 6750 50  0001 C CNN
@@
 $EndComp
 $Comp
-L C C?
+L C C9
 U 1 1 59F0D690
 P 4850 7050
-F 0 "C?" H 4875 7150 50  0000 L CNN
+F 0 "C9" H 4875 7150 50  0000 L CNN
 F 1 "1uf" H 4875 6950 50  0000 L CNN
 F 2 "" H 4888 6900 50  0001 C CNN
@@
 	4850 7250 5150 7250
 $Comp
-L R R?
+L R R62
 U 1 1 59F0DD42
 P 5250 6750
-F 0 "R?" V 5330 6750 50  0000 C CNN
+F 0 "R62" V 5330 6750 50  0000 C CNN
 F 1 "0R" V 5250 6750 50  0000 C CNN
 F 2 "" V 5180 6750 50  0001 C CNN
@@
 $EndComp
 $Comp
-L C C?
+L C C10
 U 1 1 59F0DD9A
 P 5250 7050
-F 0 "C?" H 5275 7150 50  0000 L CNN
+F 0 "C10" H 5275 7150 50  0000 L CNN
 F 1 "1uf" H 5275 6950 50  0000 L CNN
 F 2 "" H 5288 6900 50  0001 C CNN
@@
 	5250 7200 5250 7250
 $Comp
-L C C?
+L C C11
 U 1 1 59F0E267
 P 5550 7050
-F 0 "C?" H 5575 7150 50  0000 L CNN
+F 0 "C11" H 5575 7150 50  0000 L CNN
 F 1 "1uf" H 5575 6950 50  0000 L CNN
 F 2 "" H 5588 6900 50  0001 C CNN
@@
 $EndComp
 $Comp
-L C C?
+L C C12
 U 1 1 59F0E2C1
 P 5750 7050
-F 0 "C?" H 5775 7150 50  0000 L CNN
+F 0 "C12" H 5775 7150 50  0000 L CNN
 F 1 "1uf" H 5775 6950 50  0000 L CNN
 F 2 "" H 5788 6900 50  0001 C CNN
@@
 $EndComp
 $Comp
-L GND #PWR?
+L GND #PWR058
 U 1 1 59F0E393
 P 5750 7650
-F 0 "#PWR?" H 5750 7400 50  0001 C CNN
+F 0 "#PWR058" H 5750 7400 50  0001 C CNN
 F 1 "GND" H 5750 7500 50  0000 C CNN
 F 2 "" H 5750 7650 50  0001 C CNN
