File: HARDWARE/v0.01/FixtureDevKit_Switches.sch (KiCad schematic (older format))
At the start: 48 parts

Commit message: editing some files. cleaning stuff up.
Parts:
- removed D?: LED_Dual_AACC, symbol LED_Dual_AACC
- added D? (x2): LED, symbol LED
- added TP? (x2): TEST, symbol TEST
Connections:
- net at J?.1 (Pin_1): now also R?.2
- net at R?.1: now also R?.2, D?.1 (K), D?.2 (A), TP?.1
- net GND: now reaches R?.1
- net GND: now also J?.3 (Pin_3)
- new net: D?.1 (K), D?.2 (A), J?.2 (Pin_2), TP?.1
Other:
- note added: "HIGH side LED = Violet/Purple\nLOW side LED = Ultra Emerald Green"
- note added: "NOTES:\n"
- note added: "TO DO:\n- confirm LED circuit\n- how many LED's do we want? (replace\nrest of LED circuits\n- is 1K resistor correct?\n- LED part number?"
- moved on the sheet: J?, R?
Changed lines of the file:
@@
 $EndDescr
-$Comp
-L LED_Dual_AACC D?
-U 1 1 59EF70F4
-P 2650 3000
-F 0 "D?" H 2650 3225 50  0000 C CNN
-F 1 "LED_Dual_AACC" H 2650 2750 50  0000 C CNN
-F 2 "" H 2680 3000 50  0001 C CNN
-F 3 "" H 2680 3000 50  0001 C CNN
-	1    2650 3000
-	0    -1   -1   0
-$EndComp
 $Comp
 L Conn_01x03 J?
 U 1 1 59EF71A1
-P 2650 1500
-F 0 "J?" H 2650 1700 50  0000 C CNN
-F 1 "LED_0" H 2650 1300 50  0000 C CNN
-F 2 "" H 2650 1500 50  0001 C CNN
-F 3 "" H 2650 1500 50  0001 C CNN
-	1    2650 1500
-	0    -1   -1   0
-$EndComp
-Text Notes 2750 1400 1    60   ~ 0
+P 2150 1850
+F 0 "J?" H 2150 2050 50  0000 C CNN
+F 1 "LED_0" H 2150 1650 50  0000 C CNN
+F 2 "" H 2150 1850 50  0001 C CNN
+F 3 "" H 2150 1850 50  0001 C CNN
+	1    2150 1850
+	0    -1   -1   0
+$EndComp
+Text Notes 2250 1750 1    60   ~ 0
 GND\n
-Text Notes 2650 1400 1    60   ~ 0
+Text Notes 2150 1750 1    60   ~ 0
 SIG
-Text Notes 2550 1400 1    60   ~ 0
+Text Notes 2050 1750 1    60   ~ 0
 VS
-Wire Wire Line
-	2550 3400 2550 3300
 $Comp
 L R R?
 U 1 1 59EF753E
-P 2550 2550
-F 0 "R?" V 2630 2550 50  0000 C CNN
-F 1 "1K" V 2550 2550 50  0000 C CNN
-F 2 "" V 2480 2550 50  0001 C CNN
-F 3 "" H 2550 2550 50  0001 C CNN
-	1    2550 2550
-	1    0    0    1
-$EndComp
-Wire Wire Line
-	2550 2400 3050 2400
+P 2050 2700
+F 0 "R?" V 2130 2700 50  0000 C CNN
+F 1 "1K" V 2050 2700 50  0000 C CNN
+F 2 "" V 1980 2700 50  0001 C CNN
+F 3 "" H 2050 2700 50  0001 C CNN
+	1    2050 2700
+	1    0    0    1
+$EndComp
 $Comp
 L R R?
 U 1 1 59EF799A
-P 3050 2550
-F 0 "R?" V 3130 2550 50  0000 C CNN
-F 1 "1K" V 3050 2550 50  0000 C CNN
-F 2 "" V 2980 2550 50  0001 C CNN
-F 3 "" H 3050 2550 50  0001 C CNN
-	1    3050 2550
-	1    0    0    1
-$EndComp
-Wire Wire Line
-	3050 2700 3050 3400
-Wire Wire Line
-	3050 3400 2750 3400
-Wire Wire Line
-	2750 3400 2750 3300
-Wire Wire Line
-	2650 1700 2650 2400
-Connection ~ 2650 2400
-Wire Wire Line
-	2550 3400 2350 3400
-Wire Wire Line
-	2350 3400 2350 2350
-Wire Wire Line
-	2350 2350 2550 2350
-Wire Wire Line
-	2550 2350 2550 1700
-Wire Wire Line
-	2750 1700 2750 2700
+P 2050 2300
+F 0 "R?" V 2130 2300 50  0000 C CNN
+F 1 "1K" V 2050 2300 50  0000 C CNN
+F 2 "" V 1980 2300 50  0001 C CNN
+F 3 "" H 2050 2300 50  0001 C CNN
+	1    2050 2300
+	1    0    0    1
+$EndComp
 $Comp
 L LED_Dual_AACC D?
@@
 	2650 5950 2650 5350
 Wire Wire Line
-	2650 5350 2550 5350
-Wire Wire Line
-	2550 5350 2550 4900
+	2550 5350 2650 5350
 Wire Wire Line
 	2800 5550 2800 5300
@@
 Wire Wire Line
 	2900 5250 2750 5250
-Wire Wire Line
-	2750 5250 2750 4900
 $Comp
 L SW_Push_Dual SW?
@@
 Wire Notes Line
 	10550 4400 10550 4300
+$Comp
+L LED D?
+U 1 1 59EFBE3C
+P 2450 2650
+F 0 "D?" H 2450 2750 50  0000 C CNN
+F 1 "LED" H 2450 2550 50  0000 C CNN
+F 2 "" H 2450 2650 50  0001 C CNN
+F 3 "" H 2450 2650 50  0001 C CNN
+	1    2450 2650
+	1    0    0    -1
+$EndComp
+$Comp
+L LED D?
+U 1 1 59EFC041
+P 2450 2350
+F 0 "D?" H 2450 2450 50  0000 C CNN
+F 1 "LED" H 2450 2250 50  0000 C CNN
+F 2 "" H 2450 2350 50  0001 C CNN
+F 3 "" H 2450 2350 50  0001 C CNN
+	1    2450 2350
+	-1   0    0    1
+$EndComp
+$Comp
+L GND #PWR?
+U 1 1 59EFC9DE
+P 2350 2050
+F 0 "#PWR?" H 2350 1800 50  0001 C CNN
+F 1 "GND" H 2350 1900 50  0000 C CNN
+F 2 "" H 2350 2050 50  0001 C CNN
+F 3 "" H 2350 2050 50  0001 C CNN
+	1    2350 2050
+	0    -1   -1   0
+$EndComp
+$Comp
+L GND #PWR?
+U 1 1 59EFCA83
+P 2050 2900
+F 0 "#PWR?" H 2050 2650 50  0001 C CNN
+F 1 "GND" H 2050 2750 50  0000 C CNN
+F 2 "" H 2050 2900 50  0001 C CNN
+F 3 "" H 2050 2900 50  0001 C CNN
+	1    2050 2900
+	1    0    0    -1
+$EndComp
+Wire Wire Line
+	2300 2350 2300 2650
+Wire Wire Line
+	2300 2500 2050 2500
+Connection ~ 2050 2500
+Connection ~ 2300 2500
+Wire Wire Line
+	2600 2350 2600 2650
+Wire Wire Line
+	2600 2500 2700 2500
+Connection ~ 2600 2500
+Wire Wire Line
+	2250 2050 2350 2050
+Wire Wire Line
+	2050 2050 2050 2150
+Wire Wire Line
+	2050 2450 2050 2550
+Wire Wire Line
+	2050 2850 2050 2900
+Wire Wire Line
+	2150 2050 2150 2200
+Wire Wire Line
+	2150 2200 2700 2200
+Wire Wire Line
+	2700 2200 2700 2500
+Text Notes -5950 1600 0    197  ~ 0
+TO DO:\n- confirm LED circuit\n- how many LED's do we want? (replace\nrest of LED circuits\n- is 1K resistor correct?\n- LED part number?
+$Comp
+L TEST TP?
+U 1 1 59EFED90
+P 2050 2500
+F 0 "TP?" H 2050 2800 50  0000 C BNN
+F 1 "TEST" H 2050 2750 50  0000 C CNN
+F 2 "" H 2050 2500 50  0001 C CNN
+F 3 "" H 2050 2500 50  0001 C CNN
+	1    2050 2500
+	0    -1   -1   0
+$EndComp
+$Comp
+L TEST TP?
+U 1 1 59EFEE69
+P 2700 2500
+F 0 "TP?" H 2700 2800 50  0000 C BNN
+F 1 "TEST" H 2700 2750 50  0000 C CNN
+F 2 "" H 2700 2500 50  0001 C CNN
+F 3 "" H 2700 2500 50  0001 C CNN
+	1    2700 2500
+	0    1    1    0
+$EndComp
+Text Notes 1050 1300 0    60   ~ 0
+HIGH side LED = Violet/Purple\nLOW side LED = Ultra Emerald Green
+Text Notes 1050 1100 0    79   ~ 0
+NOTES:\n
+Wire Wire Line
+	2550 4900 2550 5350
+Wire Wire Line
+	2750 5250 2750 4900
+Text Notes 1050 4550 0    79   ~ 0
+NOTES:\n
 $EndSCHEMATC

Commit message: adding netlist and design rules check
Parts:
- gave numbers to parts that had none: 51
