File: HARDWARE/v0.01/FixtureDevKit-INA.sch (KiCad schematic (older format))
At the start: 25 parts

Commit message: editing some files. cleaning stuff up.
Parts:
- removed C? (x4): 0.1uF, symbol C
- removed J?: Conn_01x04, symbol Conn_01x04
- removed J?: INA_40, symbol Conn_01x02
- removed J?: INA_41, symbol Conn_01x02
- removed J?: INA_42, symbol Conn_01x02
- removed J?: INA_43, symbol Conn_01x02
- removed JP? (x4): Jumper_NO, symbol Jumper_NO_Small
- removed R? (x8): 1K, symbol R
- removed U? (x4): INA219BIDCNT, symbol INA219BIDCNT
- added C? (x4): 0.1uF, symbol C
- added J? (x4): INA_40, symbol Conn_01x02
- added J? (x10): INA0, symbol Conn_01x04
- added JP? (x4): Jumper_NO, symbol Jumper_NO_Small
- added R? (x8): 1K, symbol R
- added U? (x4): INA219BIDCNT, symbol INA219BIDCNT
Connections:
- net GND: now also C?.1, C?.1, C?.1, C?.1, J?.3 (Pin_3), J?.3 (Pin_3), J?.3 (Pin_3), J?.3 (Pin_3), J?.3 (Pin_3), J?.3 (Pin_3), J?.3 (Pin_3), J?.3 (Pin_3), J?.3 (Pin_3), J?.3 (Pin_3), R?.2, R?.2, R?.2, R?.2, R?.2, U?.3 (GND), U?.3 (GND), U?.3 (GND), U?.3 (GND)
- new net: J?.1 (Pin_1), U?.1 (VIN+) (x4)
- new net: J?.2 (Pin_2), U?.2 (VIN-) (x4)
- new net: C?.2, JP?.2, U?.4 (VCC) (x4)
- new net: R?.1, U?.7 (A0) (x4)
- new net: R?.1, U?.8 (A1) (x4)
- new net SCL: J?.1 (Pin_1), J?.1 (Pin_1), J?.1 (Pin_1), J?.1 (Pin_1), J?.1 (Pin_1), J?.1 (Pin_1), J?.1 (Pin_1), J?.1 (Pin_1), J?.1 (Pin_1), J?.1 (Pin_1), R?.2, U?.5 (SCL), U?.5 (SCL), U?.5 (SCL), U?.5 (SCL)
- new net SDA: J?.2 (Pin_2), J?.2 (Pin_2), J?.2 (Pin_2), J?.2 (Pin_2), J?.2 (Pin_2), J?.2 (Pin_2), J?.2 (Pin_2), J?.2 (Pin_2), J?.2 (Pin_2), J?.2 (Pin_2), R?.2, U?.6 (SDA), U?.6 (SDA), U?.6 (SDA), U?.6 (SDA)
- new net VCC: J?.4 (Pin_4), J?.4 (Pin_4), J?.4 (Pin_4), J?.4 (Pin_4), J?.4 (Pin_4), J?.4 (Pin_4), J?.4 (Pin_4), J?.4 (Pin_4), J?.4 (Pin_4), J?.4 (Pin_4), JP?.1, JP?.1, JP?.1, JP?.1, R?.2
Other:
- note added: "INA_0\n"
- note added: "INA_1\n"
- note added: "INA_2\n\n"
- note added: "INA_3\n"
- note added: "Main Circuit \nHeaders\n"
- note added: "TO DO:\n- is it okay to have so many headers on the I2C lines?\n- Do we want the cut trace connector or not connect?"
- note removed: "GND"
- note removed: "SCL"
- note removed: "SDA"
- note removed: "VCC"

Commit message: o gosh
Parts:
- J?: value INA_40 -> INA_0
- J?: value INA_40 -> INA1
- J? (x2): value INA0 -> INA1
- J? (x5): value INA0 -> INA3
- J?: value INA_40 -> INA_3
- J?: value INA0 -> INA
Other:
- note added: "TO DO:\n- is it okay to have so many headers on the I2C lines?\n- Do we want the cut trace connector or not connect?\n- where do we want to add test points?"
- note removed: "TO DO:\n- is it okay to have so many headers on the I2C lines?\n- Do we want the cut trace connector or not connect?"
Changed lines of the file:
@@
 P 2900 3050
 F 0 "J?" H 2900 3150 50  0000 C CNN
-F 1 "INA_40" H 2900 2850 50  0000 C CNN
+F 1 "INA_0" H 2900 2850 50  0000 C CNN
 F 2 "" H 2900 3050 50  0001 C CNN
 F 3 "" H 2900 3050 50  0001 C CNN
@@
 P 5750 3050
 F 0 "J?" H 5750 3150 50  0000 C CNN
-F 1 "INA_40" H 5750 2850 50  0000 C CNN
+F 1 "INA1" H 5750 2850 50  0000 C CNN
 F 2 "" H 5750 3050 50  0001 C CNN
 F 3 "" H 5750 3050 50  0001 C CNN
@@
 P 4850 2000
 F 0 "J?" H 4850 2200 50  0000 C CNN
-F 1 "INA0" H 4850 1700 50  0000 C CNN
+F 1 "INA1" H 4850 1700 50  0000 C CNN
 F 2 "" H 4850 2000 50  0001 C CNN
 F 3 "" H 4850 2000 50  0001 C CNN
@@
 P 4850 4350
 F 0 "J?" H 4850 4550 50  0000 C CNN
-F 1 "INA0" H 4850 4050 50  0000 C CNN
+F 1 "INA1" H 4850 4050 50  0000 C CNN
 F 2 "" H 4850 4350 50  0001 C CNN
 F 3 "" H 4850 4350 50  0001 C CNN
@@
 P 2000 5100
 F 0 "J?" H 2000 5300 50  0000 C CNN
-F 1 "INA0" H 2000 4800 50  0000 C CNN
+F 1 "INA3" H 2000 4800 50  0000 C CNN
 F 2 "" H 2000 5100 50  0001 C CNN
 F 3 "" H 2000 5100 50  0001 C CNN
@@
 P 2000 7450
 F 0 "J?" H 2000 7650 50  0000 C CNN
-F 1 "INA0" H 2000 7150 50  0000 C CNN
+F 1 "INA3" H 2000 7150 50  0000 C CNN
 F 2 "" H 2000 7450 50  0001 C CNN
 F 3 "" H 2000 7450 50  0001 C CNN
@@
 P 5750 6150
 F 0 "J?" H 5750 6250 50  0000 C CNN
-F 1 "INA_40" H 5750 5950 50  0000 C CNN
+F 1 "INA_3" H 5750 5950 50  0000 C CNN
 F 2 "" H 5750 6150 50  0001 C CNN
 F 3 "" H 5750 6150 50  0001 C CNN
@@
 P 4850 5100
 F 0 "J?" H 4850 5300 50  0000 C CNN
-F 1 "INA0" H 4850 4800 50  0000 C CNN
+F 1 "INA3" H 4850 4800 50  0000 C CNN
 F 2 "" H 4850 5100 50  0001 C CNN
 F 3 "" H 4850 5100 50  0001 C CNN
@@
 P 4850 7450
 F 0 "J?" H 4850 7650 50  0000 C CNN
-F 1 "INA0" H 4850 7150 50  0000 C CNN
+F 1 "INA3" H 4850 7150 50  0000 C CNN
 F 2 "" H 4850 7450 50  0001 C CNN
 F 3 "" H 4850 7450 50  0001 C CNN
@@
 P 6800 2200
 F 0 "J?" H 6800 2400 50  0000 C CNN
-F 1 "INA0" H 6800 1900 50  0000 C CNN
+F 1 "INA" H 6800 1900 50  0000 C CNN
 F 2 "" H 6800 2200 50  0001 C CNN
 F 3 "" H 6800 2200 50  0001 C CNN
@@
 P 6800 3050
 F 0 "J?" H 6800 3250 50  0000 C CNN
-F 1 "INA0" H 6800 2750 50  0000 C CNN
+F 1 "INA3" H 6800 2750 50  0000 C CNN
 F 2 "" H 6800 3050 50  0001 C CNN
 F 3 "" H 6800 3050 50  0001 C CNN
@@
 	6300 1900 7500 1900
 Text Notes -6800 1400 0    157  ~ 0
-TO DO:\n- is it okay to have so many headers on the I2C lines?\n- Do we want the cut trace connector or not connect?
+TO DO:\n- is it okay to have so many headers on the I2C lines?\n- Do we want the cut trace connector or not connect?\n- where do we want to add test points?
 $EndSCHEMATC

Commit message: adding netlist and design rules check
Parts:
- gave numbers to parts that had none: 34

Commit message: updating a few blocks, adding test points
Parts:
- added TP? (x4): V+, symbol TEST
- added TP? (x4): V-, symbol TEST
- J17: value INA0 -> INA_0
- J18: value INA1 -> INA_1
- J25, J26: value INA3 -> INA_3
Connections:
- net at J20.1 (Pin_1), U1.1 (VIN+): now also TP?.1
- net at J20.2 (Pin_2), U1.2 (VIN-): now also TP?.1
- net at J21.1 (Pin_1), U2.1 (VIN+): now also TP?.1
- net at J21.2 (Pin_2), U2.2 (VIN-): now also TP?.1
- net at J27.1 (Pin_1), U3.1 (VIN+): now also TP?.1
- net at J27.2 (Pin_2), U3.2 (VIN-): now also TP?.1
- net at J28.1 (Pin_1), U4.1 (VIN+): now also TP?.1
Other:
- note added: "TO DO:\n- is it okay to have so many headers on the I2C lines?\n"
- note removed: "TO DO:\n- is it okay to have so many headers on the I2C lines?\n- Do we want the cut trace connector or not connect?\n- where do we want to add test points?"
Changed lines of the file:
@@
 	0    1    1    0
 $EndComp
-Text Notes 1650 3750 0    60   ~ 0
+Text Notes 2650 1950 0    60   ~ 0
 I2C addr 0x40
 $Comp
@@
 P 2000 2000
 F 0 "J17" H 2000 2200 50  0000 C CNN
-F 1 "INA0" H 2000 1700 50  0000 C CNN
+F 1 "INA_0" H 2000 1700 50  0000 C CNN
 F 2 "" H 2000 2000 50  0001 C CNN
 F 3 "" H 2000 2000 50  0001 C CNN
@@
 P 4850 2000
 F 0 "J18" H 4850 2200 50  0000 C CNN
-F 1 "INA1" H 4850 1700 50  0000 C CNN
+F 1 "INA_1" H 4850 1700 50  0000 C CNN
 F 2 "" H 4850 2000 50  0001 C CNN
 F 3 "" H 4850 2000 50  0001 C CNN
@@
 P 2000 5100
 F 0 "J25" H 2000 5300 50  0000 C CNN
-F 1 "INA3" H 2000 4800 50  0000 C CNN
+F 1 "INA_3" H 2000 4800 50  0000 C CNN
 F 2 "" H 2000 5100 50  0001 C CNN
 F 3 "" H 2000 5100 50  0001 C CNN
@@
 	0    1    1    0
 $EndComp
-Text Notes 4500 6850 0    60   ~ 0
+Text Notes 5500 5050 0    60   ~ 0
 I2C addr 0x43
 $Comp
@@
 P 4850 5100
 F 0 "J26" H 4850 5300 50  0000 C CNN
-F 1 "INA3" H 4850 4800 50  0000 C CNN
+F 1 "INA_3" H 4850 4800 50  0000 C CNN
 F 2 "" H 4850 5100 50  0001 C CNN
 F 3 "" H 4850 5100 50  0001 C CNN
@@
 	800  6250 800  6150
 Connection ~ 800  6150
-Text Notes 4500 3750 0    60   ~ 0
+Text Notes 5500 1950 0    60   ~ 0
 I2C addr 0x41\n
-Text Notes 1650 6850 0    60   ~ 0
+Text Notes 2650 5050 0    60   ~ 0
 I2C addr 0x42
 Wire Wire Line
@@
 	6300 1900 7500 1900
 Text Notes -6800 1400 0    157  ~ 0
-TO DO:\n- is it okay to have so many headers on the I2C lines?\n- Do we want the cut trace connector or not connect?\n- where do we want to add test points?
+TO DO:\n- is it okay to have so many headers on the I2C lines?\n
+$Comp
+L TEST TP?
+U 1 1 59F0E87E
+P 2600 3000
+F 0 "TP?" H 2600 3300 50  0000 C BNN
+F 1 "V+" H 2600 3250 50  0000 C CNN
+F 2 "" H 2600 3000 50  0001 C CNN
+F 3 "" H 2600 3000 50  0001 C CNN
+	1    2600 3000
+	1    0    0    -1
+$EndComp
+$Comp
+L TEST TP?
+U 1 1 59F0E99B
+P 2600 3200
+F 0 "TP?" H 2600 3500 50  0000 C BNN
+F 1 "V-" H 2600 3450 50  0000 C CNN
+F 2 "" H 2600 3200 50  0001 C CNN
+F 3 "" H 2600 3200 50  0001 C CNN
+	1    2600 3200
+	-1   0    0    1
+$EndComp
+Wire Wire Line
+	2600 3200 2600 3150
+Connection ~ 2600 3150
+Wire Wire Line
+	2600 3000 2600 3050
+Connection ~ 2600 3050
+$Comp
+L TEST TP?
+U 1 1 59F0EB4F
+P 5450 3000
+F 0 "TP?" H 5450 3300 50  0000 C BNN
+F 1 "V+" H 5450 3250 50  0000 C CNN
+F 2 "" H 5450 3000 50  0001 C CNN
+F 3 "" H 5450 3000 50  0001 C CNN
+	1    5450 3000
+	1    0    0    -1
+$EndComp
+$Comp
+L TEST TP?
+U 1 1 59F0EC40
+P 5450 3200
+F 0 "TP?" H 5450 3500 50  0000 C BNN
+F 1 "V-" H 5450 3450 50  0000 C CNN
+F 2 "" H 5450 3200 50  0001 C CNN
+F 3 "" H 5450 3200 50  0001 C CNN
+	1    5450 3200
+	-1   0    0    1
+$EndComp
+Wire Wire Line
+	5450 3000 5450 3050
+Connection ~ 5450 3050
+Wire Wire Line
+	5450 3200 5450 3150
+Connection ~ 5450 3150
+$Comp
+L TEST TP?
+U 1 1 59F0F32E
+P 5450 6300
+F 0 "TP?" H 5450 6600 50  0000 C BNN
+F 1 "V-" H 5450 6550 50  0000 C CNN
+F 2 "" H 5450 6300 50  0001 C CNN
+F 3 "" H 5450 6300 50  0001 C CNN
+	1    5450 6300
+	-1   0    0    1
+$EndComp
+$Comp
+L TEST TP?
+U 1 1 59F0F4AA
+P 2600 6300
+F 0 "TP?" H 2600 6600 50  0000 C BNN
+F 1 "V-" H 2600 6550 50  0000 C CNN
+F 2 "" H 2600 6300 50  0001 C CNN
+F 3 "" H 2600 6300 50  0001 C CNN
+	1    2600 6300
+	-1   0    0    1
+$EndComp
+$Comp
+L TEST TP?
+U 1 1 59F0F5A4
+P 2600 6100
+F 0 "TP?" H 2600 6400 50  0000 C BNN
+F 1 "V+" H 2600 6350 50  0000 C CNN
+F 2 "" H 2600 6100 50  0001 C CNN
+F 3 "" H 2600 6100 50  0001 C CNN
+	1    2600 6100
+	1    0    0    -1
+$EndComp
+Wire Wire Line
+	2600 6100 2600 6150
+Connection ~ 2600 6150
+Wire Wire Line
+	2600 6300 2600 6250
+Connection ~ 2600 6250
+$Comp
+L TEST TP?
+U 1 1 59F0F804
+P 5450 6100
+F 0 "TP?" H 5450 6400 50  0000 C BNN
+F 1 "V+" H 5450 6350 50  0000 C CNN
+F 2 "" H 5450 6100 50  0001 C CNN
+F 3 "" H 5450 6100 50  0001 C CNN
+	1    5450 6100
+	1    0    0    -1
+$EndComp
+Wire Wire Line
+	5450 6100 5450 6150
+Connection ~ 5450 6150
 $EndSCHEMATC
