File: HARDWARE/v0.01/KiCad/FixtureDevKit-Functional-Computer.sch (KiCad schematic (older format))
At the start: 27 parts, among them J79 JST-2P, J80 Conn_01x35, J81 USB_A, J82 CHIP4B2B, J83 VBUS, J84 Conn_01x35, J85 Audio-Jack-3, J86 Conn_01x20, J87 Conn_01x20, J88 CHIP4LH, J89 CHIP4RH, J90 Conn_01x20, J91 Conn_01x20, SW10 On/Off, SW11 SW_Push

Commit message: adding footprints
Parts:
- C5, C6, C7, C8: footprint (none) -> Capacitors_SMD:C_0805_HandSoldering
- J79: footprint (none) -> Connectors_JST:JST_PH_S2B-PH-K_02x2.00mm_Angled
- J80, J84: footprint (none) -> Pin_Headers:Pin_Header_Straight_1x35_Pitch2.54mm
- J83, JP1: footprint (none) -> Pin_Headers:Pin_Header_Straight_1x02_Pitch2.54mm
- J86, J87: footprint (none) -> Pin_Headers:Pin_Header_Straight_1x20_Pitch2.54mm_SMD_Pin1Left
- J88: footprint (none) -> Pin_Headers:Pin_Header_Straight_2x20_Pitch2.54mm
- J89: footprint (none) -> Pin_Headers:Pin_Header_Straight_2x19_Pitch2.54mm
- J90, J91: footprint (none) -> Pin_Headers:Pin_Header_Straight_1x20_Pitch2.54mm
- R84, R85: footprint (none) -> Resistors_SMD:R_0805_HandSoldering
Changed lines of the file:
@@
 F 0 "J88" H 8050 7900 60  0000 C CNN
 F 1 "CHIP4LH" H 8400 5550 60  0000 C CNN
-F 2 "" H 8700 5700 60  0001 C CNN
+F 2 "Pin_Headers:Pin_Header_Straight_2x20_Pitch2.54mm" H 8700 5700 60  0001 C CNN
 F 3 "" H 8700 5700 60  0001 C CNN
 	1    8600 5700
@@
 F 0 "J89" H 8150 4950 60  0000 C CNN
 F 1 "CHIP4RH" H 8400 2800 60  0000 C CNN
-F 2 "" H 8700 2900 60  0001 C CNN
+F 2 "Pin_Headers:Pin_Header_Straight_2x19_Pitch2.54mm" H 8700 2900 60  0001 C CNN
 F 3 "" H 8700 2900 60  0001 C CNN
 	1    8650 2900
@@
 F 0 "J90" H 9500 2850 50  0000 C CNN
 F 1 "Conn_01x20" H 9500 750 50  0000 C CNN
-F 2 "" H 9500 1850 50  0001 C CNN
+F 2 "Pin_Headers:Pin_Header_Straight_1x20_Pitch2.54mm" H 9500 1850 50  0001 C CNN
 F 3 "" H 9500 1850 50  0001 C CNN
 	1    9500 1850
@@
 F 0 "J86" H 7750 2850 50  0000 C CNN
 F 1 "Conn_01x20" H 7750 750 50  0000 C CNN
-F 2 "" H 7750 1850 50  0001 C CNN
+F 2 "Pin_Headers:Pin_Header_Straight_1x20_Pitch2.54mm_SMD_Pin1Left" H 7750 1850 50  0001 C CNN
 F 3 "" H 7750 1850 50  0001 C CNN
 	1    7750 1850
@@
 F 0 "J87" H 7750 5550 50  0000 C CNN
 F 1 "Conn_01x20" H 7750 3450 50  0000 C CNN
-F 2 "" H 7750 4550 50  0001 C CNN
+F 2 "Pin_Headers:Pin_Header_Straight_1x20_Pitch2.54mm_SMD_Pin1Left" H 7750 4550 50  0001 C CNN
 F 3 "" H 7750 4550 50  0001 C CNN
 	1    7750 4550
@@
 F 0 "J91" H 9500 5550 50  0000 C CNN
 F 1 "Conn_01x20" H 9500 3450 50  0000 C CNN
-F 2 "" H 9500 4550 50  0001 C CNN
+F 2 "Pin_Headers:Pin_Header_Straight_1x20_Pitch2.54mm" H 9500 4550 50  0001 C CNN
 F 3 "" H 9500 4550 50  0001 C CNN
 	1    9500 4550
@@
 F 0 "J79" H 3150 7150 50  0000 C CNN
 F 1 "JST-2P" H 3150 6850 50  0000 C CNN
-F 2 "" H 3150 7050 50  0001 C CNN
+F 2 "Connectors_JST:JST_PH_S2B-PH-K_02x2.00mm_Angled" H 3150 7050 50  0001 C CNN
 F 3 "" H 3150 7050 50  0001 C CNN
 	1    3150 7050
@@
 F 0 "J80" H 3350 5100 50  0000 C CNN
 F 1 "Conn_01x35" H 3350 1500 50  0000 C CNN
-F 2 "" H 3350 3300 50  0001 C CNN
+F 2 "Pin_Headers:Pin_Header_Straight_1x35_Pitch2.54mm" H 3350 3300 50  0001 C CNN
 F 3 "" H 3350 3300 50  0001 C CNN
 	1    3350 3300
@@
 F 0 "J84" H 5200 5100 50  0000 C CNN
 F 1 "Conn_01x35" H 5200 1500 50  0000 C CNN
-F 2 "" H 5200 3300 50  0001 C CNN
+F 2 "Pin_Headers:Pin_Header_Straight_1x35_Pitch2.54mm" H 5200 3300 50  0001 C CNN
 F 3 "" H 5200 3300 50  0001 C CNN
 	1    5200 3300
@@
 F 0 "JP1" H 4200 7680 50  0000 C CNN
 F 1 "Jumper_NC" H 4210 7540 50  0000 C CNN
-F 2 "" H 4200 7600 50  0001 C CNN
+F 2 "Pin_Headers:Pin_Header_Straight_1x02_Pitch2.54mm" H 4200 7600 50  0001 C CNN
 F 3 "" H 4200 7600 50  0001 C CNN
 	1    4200 7600
@@
 F 0 "J83" H 4250 6600 50  0000 C CNN
 F 1 "VBUS" V 4350 6450 50  0000 C CNN
-F 2 "" H 4250 6500 50  0001 C CNN
+F 2 "Pin_Headers:Pin_Header_Straight_1x02_Pitch2.54mm" H 4250 6500 50  0001 C CNN
 F 3 "" H 4250 6500 50  0001 C CNN
 	1    4250 6500
@@
 F 0 "R84" V 4930 6750 50  0000 C CNN
 F 1 "0R" V 4850 6750 50  0000 C CNN
-F 2 "" V 4780 6750 50  0001 C CNN
+F 2 "Resistors_SMD:R_0805_HandSoldering" V 4780 6750 50  0001 C CNN
 F 3 "" H 4850 6750 50  0001 C CNN
 	1    4850 6750
@@
 F 0 "C5" H 4875 7150 50  0000 L CNN
 F 1 "1uf" H 4875 6950 50  0000 L CNN
-F 2 "" H 4888 6900 50  0001 C CNN
+F 2 "Capacitors_SMD:C_0805_HandSoldering" H 4888 6900 50  0001 C CNN
 F 3 "" H 4850 7050 50  0001 C CNN
 	1    4850 7050
@@
 F 0 "R85" V 5330 6750 50  0000 C CNN
 F 1 "0R" V 5250 6750 50  0000 C CNN
-F 2 "" V 5180 6750 50  0001 C CNN
+F 2 "Resistors_SMD:R_0805_HandSoldering" V 5180 6750 50  0001 C CNN
 F 3 "" H 5250 6750 50  0001 C CNN
 	1    5250 6750
@@
 F 0 "C6" H 5275 7150 50  0000 L CNN
 F 1 "1uf" H 5275 6950 50  0000 L CNN
-F 2 "" H 5288 6900 50  0001 C CNN
+F 2 "Capacitors_SMD:C_0805_HandSoldering" H 5288 6900 50  0001 C CNN
 F 3 "" H 5250 7050 50  0001 C CNN
 	1    5250 7050
@@
 F 0 "C7" H 5575 7150 50  0000 L CNN
 F 1 "1uf" H 5575 6950 50  0000 L CNN
-F 2 "" H 5588 6900 50  0001 C CNN
+F 2 "Capacitors_SMD:C_0805_HandSoldering" H 5588 6900 50  0001 C CNN
 F 3 "" H 5550 7050 50  0001 C CNN
 	1    5550 7050
@@
 F 0 "C8" H 5775 7150 50  0000 L CNN
 F 1 "1uf" H 5775 6950 50  0000 L CNN
-F 2 "" H 5788 6900 50  0001 C CNN
+F 2 "Capacitors_SMD:C_0805_HandSoldering" H 5788 6900 50  0001 C CNN
 F 3 "" H 5750 7050 50  0001 C CNN
 	1    5750 7050

Commit message: adding footprints, starting layout
Parts:
- D14: footprint (none) -> LEDs:LED_0805_HandSoldering
- F1: value 3A -> 1206SFP300F; footprint (none) -> Fuse_Holders_and_Fuses:Fuse_SMD1206_HandSoldering
- R95: renamed from 10K1; value R -> 10K; footprint (none) -> Resistors_SMD:R_0805_HandSoldering
- TP103, TP104: footprint (none) -> TestPoint:TestPoint
Changed lines of the file:
@@
 LIBS:contrib
 LIBS:valves
-LIBS:FDN337N
+LIBS:TCA6424ARGJR
 LIBS:Fixture-Dev-Kit-cache
 EELAYER 25 0
@@
 F 0 "D14" H 1900 7300 50  0000 C CNN
 F 1 "LED" H 1900 7100 50  0000 C CNN
-F 2 "" H 1900 7200 50  0001 C CNN
+F 2 "LEDs:LED_0805_HandSoldering" H 1900 7200 50  0001 C CNN
 F 3 "" H 1900 7200 50  0001 C CNN
 	1    1900 7200
@@
 TS
 $Comp
-L R 10K1
+L R R95
 U 1 1 59EEAD6D
 P 2650 6950
-F 0 "10K1" V 2730 6950 50  0000 C CNN
-F 1 "R" V 2650 6950 50  0000 C CNN
-F 2 "" V 2580 6950 50  0001 C CNN
+F 0 "R95" V 2730 6950 50  0000 C CNN
+F 1 "10K" V 2650 6950 50  0000 C CNN
+F 2 "Resistors_SMD:R_0805_HandSoldering" V 2580 6950 50  0001 C CNN
 F 3 "" H 2650 6950 50  0001 C CNN
 	1    2650 6950
@@
 P 800 5000
 F 0 "F1" V 880 5000 50  0000 C CNN
-F 1 "3A" V 725 5000 50  0000 C CNN
-F 2 "" V 730 5000 50  0001 C CNN
+F 1 "1206SFP300F" V 725 5000 50  0000 C CNN
+F 2 "Fuse_Holders_and_Fuses:Fuse_SMD1206_HandSoldering" V 730 5000 50  0001 C CNN
 F 3 "" H 800 5000 50  0001 C CNN
 	1    800  5000
@@
 F 0 "TP104" H 4000 7400 50  0000 C BNN
 F 1 "D+" H 4000 7350 50  0000 C CNN
-F 2 "" H 4000 7100 50  0001 C CNN
+F 2 "TestPoint:TestPoint" H 4000 7100 50  0001 C CNN
 F 3 "" H 4000 7100 50  0001 C CNN
 	1    4000 7100
@@
 F 0 "TP103" H 3950 7500 50  0000 C BNN
 F 1 "D-" H 3950 7450 50  0000 C CNN
-F 2 "" H 3950 7200 50  0001 C CNN
+F 2 "TestPoint:TestPoint" H 3950 7200 50  0001 C CNN
 F 3 "" H 3950 7200 50  0001 C CNN
 	1    3950 7200

Commit message: adding datasheets, cleaning up schematic
Parts:
- D14: value LED -> LNJP12X8ARA
- J79: value JST-2P -> JST-2P-RA
- J85: value Audio-Jack-3 -> SF-352X-SMT
- SW10: value On/Off -> YSS-19-1202-N
- SW11: value SW_Push -> TL9210AF260Q
Changed lines of the file:
@@
 P 1900 7200
 F 0 "D14" H 1900 7300 50  0000 C CNN
-F 1 "LED" H 1900 7100 50  0000 C CNN
+F 1 "LNJP12X8ARA" H 1900 7100 50  0000 C CNN
 F 2 "LEDs:LED_0805_HandSoldering" H 1900 7200 50  0001 C CNN
 F 3 "" H 1900 7200 50  0001 C CNN
@@
 P 900 7100
 F 0 "SW11" H 950 7200 50  0000 L CNN
-F 1 "SW_Push" H 900 7040 50  0000 C CNN
+F 1 "TL9210AF260Q" H 900 7040 50  0000 C CNN
 F 2 "" H 900 7300 50  0001 C CNN
 F 3 "" H 900 7300 50  0001 C CNN
@@
 P 3150 7050
 F 0 "J79" H 3150 7150 50  0000 C CNN
-F 1 "JST-2P" H 3150 6850 50  0000 C CNN
+F 1 "JST-2P-RA" H 3150 6850 50  0000 C CNN
 F 2 "Connectors_JST:JST_PH_S2B-PH-K_02x2.00mm_Angled" H 3150 7050 50  0001 C CNN
 F 3 "" H 3150 7050 50  0001 C CNN
@@
 P 5250 7450
 F 0 "J85" H 5200 7625 50  0000 C CNN
-F 1 "Audio-Jack-3" H 5350 7380 50  0000 C CNN
+F 1 "SF-352X-SMT" H 5350 7380 50  0000 C CNN
 F 2 "" H 5500 7550 50  0001 C CNN
 F 3 "" H 5500 7550 50  0001 C CNN
@@
 P 800 5400
 F 0 "SW10" H 800 5570 50  0000 C CNN
-F 1 "On/Off" H 800 5200 50  0000 C CNN
+F 1 "YSS-19-1202-N" H 800 5200 50  0000 C CNN
 F 2 "" H 800 5400 50  0001 C CNN
 F 3 "" H 800 5400 50  0001 C CNN
