File: HARDWARE/v0.01/KiCad/Fixture-Dev-Kit.kicad_pcb (KiCad board)
At the start: 2 copper layers, 364 parts, among them J1 POWER, J10 LED_4, J100 INA_43, J101 INA_43, J102 INA_41, J103 INA_43, J104 INA, J105 INA, J11 SW_5, J12 LED_5, J13 SW_6, J14 LED_6, J15 SW_7, J16 ADS_48, J17 ADS_48, J18 ADS_4A, J19 ADS_4A, J2 LED_0, J20 ADS_48, J21 ADS_4A, J22 ADS, J23 ADS, J24 ADS_49, J25 ADS_49, J26 ADS_49, J27 ADS_4B, J28 ADS_4B, J29 ADS_4B, J3 SW_0, J30 LOAD_0, J31 LOAD_1, J32 LOAD_2, J33 LOAD_3, J34 Conn_01x20, J35 BAT, J36 CHIP4LH, J38 Conn_01x20, J39 VBUS, J4 SW_1, J40 VBUS, J41 B_D+, J42 D-TP's, J43 B_D-, J44 USB_ID, J45 UPDATE, J46 ANT--SELECT, J47 Conn_01x20, J49 VBUS, J5 LED_1, J50 A_D+, J51 A_D-, J53 Conn_01x20, J54 Conn_01x35, J56 Conn_01x35, J57 IOExp_0, J58 IOExp_0, J59 Conn_01x24, J6 SW_2, J60 IOExp_0, J61 IOExp_0, J62 Conn_01x24, J63 FET_0, J64 FET_4, J65 FET_1, J66 FET_5, J67 FET_2, J68 FET_6, J69 FET_3, J7 LED_3, J70 FET_7, J71 NFET_0, J72 NFET_4, J73 NFET_1, J74 NFET_5, J75 NFET_2, J76 NFET_6, J77 NFET_3, J78 NFET_7, J79 JST-2P, J8 SW_3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

Commit message: updating pcb layout
Parts:
- J36: footprint Pin_Headers:Pin_Header_Angled_2x20_Pitch2.54mm -> Pin_Headers:Pin_Header_Straight_2x20_Pitch2.54mm
- J38: footprint Pin_Headers:Pin_Header_Angled_1x20_Pitch2.54mm -> Pin_Headers:Pin_Header_Straight_1x20_Pitch2.54mm
- J86, J87: footprint Pin_Headers:Pin_Header_Straight_1x20_Pitch2.54mm_SMD_Pin1Left -> Pin_Headers:Pin_Header_Straight_1x20_Pitch2.54mm
- J89: footprint Pin_Headers:Pin_Header_Straight_2x19_Pitch2.54mm -> Pin_Headers:Pin_Header_Straight_2x20_Pitch2.54mm
- moved TP34 527.8 mm to (-69.3, 213.7)
- moved TP45 527.0 mm to (-69.3, 209.0)
- moved TP46 526.3 mm to (-69.3, 204.3)
- moved TP62 525.6 mm to (-69.3, 199.6)
- moved TP63 524.9 mm to (-69.3, 194.9)
- moved TP78 524.3 mm to (-69.3, 190.2)
- moved TP68 523.7 mm to (-69.3, 185.5)
- moved J60 522.0 mm to (-69.5, 167.8)
- moved TP43 520.6 mm to (-62.8, 209.0)
- moved TP40 519.8 mm to (-62.8, 204.3)
- moved TP47 519.1 mm to (-62.8, 199.6)
- moved TP61 518.4 mm to (-62.8, 194.9)
- moved TP64 517.8 mm to (-62.8, 190.2)
- moved TP67 517.2 mm to (-62.8, 185.5)
- moved J57 515.7 mm to (-63.1, 167.8)
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Connections:
- J71 pad 2: /Fixture Dev Kits - NMosfets/Gate_0 -> /Fixture Dev Kits - NMosfets/Source_0
- J71 pad 3: /Fixture Dev Kits - NMosfets/Drain_0 -> /Fixture Dev Kits - NMosfets/Gate_0
- J71 pad 4: /Fixture Dev Kits - NMosfets/Drain_0 -> /Fixture Dev Kits - NMosfets/Gate_0
- J71 pad 5: /Fixture Dev Kits - NMosfets/Gate_0 -> /Fixture Dev Kits - NMosfets/Drain_0
- J71 pad 6: /Fixture Dev Kits - NMosfets/Source_0 -> /Fixture Dev Kits - NMosfets/Drain_0
- J72 pad 1: /Fixture Dev Kits - NMosfets/Source_4 -> /Fixture Dev Kits - NMosfets/Drain_4
- J72 pad 2: /Fixture Dev Kits - NMosfets/Gate_4 -> /Fixture Dev Kits - NMosfets/Drain_4
- J72 pad 3: /Fixture Dev Kits - NMosfets/Drain_4 -> /Fixture Dev Kits - NMosfets/Gate_4
- J72 pad 4: /Fixture Dev Kits - NMosfets/Drain_4 -> /Fixture Dev Kits - NMosfets/Gate_4
- J72 pad 5: /Fixture Dev Kits - NMosfets/Gate_4 -> /Fixture Dev Kits - NMosfets/Drain_4
- J72 pad 6: /Fixture Dev Kits - NMosfets/Source_4 -> /Fixture Dev Kits - NMosfets/Drain_4
- J73 pad 2: /Fixture Dev Kits - NMosfets/Gate_1 -> /Fixture Dev Kits - NMosfets/Source_1
- J73 pad 3: /Fixture Dev Kits - NMosfets/Drain_1 -> /Fixture Dev Kits - NMosfets/Gate_1
- J73 pad 4: /Fixture Dev Kits - NMosfets/Drain_1 -> /Fixture Dev Kits - NMosfets/Gate_1
- J73 pad 5: /Fixture Dev Kits - NMosfets/Gate_1 -> /Fixture Dev Kits - NMosfets/Drain_1
- J73 pad 6: /Fixture Dev Kits - NMosfets/Source_1 -> /Fixture Dev Kits - NMosfets/Drain_1
- J74 pad 1: /Fixture Dev Kits - NMosfets/Source_5 -> /Fixture Dev Kits - NMosfets/Drain_5
- J74 pad 2: /Fixture Dev Kits - NMosfets/Gate_5 -> /Fixture Dev Kits - NMosfets/Drain_5
- J74 pad 3: /Fixture Dev Kits - NMosfets/Drain_5 -> /Fixture Dev Kits - NMosfets/Gate_5
- J74 pad 4: /Fixture Dev Kits - NMosfets/Drain_5 -> /Fixture Dev Kits - NMosfets/Gate_5
- J74 pad 5: /Fixture Dev Kits - NMosfets/Gate_5 -> /Fixture Dev Kits - NMosfets/Drain_5
- J74 pad 6: /Fixture Dev Kits - NMosfets/Source_5 -> /Fixture Dev Kits - NMosfets/Drain_5
- J75 pad 1: /Fixture Dev Kits - NMosfets/Source_2 -> /Fixture Dev Kits - NMosfets/Drain_2
- J75 pad 2: /Fixture Dev Kits - NMosfets/Gate_2 -> /Fixture Dev Kits - NMosfets/Drain_2
- J75 pad 3: /Fixture Dev Kits - NMosfets/Drain_2 -> /Fixture Dev Kits - NMosfets/Gate_2
- J75 pad 4: /Fixture Dev Kits - NMosfets/Drain_2 -> /Fixture Dev Kits - NMosfets/Gate_2
- J75 pad 5: /Fixture Dev Kits - NMosfets/Gate_2 -> /Fixture Dev Kits - NMosfets/Drain_2
- J75 pad 6: /Fixture Dev Kits - NMosfets/Source_2 -> /Fixture Dev Kits - NMosfets/Drain_2
- J76 pad 1: /Fixture Dev Kits - NMosfets/Source_6 -> /Fixture Dev Kits - NMosfets/Drain_6
- J76 pad 2: /Fixture Dev Kits - NMosfets/Gate_6 -> /Fixture Dev Kits - NMosfets/Drain_6
- J76 pad 3: /Fixture Dev Kits - NMosfets/Drain_6 -> /Fixture Dev Kits - NMosfets/Gate_6
- J76 pad 4: /Fixture Dev Kits - NMosfets/Drain_6 -> /Fixture Dev Kits - NMosfets/Gate_6
- J76 pad 5: /Fixture Dev Kits - NMosfets/Gate_6 -> /Fixture Dev Kits - NMosfets/Drain_6
- J76 pad 6: /Fixture Dev Kits - NMosfets/Source_6 -> /Fixture Dev Kits - NMosfets/Drain_6
- J77 pad 1: /Fixture Dev Kits - NMosfets/Source_3 -> /Fixture Dev Kits - NMosfets/Drain_3
- J77 pad 2: /Fixture Dev Kits - NMosfets/Gate_3 -> /Fixture Dev Kits - NMosfets/Drain_3
- J77 pad 3: /Fixture Dev Kits - NMosfets/Drain_3 -> /Fixture Dev Kits - NMosfets/Gate_3
- J77 pad 4: /Fixture Dev Kits - NMosfets/Drain_3 -> /Fixture Dev Kits - NMosfets/Gate_3
- J77 pad 5: /Fixture Dev Kits - NMosfets/Gate_3 -> /Fixture Dev Kits - NMosfets/Drain_3
- J77 pad 6: /Fixture Dev Kits - NMosfets/Source_3 -> /Fixture Dev Kits - NMosfets/Drain_3
- J78 pad 1: /Fixture Dev Kits - NMosfets/Source_7 -> /Fixture Dev Kits - NMosfets/Drain_7
- J78 pad 2: /Fixture Dev Kits - NMosfets/Gate_7 -> /Fixture Dev Kits - NMosfets/Drain_7
- J78 pad 3: /Fixture Dev Kits - NMosfets/Drain_7 -> /Fixture Dev Kits - NMosfets/Gate_7
- J78 pad 4: /Fixture Dev Kits - NMosfets/Drain_7 -> /Fixture Dev Kits - NMosfets/Gate_7
- J78 pad 5: /Fixture Dev Kits - NMosfets/Gate_7 -> /Fixture Dev Kits - NMosfets/Drain_7
- J78 pad 6: /Fixture Dev Kits - NMosfets/Source_7 -> /Fixture Dev Kits - NMosfets/Drain_7
- Q14 pad 2: /Fixture Dev Kits - NMosfets/Source_4 -> /Fixture Dev Kits - NMosfets/Drain_4
- Q16 pad 2: /Fixture Dev Kits - NMosfets/Source_5 -> /Fixture Dev Kits - NMosfets/Drain_5
- Q17 pad 2: /Fixture Dev Kits - NMosfets/Source_2 -> /Fixture Dev Kits - NMosfets/Drain_2
- Q18 pad 2: /Fixture Dev Kits - NMosfets/Source_6 -> /Fixture Dev Kits - NMosfets/Drain_6
- Q19 pad 2: /Fixture Dev Kits - NMosfets/Source_3 -> /Fixture Dev Kits - NMosfets/Drain_3
- Q20 pad 2: /Fixture Dev Kits - NMosfets/Source_7 -> /Fixture Dev Kits - NMosfets/Drain_7
- R69 pad 2: /Fixture Dev Kits - NMosfets/Source_4 -> /Fixture Dev Kits - NMosfets/Drain_4
- R73 pad 2: /Fixture Dev Kits - NMosfets/Source_5 -> /Fixture Dev Kits - NMosfets/Drain_5
- R76 pad 2: /Fixture Dev Kits - NMosfets/Source_2 -> /Fixture Dev Kits - NMosfets/Drain_2
- R77 pad 2: /Fixture Dev Kits - NMosfets/Source_6 -> /Fixture Dev Kits - NMosfets/Drain_6
- R80 pad 2: /Fixture Dev Kits - NMosfets/Source_3 -> /Fixture Dev Kits - NMosfets/Drain_3
- R81 pad 2: /Fixture Dev Kits - NMosfets/Source_7 -> /Fixture Dev Kits - NMosfets/Drain_7
Other:
- board outline added: 100.1 x 100.1 mm

Commit message: beginning pcb layout
Parts:
- added D15, D17: Purple, LEDs:LED_0805_HandSoldering, F.Cu at (68.8, 194.1)
- added D16, D18: Green, LEDs:LED_0805_HandSoldering, F.Cu at (68.8, 194.1)
- added F2: 1206SFP300F, Fuse_Holders_and_Fuses:Fuse_SMD1206_HandSoldering, F.Cu at (0.00, 0.00)
- added J106: LED_6, Pin_Headers:Pin_Header_Straight_1x03_Pitch2.54mm, F.Cu at (68.8, 194.1)
- added J107: LED_7, Pin_Headers:Pin_Header_Straight_1x03_Pitch2.54mm, F.Cu at (68.8, 194.1)
- added J52: CHIP4RH, Pin_Headers:Pin_Header_Straight_2x20_Pitch2.54mm, F.Cu at (241.3, 31.6)
- added R46: 10R, 5W, Resistors_THT:R_Axial_Power_L25.0mm_W9.0mm_P30.48mm, F.Cu at (152.4, 61.1)
- added R47: 10R, 5W, Resistors_THT:R_Axial_Power_L25.0mm_W9.0mm_P30.48mm, F.Cu at (142.6, 94.7)
- added R48: 10R, 5W, Resistors_THT:R_Axial_Power_L25.0mm_W9.0mm_P30.48mm, F.Cu at (152.4, 94.7)
- added R96, R97, R98, R99: 1K, Resistors_SMD:R_0805_HandSoldering, F.Cu at (68.8, 194.1)
- D1, D11, D3, D5, D7, D9: value LED -> Purple
- D10, D12, D2, D4, D6, D8: value LED -> Green
- D13, D14: value LED -> LNJP12X8ARA
- J10: value LED_4 -> LED_3
- J12: value LED_5 -> LED_4
- J14: value LED_6 -> LED_5
- J64: value FET_4 -> FET_0
- J65: value FET_1 -> FET_0
- J66: value FET_5 -> FET_0
- J67: value FET_2 -> FET_0
- J68: value FET_6 -> FET_0
- J69: value FET_3 -> FET_0
- J7: value LED_3 -> LED_2
- J70: value FET_7 -> FET_0
- J79: value JST-2P -> JST-2P-RA
- J89: footprint Pin_Headers:Pin_Header_Straight_2x20_Pitch2.54mm -> Pin_Headers:Pin_Header_Straight_2x19_Pitch2.54mm
- R45: footprint Resistors_SMD:R_0805_HandSoldering -> Resistors_THT:R_Axial_Power_L25.0mm_W9.0mm_P30.48mm
- TP1, TP3, TP5, TP7: value VS -> SIG
- moved R52 289.0 mm to (126.2, 37.9), turned to 270 degrees
- moved J104 283.5 mm to (132.1, 13.8), turned to 270 degrees
- moved R54 283.2 mm to (126.3, 33.1), turned to 270 degrees
- moved J63 254.2 mm to (120.8, 32.8)
- moved Q5 253.7 mm to (130.9, 35.2), turned to 270 degrees
- moved R45 174.5 mm to (142.6, 61.1), turned to 90 degrees
- moved F1 119.2 mm to (70.6, 33.3), turned to 90 degrees
- moved J96 106.6 mm to (169.8, 40.3), turned to 180 degrees
- moved C1 103.0 mm to (187.0, 43.1), turned to 0 degrees
- moved U1 102.7 mm to (186.4, 38.9)
- moved U7 101.3 mm to (165.7, 38.7), turned to 180 degrees
- moved J93 100.2 mm to (162.2, 34.1), turned to 90 degrees
- moved C9 98.7 mm to (165.7, 41.2), turned to 180 degrees
- moved R13 98.7 mm to (182.3, 43.0), turned to 180 degrees
- moved J17 98.3 mm to (176.9, 45.8), turned to 90 degrees
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Connections:
- D12 pad 1: Net-(D11-Pad2) -> Net-(D12-Pad1)
- D2 pad 1: Net-(D1-Pad2) -> Net-(D2-Pad1)
- D4 pad 1: Net-(D3-Pad2) -> Net-(D4-Pad1)
- D6 pad 1: Net-(D5-Pad2) -> Net-(D6-Pad1)
- D8 pad 1: Net-(D7-Pad2) -> Net-(D8-Pad1)
- D9 pad 2: Net-(D10-Pad1) -> Net-(D9-Pad2)
- F1 pad 1: +5V -> Net-(F1-Pad1)
- F1 pad 2: Net-(F1-Pad2) -> /Fixture Dev Kit - Functional Computer/C4-PWR-IN
- J100 pad 1: /Fixture Dev Kit - Functional Computer/I2C-SCK -> /Fixture Dev Kit - ADS/C4-VCC-3V3
- J100 pad 2: /Fixture Dev Kit - Functional Computer/I2C-SDA -> GND
- J100 pad 3: GND -> /Fixture Dev Kit - Functional Computer/I2C-SDA
- J100 pad 4: /Fixture Dev Kit - ADS/C4-VCC-3V3 -> /Fixture Dev Kit - Functional Computer/I2C-SCK
- J101 pad 1: /Fixture Dev Kit - Functional Computer/I2C-SCK -> /Fixture Dev Kit - ADS/C4-VCC-3V3
- J101 pad 2: /Fixture Dev Kit - Functional Computer/I2C-SDA -> GND
- J101 pad 3: GND -> /Fixture Dev Kit - Functional Computer/I2C-SDA
- J101 pad 4: /Fixture Dev Kit - ADS/C4-VCC-3V3 -> /Fixture Dev Kit - Functional Computer/I2C-SCK
- J18 pad 1: /Fixture Dev Kit - ADS/I2C-SCK -> /Fixture Dev Kit - ADS/C4-VCC-3V3
- J18 pad 2: /Fixture Dev Kit - ADS/I2C-SDA -> GND
- J18 pad 3: GND -> /Fixture Dev Kit - ADS/I2C-SDA
- J18 pad 4: /Fixture Dev Kit - ADS/C4-VCC-3V3 -> /Fixture Dev Kit - ADS/I2C-SCK
- J19 pad 1: /Fixture Dev Kit - ADS/I2C-SCK -> /Fixture Dev Kit - ADS/C4-VCC-3V3
- J19 pad 2: /Fixture Dev Kit - ADS/I2C-SDA -> GND
- J19 pad 3: GND -> /Fixture Dev Kit - ADS/I2C-SDA
- J19 pad 4: /Fixture Dev Kit - ADS/C4-VCC-3V3 -> /Fixture Dev Kit - ADS/I2C-SCK
- J24 pad 1: /Fixture Dev Kit - ADS/I2C-SCK -> /Fixture Dev Kit - ADS/C4-VCC-3V3
- J24 pad 2: /Fixture Dev Kit - ADS/I2C-SDA -> GND
- J24 pad 3: GND -> /Fixture Dev Kit - ADS/I2C-SDA
- J24 pad 4: /Fixture Dev Kit - ADS/C4-VCC-3V3 -> /Fixture Dev Kit - ADS/I2C-SCK
- J25 pad 1: /Fixture Dev Kit - ADS/I2C-SCK -> /Fixture Dev Kit - ADS/C4-VCC-3V3
- J25 pad 2: /Fixture Dev Kit - ADS/I2C-SDA -> GND
- J25 pad 3: GND -> /Fixture Dev Kit - ADS/I2C-SDA
- J25 pad 4: /Fixture Dev Kit - ADS/C4-VCC-3V3 -> /Fixture Dev Kit - ADS/I2C-SCK
- J27 pad 1: /Fixture Dev Kit - ADS/I2C-SCK -> /Fixture Dev Kit - ADS/C4-VCC-3V3
- J27 pad 2: /Fixture Dev Kit - ADS/I2C-SDA -> GND
- J27 pad 3: GND -> /Fixture Dev Kit - ADS/I2C-SDA
- J27 pad 4: /Fixture Dev Kit - ADS/C4-VCC-3V3 -> /Fixture Dev Kit - ADS/I2C-SCK
- J28 pad 1: /Fixture Dev Kit - ADS/I2C-SCK -> /Fixture Dev Kit - ADS/C4-VCC-3V3
- J28 pad 2: /Fixture Dev Kit - ADS/I2C-SDA -> GND
- J28 pad 3: GND -> /Fixture Dev Kit - ADS/I2C-SDA
- J28 pad 4: /Fixture Dev Kit - ADS/C4-VCC-3V3 -> /Fixture Dev Kit - ADS/I2C-SCK
- J36 pad 2: Net-(J36-Pad2) -> /Fixture Dev Kit - DUT/DUT-CHG-IN
- J38 pad 1: Net-(J36-Pad2) -> /Fixture Dev Kit - DUT/DUT-CHG-IN
- J56 pad 31: Net-(J55-Pad61) -> /Fixture Dev Kit - DUT/DUT-CHG-IN
- J56 pad 32: Net-(J55-Pad61) -> /Fixture Dev Kit - DUT/DUT-CHG-IN
- J56 pad 33: Net-(J55-Pad61) -> /Fixture Dev Kit - DUT/DUT-CHG-IN
- J56 pad 34: Net-(J55-Pad61) -> /Fixture Dev Kit - DUT/DUT-CHG-IN
- J56 pad 35: Net-(J55-Pad61) -> /Fixture Dev Kit - DUT/DUT-CHG-IN
- J63 pad 1: /Fixture Dev Kit - PMosfets/Drain0 -> /Fixture Dev Kit - PMosfets/Source0
- J63 pad 2: /Fixture Dev Kit - PMosfets/Gate0 -> /Fixture Dev Kit - PMosfets/Source0
- J63 pad 3: /Fixture Dev Kit - PMosfets/Source0 -> /Fixture Dev Kit - PMosfets/Gate0
- J63 pad 4: /Fixture Dev Kit - PMosfets/Source0 -> /Fixture Dev Kit - PMosfets/Gate0
- J63 pad 5: /Fixture Dev Kit - PMosfets/Gate0 -> Net-(J63-Pad5)
- J64 pad 1: /Fixture Dev Kit - PMosfets/Drain4 -> /Fixture Dev Kit - PMosfets/Source4
- J64 pad 2: /Fixture Dev Kit - PMosfets/Gate4 -> /Fixture Dev Kit - PMosfets/Source4
- J64 pad 3: /Fixture Dev Kit - PMosfets/Source4 -> /Fixture Dev Kit - PMosfets/Gate4
- J64 pad 4: /Fixture Dev Kit - PMosfets/Source4 -> /Fixture Dev Kit - PMosfets/Gate4
- J64 pad 5: /Fixture Dev Kit - PMosfets/Gate4 -> Net-(J64-Pad5)
- J65 pad 1: /Fixture Dev Kit - PMosfets/Drain1 -> /Fixture Dev Kit - PMosfets/Source1
- J65 pad 2: /Fixture Dev Kit - PMosfets/Gate1 -> /Fixture Dev Kit - PMosfets/Source1
- J65 pad 3: /Fixture Dev Kit - PMosfets/Source1 -> /Fixture Dev Kit - PMosfets/Gate1
- J65 pad 4: /Fixture Dev Kit - PMosfets/Source1 -> /Fixture Dev Kit - PMosfets/Gate1
- J65 pad 5: /Fixture Dev Kit - PMosfets/Gate1 -> Net-(J65-Pad5)
- J66 pad 1: /Fixture Dev Kit - PMosfets/Drain5 -> /Fixture Dev Kit - PMosfets/Source5
- J66 pad 2: /Fixture Dev Kit - PMosfets/Gate5 -> /Fixture Dev Kit - PMosfets/Source5
- J66 pad 3: /Fixture Dev Kit - PMosfets/Source5 -> /Fixture Dev Kit - PMosfets/Gate5
- J66 pad 4: /Fixture Dev Kit - PMosfets/Source5 -> /Fixture Dev Kit - PMosfets/Gate5
- J66 pad 5: /Fixture Dev Kit - PMosfets/Gate5 -> Net-(J66-Pad5)
- J67 pad 1: /Fixture Dev Kit - PMosfets/Drain2 -> /Fixture Dev Kit - PMosfets/Source2
- J67 pad 2: /Fixture Dev Kit - PMosfets/Gate2 -> /Fixture Dev Kit - PMosfets/Source2
- J67 pad 3: /Fixture Dev Kit - PMosfets/Source2 -> /Fixture Dev Kit - PMosfets/Gate2
- J67 pad 4: /Fixture Dev Kit - PMosfets/Source2 -> /Fixture Dev Kit - PMosfets/Gate2
- J67 pad 5: /Fixture Dev Kit - PMosfets/Gate2 -> Net-(J67-Pad5)
- J68 pad 1: /Fixture Dev Kit - PMosfets/Drain6 -> /Fixture Dev Kit - PMosfets/Source6
- J68 pad 2: /Fixture Dev Kit - PMosfets/Gate6 -> /Fixture Dev Kit - PMosfets/Source6
- J68 pad 3: /Fixture Dev Kit - PMosfets/Source6 -> /Fixture Dev Kit - PMosfets/Gate6
- J68 pad 4: /Fixture Dev Kit - PMosfets/Source6 -> /Fixture Dev Kit - PMosfets/Gate6
- J68 pad 5: /Fixture Dev Kit - PMosfets/Gate6 -> Net-(J68-Pad5)
- J69 pad 1: /Fixture Dev Kit - PMosfets/Drain3 -> /Fixture Dev Kit - PMosfets/Source3
- J69 pad 2: /Fixture Dev Kit - PMosfets/Gate3 -> /Fixture Dev Kit - PMosfets/Source3
- J69 pad 3: /Fixture Dev Kit - PMosfets/Source3 -> /Fixture Dev Kit - PMosfets/Gate3
- J69 pad 4: /Fixture Dev Kit - PMosfets/Source3 -> /Fixture Dev Kit - PMosfets/Gate3
- J69 pad 5: /Fixture Dev Kit - PMosfets/Gate3 -> Net-(J69-Pad5)
- J70 pad 1: /Fixture Dev Kit - PMosfets/Drain7 -> /Fixture Dev Kit - PMosfets/Source7
- J70 pad 2: /Fixture Dev Kit - PMosfets/Gate7 -> /Fixture Dev Kit - PMosfets/Source7
- J70 pad 3: /Fixture Dev Kit - PMosfets/Source7 -> /Fixture Dev Kit - PMosfets/Gate7
- J70 pad 4: /Fixture Dev Kit - PMosfets/Source7 -> /Fixture Dev Kit - PMosfets/Gate7
- J70 pad 5: /Fixture Dev Kit - PMosfets/Gate7 -> Net-(J70-Pad5)
- J84 pad 1: Net-(J82-Pad2) -> GND
- J84 pad 2: Net-(J82-Pad2) -> GND
- J84 pad 3: Net-(J82-Pad2) -> GND
- J84 pad 31: Net-(J82-Pad62) -> GND
- J84 pad 32: Net-(J82-Pad62) -> GND
- J84 pad 33: Net-(J82-Pad62) -> GND
- J84 pad 34: Net-(J82-Pad62) -> GND
- J84 pad 35: Net-(J82-Pad62) -> GND
- J84 pad 4: Net-(J82-Pad2) -> GND
- J92 pad 1: /Fixture Dev Kit - Functional Computer/I2C-SCK -> /Fixture Dev Kit - ADS/C4-VCC-3V3
- J92 pad 2: /Fixture Dev Kit - Functional Computer/I2C-SDA -> GND
- J92 pad 3: GND -> /Fixture Dev Kit - Functional Computer/I2C-SDA
- J92 pad 4: /Fixture Dev Kit - ADS/C4-VCC-3V3 -> /Fixture Dev Kit - Functional Computer/I2C-SCK
- J93 pad 1: /Fixture Dev Kit - Functional Computer/I2C-SCK -> /Fixture Dev Kit - ADS/C4-VCC-3V3
- J93 pad 2: /Fixture Dev Kit - Functional Computer/I2C-SDA -> GND
- J93 pad 3: GND -> /Fixture Dev Kit - Functional Computer/I2C-SDA
- J93 pad 4: /Fixture Dev Kit - ADS/C4-VCC-3V3 -> /Fixture Dev Kit - Functional Computer/I2C-SCK
- J94 pad 1: /Fixture Dev Kit - Functional Computer/I2C-SCK -> /Fixture Dev Kit - ADS/C4-VCC-3V3
- J94 pad 2: /Fixture Dev Kit - Functional Computer/I2C-SDA -> GND
- J94 pad 3: GND -> /Fixture Dev Kit - Functional Computer/I2C-SDA
- J94 pad 4: /Fixture Dev Kit - ADS/C4-VCC-3V3 -> /Fixture Dev Kit - Functional Computer/I2C-SCK
- J95 pad 1: /Fixture Dev Kit - Functional Computer/I2C-SCK -> /Fixture Dev Kit - ADS/C4-VCC-3V3
- J95 pad 2: /Fixture Dev Kit - Functional Computer/I2C-SDA -> GND
- J95 pad 3: GND -> /Fixture Dev Kit - Functional Computer/I2C-SDA
- J95 pad 4: /Fixture Dev Kit - ADS/C4-VCC-3V3 -> /Fixture Dev Kit - Functional Computer/I2C-SCK
- J98 pad 1: /Fixture Dev Kit - Functional Computer/I2C-SCK -> /Fixture Dev Kit - ADS/C4-VCC-3V3
- J98 pad 2: /Fixture Dev Kit - Functional Computer/I2C-SDA -> GND
- J98 pad 3: GND -> /Fixture Dev Kit - Functional Computer/I2C-SDA
- J98 pad 4: /Fixture Dev Kit - ADS/C4-VCC-3V3 -> /Fixture Dev Kit - Functional Computer/I2C-SCK
- J99 pad 1: /Fixture Dev Kit - Functional Computer/I2C-SCK -> /Fixture Dev Kit - ADS/C4-VCC-3V3
- J99 pad 2: /Fixture Dev Kit - Functional Computer/I2C-SDA -> GND
- J99 pad 3: GND -> /Fixture Dev Kit - Functional Computer/I2C-SDA
- J99 pad 4: /Fixture Dev Kit - ADS/C4-VCC-3V3 -> /Fixture Dev Kit - Functional Computer/I2C-SCK
- R12 pad 2: Net-(D11-Pad2) -> Net-(D12-Pad1)
- R2 pad 2: Net-(D1-Pad2) -> Net-(D2-Pad1)
- R4 pad 2: Net-(D3-Pad2) -> Net-(D4-Pad1)
- R6 pad 2: Net-(D5-Pad2) -> Net-(D6-Pad1)
- R8 pad 2: Net-(D7-Pad2) -> Net-(D8-Pad1)
- R9 pad 1: Net-(D10-Pad1) -> Net-(D9-Pad2)
- TP1 pad 1: Net-(D1-Pad2) -> Net-(D1-Pad1)
- TP2 pad 1: Net-(D1-Pad1) -> Net-(D3-Pad1)
- TP3 pad 1: Net-(D3-Pad2) -> Net-(D5-Pad1)
- TP4 pad 1: Net-(D3-Pad1) -> Net-(D7-Pad1)
- TP5 pad 1: Net-(D5-Pad2) -> Net-(D10-Pad2)
- TP6 pad 1: Net-(D5-Pad1) -> Net-(D11-Pad1)
- TP7 pad 1: Net-(D7-Pad2) -> Net-(D15-Pad1)
- TP8 pad 1: Net-(D7-Pad1) -> Net-(D17-Pad1)
Other:
- board outline removed
- board text added: "3V3"
- board text added: "ADS CIRCUITS"
- board text added: "Audio Jack"
- board text added: "D"
- board text added: "D14"
- board text added: "G"
- board text added: "GND"
- board text added: "INA CIRCUITS"
- board text added: "PWRON"
- board text added: "PWRSW"
- board text added: "S"
- board text added: "SCK"
- board text added: "SDA"
- board text added: "USB-A"
