File: HARDWARE/v0.01/KiCad/Fixture-Dev-Kit.kicad_pcb (KiCad board)
At the start: 2 copper layers, 151.4 x 138.2 mm, 381 parts, among them J1 POWER, J10 LED_3, J100 INA_43, J101 INA_43, J102 INA_41, J103 INA_43, J104 INA, J105 INA, J106 LED_6, J107 LED_7, J11 SW_5, J12 LED_4, J13 SW_6, J14 LED_5, J15 SW_7, J16 ADS_48, J17 ADS_48, J18 ADS_4A, J19 ADS_4A, J2 LED_0, J20 ADS_48, J21 ADS_4A, J22 ADS, J23 ADS, J24 ADS_49, J25 ADS_49, J26 ADS_49, J27 ADS_4B, J28 ADS_4B, J29 ADS_4B, J3 SW_0, J30 LOAD_0, J31 LOAD_1, J32 LOAD_2, J33 LOAD_3, J34 Conn_01x20, J35 BAT, J36 CHIP4LH, J37 USB_OTG, J38 Conn_01x20, J39 VBUS, J4 SW_1, J40 VBUS, J41 B_D+, J42 D-TP's, J43 B_D-, J44 USB_ID, J45 UPDATE, J46 ANT--SELECT, J47 Conn_01x20, J49 VBUS, J5 LED_1, J50 A_D+, J51 A_D-, J52 CHIP4RH, J53 Conn_01x20, J54 Conn_01x35, J56 Conn_01x35, J57 IOExp_0, J58 IOExp_0, J59 Conn_01x24, J6 SW_2, J60 IOExp_0, J61 IOExp_0, J62 Conn_01x24, J63 FET_0, J64 FET_0, J65 FET_0, J66 FET_0, J67 FET_0, J68 FET_0, J69 FET_0, J7 LED_2, J70 FET_0, J71 NFET_0, J72 NFET_4, J73 NFET_1, J74 NFET_5, J75 NFET_2, J76 NFET_6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

Commit message: quasi-redoing entire schematic and layout
Parts:
- removed C10, C11, C12: 0.1uF, Capacitors_SMD:C_0805_HandSoldering
- removed D18: Green, LEDs:LED_0805_HandSoldering
- removed J100, J101: INA_43, Pin_Headers:Pin_Header_Straight_1x04_Pitch2.54mm
- removed J102: INA_41, Pin_Headers:Pin_Header_Straight_1x02_Pitch2.54mm
- removed J103: INA_43, Pin_Headers:Pin_Header_Straight_1x02_Pitch2.54mm
- removed J104, J105: INA, Pin_Headers:Pin_Header_Straight_1x04_Pitch2.54mm
- removed J106: LED_6, Pin_Headers:Pin_Header_Straight_1x03_Pitch2.54mm
- removed J107: LED_7, Pin_Headers:Pin_Header_Straight_1x03_Pitch2.54mm
- removed J22: ADS, Pin_Headers:Pin_Header_Straight_1x04_Pitch2.54mm
- removed J26: ADS_49, Pin_Headers:Pin_Header_Straight_1x04_Pitch2.54mm
- removed J32: LOAD_2, Pin_Headers:Pin_Header_Straight_1x03_Pitch2.54mm
- removed J33: LOAD_3, Pin_Headers:Pin_Header_Straight_1x03_Pitch2.54mm
- removed J34, J38, J47, J53, J86, J87, J90, J91: Conn_01x20, Pin_Headers:Pin_Header_Straight_1x20_Pitch2.54mm
- removed J35: BAT, Connectors_JST:JST_PH_S2B-PH-K_02x2.00mm_Angled
- removed J36, J88: CHIP4LH, Pin_Headers:Pin_Header_Straight_2x20_Pitch2.54mm
- removed J37: USB_OTG, Connectors_USB:USB_Micro-B_Molex_47346-0001
- removed J39, J40, J49: VBUS, Pin_Headers:Pin_Header_Angled_1x01_Pitch2.54mm
- removed J41: B_D+, Pin_Headers:Pin_Header_Angled_1x01_Pitch2.54mm
- removed J42: D-TP's, Pin_Headers:Pin_Header_Straight_1x02_Pitch2.54mm
- removed J43: B_D-, Pin_Headers:Pin_Header_Angled_1x01_Pitch2.54mm
- removed J44: USB_ID, Pin_Headers:Pin_Header_Angled_1x01_Pitch2.54mm
- removed J45: UPDATE, Pin_Headers:Pin_Header_Angled_1x01_Pitch2.54mm
- removed J46: ANT--SELECT, Pin_Headers:Pin_Header_Angled_1x01_Pitch2.54mm
- removed J50: A_D+, Pin_Headers:Pin_Header_Angled_1x01_Pitch2.54mm
- removed J51: A_D-, Pin_Headers:Pin_Header_Angled_1x01_Pitch2.54mm
- removed J52, J89: CHIP4RH, Pin_Headers:Pin_Header_Straight_2x20_Pitch2.54mm
- removed J54, J56, J80, J84: Conn_01x35, Pin_Headers:Pin_Header_Straight_1x35_Pitch2.54mm
- removed J57, J58, J60, J61: IOExp_0, Pin_Headers:Pin_Header_Straight_1x04_Pitch2.54mm
- removed J59, J62: Conn_01x24, Pin_Headers:Pin_Header_Straight_1x24_Pitch2.54mm
- removed J63, J64, J65, J66, J67, J68, J69, J70: FET_0, Pin_Headers:Pin_Header_Straight_2x03_Pitch2.54mm
- removed J71: NFET_0, Pin_Headers:Pin_Header_Straight_2x03_Pitch2.54mm
- removed J72: NFET_4, Pin_Headers:Pin_Header_Straight_2x03_Pitch2.54mm
- removed J73: NFET_1, Pin_Headers:Pin_Header_Straight_2x03_Pitch2.54mm
- removed J74: NFET_5, Pin_Headers:Pin_Header_Straight_2x03_Pitch2.54mm
- removed J75: NFET_2, Pin_Headers:Pin_Header_Straight_2x03_Pitch2.54mm
- removed J76: NFET_6, Pin_Headers:Pin_Header_Straight_2x03_Pitch2.54mm
- removed J77: NFET_3, Pin_Headers:Pin_Header_Straight_2x03_Pitch2.54mm
- removed J78: NFET_7, Pin_Headers:Pin_Header_Straight_2x03_Pitch2.54mm
- removed J79: JST-2P-RA, Connectors_JST:JST_PH_S2B-PH-K_02x2.00mm_Angled
- removed J83: VBUS, Pin_Headers:Pin_Header_Straight_1x02_Pitch2.54mm
- removed J92, J93: INA_40, Pin_Headers:Pin_Header_Straight_1x04_Pitch2.54mm
- removed J94, J95: INA_42, Pin_Headers:Pin_Header_Straight_1x04_Pitch2.54mm
- removed J96: INA_40, Pin_Headers:Pin_Header_Straight_1x02_Pitch2.54mm
- removed J97: INA_42, Pin_Headers:Pin_Header_Straight_1x02_Pitch2.54mm
- removed J98, J99: INA_41, Pin_Headers:Pin_Header_Straight_1x04_Pitch2.54mm
- removed P2: USB-A1HSW6, USB-A1HSW6:OST_USB-A1HSW6
- removed Q17, Q18, Q19, Q20: FDN337N, FDN337N:SSOT-3
- removed R56, R57, R58, R59, R60, R61, R62, R63, R64, R65, R66, R67, R68, R69, R70, R71, R72, R73, R74, R75, R76, R77, R78, R79, R80, R81, R82, R83: DNP, Resistors_SMD:R_0805_HandSoldering
- removed R84, R85: 0R, Resistors_SMD:R_0805_HandSoldering
- removed R86, R87, R88, R89, R90, R91, R92, R93, R96, R97, R98, R99: 1K, Resistors_SMD:R_0805_HandSoldering
- removed R94: 47K, Resistors_SMD:R_0805_HandSoldering
- removed R95: 10K, Resistors_SMD:R_0805_HandSoldering
- removed TP100: G6, TestPoint:TestPoint
- removed TP101, TP102, TP31, TP32, TP33, TP34, TP35, TP36, TP37, TP38, TP39, TP40, TP41, TP42, TP43, TP44, TP45, TP46, TP47, TP48, TP49, TP50, TP51, TP52, TP53, TP54, TP55, TP56, TP57, TP58, TP59, TP60, TP61, TP62, TP63, TP64, TP65, TP66, TP67, TP68, TP69, TP70, TP71, TP72, TP73, TP74, TP75, TP76, TP77, TP78, TP79, TP80, TP83, TP84, TP85, TP86, TP89, TP90, TP91, TP92, TP95, TP96, TP97, TP98: TEST, TestPoint:TestPoint
- removed TP103: D-, TestPoint:TestPoint
- removed TP104: D+, TestPoint:TestPoint
- removed TP105, TP107, TP109, TP111: V+, TestPoint:TestPoint
- removed TP106, TP108, TP110, TP112: V-, TestPoint:TestPoint
- removed TP11: VS, TestPoint:TestPoint
- removed TP12: SIG, TestPoint:TestPoint
- removed TP13, TP16, TP19, TP22: S, TestPoint:TestPoint
- removed TP14, TP17, TP20, TP23: G, TestPoint:TestPoint
- removed TP15, TP18, TP21, TP24: D, TestPoint:TestPoint
- removed TP25: VBUS, TestPoint:TestPoint
- removed TP26: B_D+, TestPoint:TestPoint
- removed TP27: B_D-, TestPoint:TestPoint
- removed TP28: USB-ID, TestPoint:TestPoint
- removed TP29: A_D+, TestPoint:TestPoint
- removed TP30: A_D-, TestPoint:TestPoint
- removed TP81: G0, TestPoint:TestPoint
- removed TP82, TP99: G3, TestPoint:TestPoint
- removed TP87: G1, TestPoint:TestPoint
- removed TP88: G4, TestPoint:TestPoint
- removed TP93: G2, TestPoint:TestPoint
- removed TP94: G5, TestPoint:TestPoint
- removed U10, U7, U8, U9: INA219BIDCNT, INA219BIDCNR:SOT65P280X145-8N
- removed U6: TCA6424ARGJR, TCA6424ARGJR:QFN50P500X500X60-33N
- added F3: 1.5A, 1206:1206, F.Cu at (194.3, 223.7)
- added F4: 1.5A, 1206:1206, F.Cu at (224.1, 195.5)
- added F5: 1.5A, 1206:1206, F.Cu at (229.5, 189.9)
- added P1: USB-A1HSW6, USB-A1HSW6:OST_USB-A1HSW6, F.Cu at (217.8, 81.7)
- C1, C2, C3, C4: value 0.1uF -> 1uf
- C5, C6, C7, C8: value 1uf -> 0.1uF
- D10, D12: value Green -> LNJP12X8ARA; footprint LEDs:LED_0805_HandSoldering -> 1206:1206
- D11: value Purple -> LNJP12X8ARA; footprint LEDs:LED_0805_HandSoldering -> 1206:1206
- D13: footprint LEDs:LED_0805_HandSoldering -> 1206:1206
- D14: value LNJP12X8ARA -> LED; footprint LEDs:LED_0805_HandSoldering -> 1206:1206
- D15, D17: value Purple -> LED; footprint LEDs:LED_0805_HandSoldering -> 1206:1206
- D16: value Green -> LED; footprint LEDs:LED_0805_HandSoldering -> 1206:1206
- D2, D4: value Green -> Purple
- D5, D7: value Purple -> Green
- D9: value Purple -> LNJP12X8ARA
- F2: value 1206SFP300F -> 1.5A
- J1: value POWER -> DUT; footprint TerminalBlocks_Phoenix:TerminalBlock_Phoenix_MPT-2.54mm_2pol -> Pin_Headers:Pin_Header_Straight_2x10_Pitch2.54mm
- J10: value LED_3 -> SW_3; footprint Pin_Headers:Pin_Header_Straight_1x03_Pitch2.54mm -> Pin_Headers:Pin_Header_Straight_1x04_Pitch2.54mm
- J11: value SW_5 -> FET_0; footprint Pin_Headers:Pin_Header_Straight_1x04_Pitch2.54mm -> Pin_Headers:Pin_Header_Straight_2x03_Pitch2.54mm
- J12: value LED_4 -> FET_0; footprint Pin_Headers:Pin_Header_Straight_1x03_Pitch2.54mm -> Pin_Headers:Pin_Header_Straight_2x03_Pitch2.54mm
- J13: value SW_6 -> NFET_0; footprint Pin_Headers:Pin_Header_Straight_1x04_Pitch2.54mm -> Pin_Headers:Pin_Header_Straight_2x03_Pitch2.54mm
- J14: value LED_5 -> NFET_1; footprint Pin_Headers:Pin_Header_Straight_1x03_Pitch2.54mm -> Pin_Headers:Pin_Header_Straight_2x03_Pitch2.54mm
- J15: value SW_7 -> Conn_01x20; footprint Pin_Headers:Pin_Header_Straight_1x04_Pitch2.54mm -> Pin_Headers:Pin_Header_Straight_1x20_Pitch2.54mm
- J16, J20: value ADS_48 -> Conn_01x20; footprint Pin_Headers:Pin_Header_Straight_1x04_Pitch2.54mm -> Pin_Headers:Pin_Header_Straight_1x20_Pitch2.54mm
- J17: value ADS_48 -> CHIP4RH; footprint Pin_Headers:Pin_Header_Straight_1x04_Pitch2.54mm -> Pin_Headers:Pin_Header_Straight_2x20_Pitch2.54mm
- J18, J19: value ADS_4A -> Conn_01x35; footprint Pin_Headers:Pin_Header_Straight_1x04_Pitch2.54mm -> Pin_Headers:Pin_Header_Straight_1x35_Pitch2.54mm
- J2: value LED_0 -> POWER; footprint Pin_Headers:Pin_Header_Straight_1x03_Pitch2.54mm -> TerminalBlocks_Phoenix:TerminalBlock_Phoenix_MPT-2.54mm_2pol
- J21: value ADS_4A -> Conn_01x20; footprint Pin_Headers:Pin_Header_Straight_1x04_Pitch2.54mm -> Pin_Headers:Pin_Header_Straight_1x20_Pitch2.54mm
- J23: value ADS -> CHIP4LH; footprint Pin_Headers:Pin_Header_Straight_1x04_Pitch2.54mm -> Pin_Headers:Pin_Header_Straight_2x20_Pitch2.54mm
- J24: value ADS_49 -> VBUS; footprint Pin_Headers:Pin_Header_Straight_1x04_Pitch2.54mm -> Pin_Headers:Pin_Header_Straight_1x02_Pitch2.54mm
- J25: value ADS_49 -> JST-2P-RA; footprint Pin_Headers:Pin_Header_Straight_1x04_Pitch2.54mm -> Connectors_JST:JST_PH_S2B-PH-K_02x2.00mm_Angled
- J27, J28, J29: value ADS_4B -> INA_40; footprint Pin_Headers:Pin_Header_Straight_1x04_Pitch2.54mm -> Pin_Headers:Pin_Header_Straight_1x02_Pitch2.54mm
- J3: value SW_0 -> LED_0; footprint Pin_Headers:Pin_Header_Straight_1x04_Pitch2.54mm -> Pin_Headers:Pin_Header_Straight_1x03_Pitch2.54mm
- J30: value LOAD_0 -> INA_40; footprint Pin_Headers:Pin_Header_Straight_1x03_Pitch2.54mm -> Pin_Headers:Pin_Header_Straight_1x02_Pitch2.54mm
- J31: value LOAD_1 -> ADS; footprint Pin_Headers:Pin_Header_Straight_1x03_Pitch2.54mm -> Pin_Headers:Pin_Header_Straight_1x04_Pitch2.54mm
- J4: value SW_1 -> LED_1; footprint Pin_Headers:Pin_Header_Straight_1x04_Pitch2.54mm -> Pin_Headers:Pin_Header_Straight_1x03_Pitch2.54mm
- J5: value LED_1 -> LED_2
- J6: value SW_2 -> LED_3; footprint Pin_Headers:Pin_Header_Straight_1x04_Pitch2.54mm -> Pin_Headers:Pin_Header_Straight_1x03_Pitch2.54mm
- J7: value LED_2 -> SW_0; footprint Pin_Headers:Pin_Header_Straight_1x03_Pitch2.54mm -> Pin_Headers:Pin_Header_Straight_1x04_Pitch2.54mm
- J8: value SW_3 -> SW_1
- J9: value SW_4 -> SW_2
- Q10, Q11, Q12, Q5, Q6, Q7, Q8, Q9: value NTF2955T1G -> NTF2955-D; footprint TO_SOT_Packages_SMD:SOT-223 -> NTF2955T1G:SOT230P700X180-4N
- Q3, Q4: value NTF2955T1G -> FDN337N; footprint TO_SOT_Packages_SMD:SOT-223 -> FDN337N:SSOT-3
- R10, R11, R12, R13, R14, R15, R16, R9: value 1K -> DNP
- R17, R18: value 1K -> 0R
- R19: value 1K -> 10K
- R20, R21, R30, R31, R40, R41, R42, R43: value 1K -> 160R
- R22, R23, R32, R33: value 1K -> 10R 5W; footprint Resistors_SMD:R_0805_HandSoldering -> RES_TWM3J560E:RES_TWM3J560E
- R24, R25, R34, R35: value 1K -> 0.1R
- R44: value 1K -> 10R5W; footprint Resistors_SMD:R_0805_HandSoldering -> RES_TWM3J560E:RES_TWM3J560E
- R45, R46, R47: value SQP500JB-10R -> 10R5W
- R48: value SQP500JB-10R -> 1K; footprint RES_TWM3J560E:RES_TWM3J560E -> Resistors_SMD:R_0805_HandSoldering
- R49: value 10K -> 1K
- R52, R53, R54, R55: value DNP -> 1K
- TP10, TP7, TP8: value SIG -> TEST
- TP5: value SIG -> G0
- TP6: value SIG -> G1
- TP9: value VS -> TEST
- U1, U2, U3, U4: value ADS1015IDGST -> INA219BIDCNT; footprint ADS1015IDGST:SOP50P490X110-10N -> INA219BIDCNR:SOT65P280X145-8N
- U5: value TCA6424ARGJR -> ADS1015IDGST; footprint TCA6424ARGJR:QFN50P500X500X60-33N -> ADS1015IDGST:SOP50P490X110-10N
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Connections:
- C1 pad 1: /Fixture Dev Kit - ADS/C4-VCC-3V3 -> Net-(C1-Pad1)
- C1 pad 2: GND -> (no net)
- C2 pad 1: /Fixture Dev Kit - ADS/C4-VCC-3V3 -> Net-(C2-Pad1)
- C2 pad 2: GND -> (no net)
- C3 pad 1: /Fixture Dev Kit - ADS/C4-VCC-3V3 -> /Fixture Dev Kit - Functional Computer/LOLN
- C4 pad 1: /Fixture Dev Kit - ADS/C4-VCC-3V3 -> /Fixture Dev Kit - Functional Computer/LORN
- C5 pad 1: Net-(C5-Pad1) -> GND
- C6 pad 1: Net-(C6-Pad1) -> GND
- C7 pad 1: /Fixture Dev Kit - Functional Computer/LOLN -> GND
- C7 pad 2: GND -> Net-(C7-Pad2)
- C8 pad 1: /Fixture Dev Kit - Functional Computer/LORN -> GND
- C8 pad 2: GND -> Net-(C8-Pad2)
- C9 pad 1: GND -> +5V
- C9 pad 2: Net-(C9-Pad2) -> GND
- D10 pad 1: Net-(D10-Pad1) -> /Fixture Dev Kit - INA/INA40_XIO
- D11 pad 1: Net-(D11-Pad1) -> /Fixture Dev Kit - INA/INA41_XIO
- D12 pad 1: Net-(D12-Pad1) -> /Fixture Dev Kit - INA/INA42_XIO
- D12 pad 2: Net-(D11-Pad1) -> Net-(D12-Pad2)
- D13 pad 1: GND -> /Fixture Dev Kit - INA/INA43_XIO
- D14 pad 1: GND -> /Fixture Dev Kit - ADS/AIN0_XIO
- D14 pad 2: /Fixture Dev Kit - ADS/C4-VCC-3V3 -> Net-(D14-Pad2)
- D15 pad 1: Net-(D15-Pad1) -> /Fixture Dev Kit - ADS/AIN1_XIO
- D16 pad 1: Net-(D16-Pad1) -> /Fixture Dev Kit - ADS/AIN2_XIO
- D16 pad 2: Net-(D15-Pad1) -> Net-(D16-Pad2)
- D17 pad 1: Net-(D17-Pad1) -> /Fixture Dev Kit - ADS/AIN3_XIO
- D2 pad 2: Net-(D1-Pad1) -> Net-(D2-Pad2)
- D4 pad 2: Net-(D3-Pad1) -> Net-(D4-Pad2)
- D5 pad 2: Net-(D5-Pad2) -> Net-(D1-Pad1)
- D6 pad 2: Net-(D5-Pad1) -> Net-(D2-Pad1)
- D7 pad 2: Net-(D7-Pad2) -> Net-(D3-Pad1)
- D8 pad 2: Net-(D7-Pad1) -> Net-(D4-Pad1)
- D9 pad 1: Net-(D10-Pad2) -> GND
- D9 pad 2: Net-(D9-Pad2) -> /C4-VCC-3V3
- F1 pad 1: Net-(F1-Pad1) -> (no net)
- F2 pad 2: /Fixture Dev Kit - DUT/DUT-CHG-IN -> +5V
- J1 pad 1: GND -> /AIN0
- J1 pad 2: +5V -> /AIN1
- J10 pad 1: Net-(J10-Pad1) -> (no net)
- J10 pad 2: Net-(D7-Pad1) -> (no net)
- J10 pad 3: GND -> (no net)
- J11 pad 1: Net-(J11-Pad1) -> /Fixture Dev Kit - PMosfets/Source0
- J11 pad 2: Net-(J11-Pad2) -> /Fixture Dev Kit - PMosfets/Source0
- J11 pad 3: Net-(J11-Pad3) -> /Fixture Dev Kit - PMosfets/Gate0
- J11 pad 4: Net-(J11-Pad4) -> /Fixture Dev Kit - PMosfets/Gate0
- J12 pad 1: Net-(J12-Pad1) -> /Fixture Dev Kit - PMosfets/Source1
- J12 pad 2: Net-(D10-Pad2) -> /Fixture Dev Kit - PMosfets/Source1
- J12 pad 3: GND -> /Fixture Dev Kit - PMosfets/Gate1
- J13 pad 1: Net-(J13-Pad1) -> /Fixture Dev Kits - NMosfets/Source_0
- J13 pad 2: Net-(J13-Pad2) -> /Fixture Dev Kits - NMosfets/Source_0
- J13 pad 3: Net-(J13-Pad3) -> /Fixture Dev Kits - NMosfets/Gate_0
- J13 pad 4: Net-(J13-Pad4) -> /Fixture Dev Kits - NMosfets/Gate_0
- J14 pad 1: Net-(J14-Pad1) -> /Fixture Dev Kits - NMosfets/Source_1
- J14 pad 2: Net-(D11-Pad1) -> /Fixture Dev Kits - NMosfets/Source_1
- J14 pad 3: GND -> /Fixture Dev Kits - NMosfets/Gate_1
- J15 pad 1: Net-(J15-Pad1) -> GND
- J15 pad 2: Net-(J15-Pad2) -> /UART-TX
- J15 pad 3: Net-(J15-Pad3) -> /UART-RX
- J16 pad 1: /Fixture Dev Kit - ADS/C4-VCC-3V3 -> Net-(J16-Pad1)
- J16 pad 2: GND -> /Fixture Dev Kit - Functional Computer/LOLP
- J16 pad 3: /Fixture Dev Kit - ADS/I2C-SDA -> /Fixture Dev Kit - Functional Computer/LOLN
- J16 pad 4: /Fixture Dev Kit - ADS/I2C-SCK -> /Fixture Dev Kit - Functional Computer/LORP
- J17 pad 1: /Fixture Dev Kit - ADS/C4-VCC-3V3 -> GND
- J17 pad 2: GND -> Net-(J16-Pad1)
- J17 pad 3: /Fixture Dev Kit - ADS/I2C-SDA -> /UART-TX
- J17 pad 4: /Fixture Dev Kit - ADS/I2C-SCK -> /Fixture Dev Kit - Functional Computer/LOLP
- J18 pad 1: /Fixture Dev Kit - ADS/C4-VCC-3V3 -> /Fixture Dev Kit - Functional Computer/BAT
- J18 pad 2: GND -> /Fixture Dev Kit - Functional Computer/BAT
- J18 pad 3: /Fixture Dev Kit - ADS/I2C-SDA -> /Fixture Dev Kit - Functional Computer/BAT
- J18 pad 4: /Fixture Dev Kit - ADS/I2C-SCK -> /Fixture Dev Kit - Functional Computer/BAT
- J19 pad 1: /Fixture Dev Kit - ADS/C4-VCC-3V3 -> GND
- J19 pad 3: /Fixture Dev Kit - ADS/I2C-SDA -> GND
- J19 pad 4: /Fixture Dev Kit - ADS/I2C-SCK -> GND
- J2 pad 1: Net-(J2-Pad1) -> GND
- J2 pad 2: Net-(D1-Pad1) -> +5V
- J20 pad 1: Net-(J20-Pad1) -> GND
- J21 pad 1: Net-(J21-Pad1) -> /Fixture Dev Kit - Functional Computer/C4-PWR-IN
- J21 pad 2: Net-(J21-Pad2) -> GND
- J21 pad 3: Net-(J21-Pad3) -> /Fixture Dev Kit - Functional Computer/TS
- J21 pad 4: Net-(J21-Pad4) -> /Fixture Dev Kit - Functional Computer/BAT
- J23 pad 1: /Fixture Dev Kit - ADS/I2C-SCK -> GND
- J23 pad 2: /Fixture Dev Kit - ADS/I2C-SDA -> /Fixture Dev Kit - Functional Computer/C4-PWR-IN
- J23 pad 3: GND -> Net-(J20-Pad2)
- J23 pad 4: /Fixture Dev Kit - ADS/C4-VCC-3V3 -> GND
- J24 pad 1: /Fixture Dev Kit - ADS/C4-VCC-3V3 -> Net-(J24-Pad1)
- J24 pad 2: GND -> Net-(J24-Pad1)
- J25 pad 1: /Fixture Dev Kit - ADS/C4-VCC-3V3 -> GND
- J25 pad 2: GND -> /Fixture Dev Kit - Functional Computer/BAT
- J27 pad 1: /Fixture Dev Kit - ADS/C4-VCC-3V3 -> /Fixture Dev Kit - INA/LOAD40_XIO
- J27 pad 2: GND -> /Fixture Dev Kit - INA/INA40_XIO
- J28 pad 1: /Fixture Dev Kit - ADS/C4-VCC-3V3 -> /Fixture Dev Kit - INA/LOAD41_XIO
- J28 pad 2: GND -> /Fixture Dev Kit - INA/INA41_XIO
- J29 pad 1: Net-(J29-Pad1) -> /Fixture Dev Kit - INA/LOAD42_XIO
- J29 pad 2: Net-(J29-Pad2) -> /Fixture Dev Kit - INA/INA42_XIO
- J3 pad 2: Net-(J3-Pad2) -> Net-(D1-Pad1)
- J3 pad 3: Net-(J3-Pad3) -> GND
- J30 pad 1: Net-(J30-Pad1) -> /Fixture Dev Kit - INA/LOAD43_XIO
- J30 pad 2: Net-(J30-Pad2) -> /Fixture Dev Kit - INA/INA43_XIO
- J31 pad 1: Net-(J31-Pad1) -> /Fixture Dev Kit - ADS/AIN0_XIO
- J31 pad 2: Net-(J31-Pad2) -> /Fixture Dev Kit - ADS/AIN1_XIO
- J31 pad 3: Net-(J31-Pad3) -> /Fixture Dev Kit - ADS/AIN2_XIO
- J4 pad 2: Net-(J4-Pad2) -> Net-(D2-Pad1)
- J4 pad 3: Net-(J4-Pad3) -> GND
- J6 pad 2: Net-(J6-Pad2) -> Net-(D4-Pad1)
- J6 pad 3: Net-(J6-Pad3) -> GND
- J7 pad 1: Net-(J7-Pad1) -> (no net)
- J7 pad 2: Net-(D5-Pad1) -> (no net)
- J7 pad 3: GND -> (no net)
- J8 pad 1: Net-(J8-Pad1) -> (no net)
- J8 pad 2: Net-(J8-Pad2) -> (no net)
- J8 pad 3: Net-(J8-Pad3) -> (no net)
- J8 pad 4: Net-(J8-Pad4) -> (no net)
- J9 pad 1: Net-(J9-Pad1) -> (no net)
- J9 pad 2: Net-(J9-Pad2) -> (no net)
- J9 pad 3: Net-(J9-Pad3) -> (no net)
- J9 pad 4: Net-(J9-Pad4) -> (no net)
- JP2 pad 1: /Fixture Dev Kit - ADS/C4-VCC-3V3 -> /C4-VCC-3V3
- JP2 pad 2: Net-(C9-Pad2) -> Net-(C5-Pad2)
- JP3 pad 1: /Fixture Dev Kit - ADS/C4-VCC-3V3 -> /C4-VCC-3V3
- JP3 pad 2: Net-(C10-Pad2) -> Net-(C6-Pad2)
- JP4 pad 1: /Fixture Dev Kit - ADS/C4-VCC-3V3 -> /C4-VCC-3V3
- JP4 pad 2: Net-(C11-Pad2) -> Net-(C7-Pad2)
- JP5 pad 1: /Fixture Dev Kit - ADS/C4-VCC-3V3 -> /C4-VCC-3V3
- JP5 pad 2: Net-(C12-Pad2) -> Net-(C8-Pad2)
- Q1 pad 1: Net-(J30-Pad2) -> /Fixture Dev Kit - PMosfets/Gate0
- Q1 pad 2: Net-(Q1-Pad2) -> /Fixture Dev Kit - PMosfets/Drain0
- Q1 pad 3: Net-(J30-Pad3) -> /Fixture Dev Kit - PMosfets/Source0
- Q1 pad 4: Net-(Q1-Pad2) -> /Fixture Dev Kit - PMosfets/Drain0
- Q10 pad 1: /Fixture Dev Kit - PMosfets/Gate6 -> /Fixture Dev Kit - INA/LOAD43_XIO
- Q10 pad 2: /Fixture Dev Kit - PMosfets/Drain6 -> Net-(Q10-Pad2)
- Q10 pad 3: /Fixture Dev Kit - PMosfets/Source6 -> GND
- Q10 pad 4: /Fixture Dev Kit - PMosfets/Drain6 -> Net-(Q10-Pad2)
- Q11 pad 1: /Fixture Dev Kit - PMosfets/Gate3 -> /Fixture Dev Kit - INA/INA42_XIO
- Q11 pad 2: /Fixture Dev Kit - PMosfets/Drain3 -> Net-(Q11-Pad2)
- Q11 pad 3: /Fixture Dev Kit - PMosfets/Source3 -> Net-(F4-Pad1)
- Q11 pad 4: /Fixture Dev Kit - PMosfets/Drain3 -> Net-(Q11-Pad2)
- Q12 pad 1: /Fixture Dev Kit - PMosfets/Gate7 -> /Fixture Dev Kit - INA/INA43_XIO
- Q12 pad 2: /Fixture Dev Kit - PMosfets/Drain7 -> Net-(Q12-Pad2)
- Q12 pad 3: /Fixture Dev Kit - PMosfets/Source7 -> Net-(F5-Pad1)
- Q12 pad 4: /Fixture Dev Kit - PMosfets/Drain7 -> Net-(Q12-Pad2)
- Q13 pad 1: /Fixture Dev Kits - NMosfets/Gate_0 -> /Fixture Dev Kit - ADS/AIN0_XIO
- Q13 pad 2: /Fixture Dev Kits - NMosfets/Source_0 -> Net-(Q13-Pad2)
- Q13 pad 3: /Fixture Dev Kits - NMosfets/Drain_0 -> GND
- Q14 pad 1: /Fixture Dev Kits - NMosfets/Gate_4 -> /Fixture Dev Kit - ADS/AIN1_XIO
- Q14 pad 2: /Fixture Dev Kits - NMosfets/Drain_4 -> Net-(Q14-Pad2)
- Q14 pad 3: /Fixture Dev Kits - NMosfets/Drain_4 -> GND
- Q15 pad 1: /Fixture Dev Kits - NMosfets/Gate_1 -> /Fixture Dev Kit - ADS/AIN2_XIO
- Q15 pad 2: /Fixture Dev Kits - NMosfets/Source_1 -> Net-(Q15-Pad2)
- Q15 pad 3: /Fixture Dev Kits - NMosfets/Drain_1 -> GND
- Q16 pad 1: /Fixture Dev Kits - NMosfets/Gate_5 -> /Fixture Dev Kit - ADS/AIN3_XIO
- Q16 pad 2: /Fixture Dev Kits - NMosfets/Drain_5 -> Net-(Q16-Pad2)
- Q16 pad 3: /Fixture Dev Kits - NMosfets/Drain_5 -> GND
- Q2 pad 1: Net-(J31-Pad2) -> /Fixture Dev Kit - PMosfets/Gate1
- Q2 pad 2: Net-(Q2-Pad2) -> /Fixture Dev Kit - PMosfets/Drain1
- Q2 pad 3: Net-(J31-Pad3) -> /Fixture Dev Kit - PMosfets/Source1
- Q2 pad 4: Net-(Q2-Pad2) -> /Fixture Dev Kit - PMosfets/Drain1
- Q3 pad 1: Net-(J32-Pad2) -> /Fixture Dev Kits - NMosfets/Gate_0
- Q3 pad 2: Net-(Q3-Pad2) -> /Fixture Dev Kits - NMosfets/Source_0
- Q3 pad 3: Net-(J32-Pad3) -> /Fixture Dev Kits - NMosfets/Drain_0
- Q4 pad 1: Net-(J33-Pad2) -> /Fixture Dev Kits - NMosfets/Gate_1
- Q4 pad 2: Net-(Q4-Pad2) -> /Fixture Dev Kits - NMosfets/Source_1
- Q4 pad 3: Net-(J33-Pad3) -> /Fixture Dev Kits - NMosfets/Drain_1
- Q5 pad 1: /Fixture Dev Kit - PMosfets/Gate0 -> /Fixture Dev Kit - INA/LOAD40_XIO
- Q5 pad 2: /Fixture Dev Kit - PMosfets/Drain0 -> Net-(Q5-Pad2)
- Q5 pad 3: /Fixture Dev Kit - PMosfets/Source0 -> GND
- Q5 pad 4: /Fixture Dev Kit - PMosfets/Drain0 -> Net-(Q5-Pad2)
- Q6 pad 1: /Fixture Dev Kit - PMosfets/Gate4 -> /Fixture Dev Kit - INA/LOAD41_XIO
- Q6 pad 2: /Fixture Dev Kit - PMosfets/Drain4 -> Net-(Q6-Pad2)
- Q6 pad 3: /Fixture Dev Kit - PMosfets/Source4 -> GND
- Q6 pad 4: /Fixture Dev Kit - PMosfets/Drain4 -> Net-(Q6-Pad2)
- Q7 pad 1: /Fixture Dev Kit - PMosfets/Gate1 -> /Fixture Dev Kit - INA/INA40_XIO
- Q7 pad 2: /Fixture Dev Kit - PMosfets/Drain1 -> Net-(Q7-Pad2)
- Q7 pad 3: /Fixture Dev Kit - PMosfets/Source1 -> Net-(F2-Pad1)
- Q7 pad 4: /Fixture Dev Kit - PMosfets/Drain1 -> Net-(Q7-Pad2)
- Q8 pad 1: /Fixture Dev Kit - PMosfets/Gate5 -> /Fixture Dev Kit - INA/INA41_XIO
- Q8 pad 2: /Fixture Dev Kit - PMosfets/Drain5 -> Net-(Q8-Pad2)
- Q8 pad 3: /Fixture Dev Kit - PMosfets/Source5 -> Net-(F3-Pad1)
- Q8 pad 4: /Fixture Dev Kit - PMosfets/Drain5 -> Net-(Q8-Pad2)
- Q9 pad 1: /Fixture Dev Kit - PMosfets/Gate2 -> /Fixture Dev Kit - INA/LOAD42_XIO
- Q9 pad 2: /Fixture Dev Kit - PMosfets/Drain2 -> Net-(Q9-Pad2)
- Q9 pad 3: /Fixture Dev Kit - PMosfets/Source2 -> GND
- Q9 pad 4: /Fixture Dev Kit - PMosfets/Drain2 -> Net-(Q9-Pad2)
- R1 pad 2: Net-(J2-Pad1) -> Net-(J3-Pad1)
- R10 pad 1: GND -> /Fixture Dev Kit - PMosfets/Source0
- R10 pad 2: Net-(D10-Pad1) -> /Fixture Dev Kit - PMosfets/Gate0
- R11 pad 1: Net-(D11-Pad2) -> /Fixture Dev Kit - PMosfets/Gate1
- R11 pad 2: Net-(J14-Pad1) -> /Fixture Dev Kit - PMosfets/Drain1
- R12 pad 1: GND -> /Fixture Dev Kit - PMosfets/Source1
- R12 pad 2: Net-(D12-Pad1) -> /Fixture Dev Kit - PMosfets/Gate1
- R13 pad 1: Net-(J20-Pad1) -> /Fixture Dev Kits - NMosfets/Gate_0
- R13 pad 2: Net-(R13-Pad2) -> /Fixture Dev Kits - NMosfets/Source_0
- R14 pad 1: Net-(J21-Pad1) -> /Fixture Dev Kits - NMosfets/Drain_0
- R14 pad 2: Net-(R14-Pad2) -> /Fixture Dev Kits - NMosfets/Gate_0
- R15 pad 1: GND -> /Fixture Dev Kits - NMosfets/Gate_1
- R15 pad 2: Net-(J20-Pad1) -> /Fixture Dev Kits - NMosfets/Source_1
- R16 pad 1: GND -> /Fixture Dev Kits - NMosfets/Drain_1
- R16 pad 2: Net-(J21-Pad1) -> /Fixture Dev Kits - NMosfets/Gate_1
- R17 pad 1: Net-(J20-Pad2) -> /Fixture Dev Kit - Functional Computer/LORP
- R17 pad 2: Net-(R17-Pad2) -> Net-(C1-Pad1)
- R18 pad 1: Net-(J21-Pad2) -> /Fixture Dev Kit - Functional Computer/LOLP
- R18 pad 2: Net-(R18-Pad2) -> Net-(C2-Pad1)
- R19 pad 1: GND -> /Fixture Dev Kit - Functional Computer/TS
- R19 pad 2: Net-(J20-Pad2) -> GND
- R2 pad 1: GND -> Net-(D2-Pad2)
- R2 pad 2: Net-(D2-Pad1) -> Net-(J4-Pad1)
- R20 pad 1: GND -> Net-(D10-Pad2)
- R20 pad 2: Net-(J21-Pad2) -> /C4-VCC-3V3
- R21 pad 1: Net-(J20-Pad3) -> Net-(D11-Pad2)
- R21 pad 2: Net-(R21-Pad2) -> /C4-VCC-3V3
- R22 pad 1: Net-(J21-Pad3) -> Net-(Q5-Pad2)
- R22 pad 2: Net-(R22-Pad2) -> Net-(Q7-Pad2)
- R23 pad 1: GND -> Net-(Q6-Pad2)
- R23 pad 2: Net-(J20-Pad3) -> Net-(Q8-Pad2)
- R24 pad 1: GND -> Net-(Q7-Pad2)
- R24 pad 2: Net-(J21-Pad3) -> /INA40_V-
- R25 pad 1: Net-(J20-Pad4) -> Net-(Q8-Pad2)
- R25 pad 2: Net-(R25-Pad2) -> /INA41_V-
- R26 pad 1: Net-(J21-Pad4) -> Net-(R26-Pad1)
- R26 pad 2: Net-(R26-Pad2) -> GND
- R27 pad 1: GND -> Net-(R27-Pad1)
- R27 pad 2: Net-(J20-Pad4) -> /C4-VCC-3V3
- R28 pad 1: GND -> Net-(R28-Pad1)
- R28 pad 2: Net-(J21-Pad4) -> GND
- R29 pad 1: Net-(J26-Pad1) -> Net-(R29-Pad1)
- R29 pad 2: Net-(R29-Pad2) -> (no net)
- R30 pad 1: GND -> Net-(D12-Pad2)
- R30 pad 2: Net-(J26-Pad1) -> /C4-VCC-3V3
- R31 pad 1: Net-(J26-Pad2) -> Net-(D13-Pad2)
- R31 pad 2: Net-(R31-Pad2) -> /C4-VCC-3V3
- R32 pad 1: GND -> Net-(Q9-Pad2)
- R32 pad 2: Net-(J26-Pad2) -> Net-(Q11-Pad2)
- R33 pad 1: Net-(J26-Pad3) -> Net-(Q10-Pad2)
- R33 pad 2: Net-(R33-Pad2) -> Net-(Q12-Pad2)
- R34 pad 1: GND -> Net-(Q11-Pad2)
- R34 pad 2: Net-(J26-Pad3) -> /INA42_V-
- R35 pad 1: Net-(J26-Pad4) -> Net-(Q12-Pad2)
- R35 pad 2: Net-(R35-Pad2) -> /INA43_V-
- R36 pad 1: GND -> Net-(R36-Pad1)
- R36 pad 2: Net-(J26-Pad4) -> /I2C-SDA
- R37 pad 1: Net-(J29-Pad1) -> Net-(R37-Pad1)
- R37 pad 2: Net-(R37-Pad2) -> /I2C-SCK
- R38 pad 1: GND -> Net-(R38-Pad1)
- R38 pad 2: Net-(J29-Pad1) -> (no net)
- R39 pad 1: Net-(J29-Pad2) -> Net-(R39-Pad1)
- R39 pad 2: Net-(R39-Pad2) -> GND
- R4 pad 1: GND -> Net-(D4-Pad2)
- R4 pad 2: Net-(D4-Pad1) -> Net-(J6-Pad1)
- R40 pad 1: GND -> Net-(D14-Pad2)
- R40 pad 2: Net-(J29-Pad2) -> /C4-VCC-3V3
- R41 pad 1: Net-(J29-Pad3) -> Net-(D15-Pad2)
- R41 pad 2: Net-(R41-Pad2) -> /C4-VCC-3V3
- R42 pad 1: GND -> Net-(D16-Pad2)
- R42 pad 2: Net-(J29-Pad3) -> /C4-VCC-3V3
- R43 pad 1: Net-(J29-Pad4) -> Net-(D17-Pad2)
- R43 pad 2: Net-(R43-Pad2) -> /C4-VCC-3V3
- R44 pad 1: GND -> Net-(Q13-Pad2)
- R44 pad 2: Net-(J29-Pad4) -> /AIN0
- R45 pad 1: Net-(Q1-Pad2) -> Net-(Q14-Pad2)
- R45 pad 2: Net-(J30-Pad1) -> /AIN1
- R46 pad 1: Net-(Q2-Pad2) -> Net-(Q15-Pad2)
- R46 pad 2: Net-(J31-Pad1) -> /AIN2
- R47 pad 1: Net-(Q3-Pad2) -> Net-(Q16-Pad2)
- R47 pad 2: Net-(J32-Pad1) -> /AIN3
- R48 pad 1: Net-(Q4-Pad2) -> GND
- R48 pad 2: Net-(J33-Pad1) -> /AIN0
- R49 pad 1: /Fixture Dev Kit - DUT/D-TS -> GND
- R49 pad 2: GND -> /AIN1
- R5 pad 1: Net-(D5-Pad2) -> GND
- R5 pad 2: Net-(J7-Pad1) -> Net-(D5-Pad1)
- R50 pad 1: Net-(R50-Pad1) -> GND
- R50 pad 2: /Fixture Dev Kit - ADS/C4-VCC-3V3 -> /AIN2
- R51 pad 1: Net-(R51-Pad1) -> GND
- R51 pad 2: /Fixture Dev Kit - ADS/C4-VCC-3V3 -> /AIN3
- R52 pad 1: /Fixture Dev Kit - PMosfets/Gate0 -> /AIN0
- R52 pad 2: /Fixture Dev Kit - PMosfets/Drain0 -> Net-(R52-Pad2)
- R53 pad 1: /Fixture Dev Kit - PMosfets/Gate4 -> /AIN1
- R53 pad 2: /Fixture Dev Kit - PMosfets/Drain4 -> Net-(R53-Pad2)
- R54 pad 1: /Fixture Dev Kit - PMosfets/Source0 -> /AIN2
- R54 pad 2: /Fixture Dev Kit - PMosfets/Gate0 -> Net-(R54-Pad2)
- R55 pad 1: /Fixture Dev Kit - PMosfets/Source4 -> /AIN3
- R55 pad 2: /Fixture Dev Kit - PMosfets/Gate4 -> Net-(R55-Pad2)
- R7 pad 1: Net-(D7-Pad2) -> GND
- R7 pad 2: Net-(J10-Pad1) -> Net-(D7-Pad1)
- R9 pad 1: Net-(D9-Pad2) -> /Fixture Dev Kit - PMosfets/Gate0
- R9 pad 2: Net-(J12-Pad1) -> /Fixture Dev Kit - PMosfets/Drain0
- TP10 pad 1: Net-(D10-Pad2) -> /Fixture Dev Kit - PMosfets/Source1
- TP2 pad 1: Net-(D3-Pad1) -> Net-(D2-Pad1)
- TP3 pad 1: Net-(D5-Pad1) -> Net-(D3-Pad1)
- TP4 pad 1: Net-(D7-Pad1) -> Net-(D4-Pad1)
- TP5 pad 1: Net-(D10-Pad2) -> /Fixture Dev Kit - PMosfets/Gate0
- TP6 pad 1: Net-(D11-Pad1) -> /Fixture Dev Kit - PMosfets/Gate1
- TP7 pad 1: Net-(D15-Pad1) -> /Fixture Dev Kit - PMosfets/Drain0
- TP8 pad 1: Net-(D17-Pad1) -> /Fixture Dev Kit - PMosfets/Source0
- TP9 pad 1: Net-(D10-Pad1) -> /Fixture Dev Kit - PMosfets/Drain1
- U1 pad 1: GND -> Net-(Q7-Pad2)
- U1 pad 2: Net-(U1-Pad2) -> /INA40_V-
- U1 pad 4: Net-(R13-Pad2) -> Net-(C5-Pad2)
- U1 pad 5: Net-(R17-Pad2) -> /I2C-SCK
- U1 pad 6: Net-(R21-Pad2) -> /I2C-SDA
- U1 pad 7: Net-(R25-Pad2) -> Net-(R26-Pad1)
- U1 pad 8: /Fixture Dev Kit - ADS/C4-VCC-3V3 -> Net-(R28-Pad1)
- U2 pad 1: /Fixture Dev Kit - ADS/I2C-SDA -> Net-(Q8-Pad2)
- U2 pad 2: Net-(U2-Pad2) -> /INA41_V-
- U2 pad 4: Net-(R14-Pad2) -> Net-(C6-Pad2)
- U2 pad 5: Net-(R18-Pad2) -> /I2C-SCK
- U2 pad 6: Net-(R22-Pad2) -> /I2C-SDA
- U2 pad 7: Net-(R26-Pad2) -> Net-(R27-Pad1)
- U2 pad 8: /Fixture Dev Kit - ADS/C4-VCC-3V3 -> Net-(R29-Pad1)
- U3 pad 1: /Fixture Dev Kit - ADS/C4-VCC-3V3 -> Net-(Q11-Pad2)
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Other:
- board outline removed
- net class Default: clearance 0.25 -> 0.2
- rule pad_to_mask_clearance: 0.2 -> 0
- rule trace_clearance: 0.25 -> 0.2
- rule trace_min: 0.25 -> 0.2
- board text removed: "1"
- board text removed: "2"
- board text removed: "3"
- board text removed: "3V3"
- board text removed: "4"
- board text removed: "Audio Jack"
- board text removed: "BUTTONS"
- board text removed: "D"
- board text removed: "D14"
- board text removed: "DUT"
- board text removed: "Functional Computer"
- board text removed: "G"
- board text removed: "GND"
- board text removed: "LED's"
- board text removed: "N-Channel MOSFETS"
- board text removed: "P-Channel MOSFETS"
- board text removed: "PWRON"
- board text removed: "PWRSW"
- board text removed: "S"
- board text removed: "SCK"
- board text removed: "SDA"
- board text removed: "USB-A"

Commit message: updating layout
Parts:
- removed C1, C2, C3, C4: 1uf, Capacitors_SMD:C_0805_HandSoldering
- removed J18, J19: Conn_01x35, Pin_Headers:Pin_Header_Straight_1x35_Pitch2.54mm
- removed J24: VBUS, Pin_Headers:Pin_Header_Straight_1x02_Pitch2.54mm
- removed JP1: Jumper_NC, Pin_Headers:Pin_Header_Straight_1x02_Pitch2.54mm
- removed P1: USB-A1HSW6, USB-A1HSW6:OST_USB-A1HSW6
- removed R17, R18: 0R, Resistors_SMD:R_0805_HandSoldering
- moved J25 145.3 mm to (86.4, 58.3), turned to 180 degrees
- moved R20 20.6 mm to (93.0, 91.4), turned to 0 degrees
- moved F2 17.6 mm to (96.4, 99.6), turned to 90 degrees
- moved D10 14.1 mm to (96.4, 94.0), turned to 90 degrees
- moved J27 13.1 mm to (87.9, 92.2), turned to 0 degrees
- moved R22 12.0 mm to (110.7, 94.9)
- moved R24 10.2 mm to (93.0, 93.5)
- moved JP2 8.52 mm to (87.9, 98.3)
- moved R28 7.31 mm to (93.0, 95.5), turned to 180 degrees
- moved C5 7.30 mm to (93.1, 89.4)
- moved Q5 6.24 mm to (101.7, 98.8)
- moved Q7 6.24 mm to (101.7, 91.4)
- moved R26 4.85 mm to (93.0, 97.5), turned to 180 degrees
- moved U1 1.52 mm to (93.0, 100.6)
Connections:
- J16 pad 17: Net-(J16-Pad17) -> (no net)
- J16 pad 18: (no net) -> Net-(J16-Pad18)
- J17 pad 34: Net-(J16-Pad17) -> Net-(J16-Pad18)

Commit message: updating rough layout
Parts:
- added D18: LNJP12X8ARA, 1206:1206, F.Cu at (92.5, 90.9)
- added D19: LNJP12X8ARA, 1206:1206, F.Cu at (92.5, 75.2)
- added D20: LNJP12X8ARA, 1206:1206, F.Cu at (93.5, 59.9)
- added D21: LNJP12X8ARA, 1206:1206, F.Cu at (93.7, 45.7)
- added R17: 160R, Resistors_SMD:R_0805_HandSoldering, F.Cu at (97.5, 90.9)
- added R18: 160R, Resistors_SMD:R_0805_HandSoldering, F.Cu at (97.5, 75.2)
- added R56: 160R, Resistors_SMD:R_0805_HandSoldering, F.Cu at (98.8, 59.9)
- added R57: 160R, Resistors_SMD:R_0805_HandSoldering, F.Cu at (98.8, 45.7)
- moved R10 272.0 mm to (140.1, 49.6), turned to 270 degrees
- moved R9 264.4 mm to (142.6, 49.5), turned to 270 degrees
- moved Q1 261.5 mm to (133.9, 50.1), turned to 180 degrees
- moved TP6 260.5 mm to (145.0, 65.4)
- moved R12 260.3 mm to (140.2, 61.9), turned to 90 degrees
- moved J12 258.9 mm to (124.6, 60.1)
- moved Q2 258.6 mm to (134.2, 62.8), turned to 180 degrees
- moved TP7 258.3 mm to (142.6, 53.4)
- moved TP5 257.1 mm to (145.0, 53.4)
- moved J11 253.7 mm to (124.3, 47.9)
- moved R11 242.1 mm to (142.7, 61.7), turned to 90 degrees
- moved TP9 241.9 mm to (142.7, 65.3)
- moved TP8 240.4 mm to (139.9, 53.2)
- moved J7 239.7 mm to (89.1, 132.0), turned to 90 degrees
- moved TP10 238.6 mm to (140.0, 65.5)
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Connections:
- R29 pad 2: (no net) -> GND
- R38 pad 2: (no net) -> GND
Other:
- board outline added: 145.7 x 113.8 mm
- board text added: "ADS"
- board text added: "BUTTONS"
- board text added: "INA"
- board text added: "LED"
- board text added: "N-CHANNEL"
- board text added: "P-CHANNEL"
- board text added: "POWER"
- board text added: "PROTO Area"

Commit message: updating rough layout
Parts:
- moved C6 14.9 mm to (96.0, 52.1)
- moved D11 14.9 mm to (89.9, 63.0)
- moved Q9 14.9 mm to (103.1, 46.0)
- moved R21 14.9 mm to (95.0, 63.0)
- moved D13 14.9 mm to (91.2, 33.8)
- moved D4 14.9 mm to (159.8, 77.2)
- moved D6 14.9 mm to (159.9, 50.9)
- moved Q2 14.9 mm to (131.7, 48.1)
- moved R10 14.9 mm to (137.5, 34.8)
- moved R3 14.9 mm to (154.8, 62.0)
- moved R31 14.9 mm to (96.3, 33.8)
- moved R34 14.9 mm to (150.9, 55.6)
- moved R36 14.9 mm to (90.9, 49.8)
- moved R37 14.9 mm to (90.9, 37.8)
- moved R6 14.9 mm to (154.9, 50.9)
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
Commit message: updading laytout
Parts:
- moved J1 30.5 mm to (75.4, 130.0), turned to 180 degrees
- moved U4 0.25 mm to (90.9, 40.4)
Changed lines of the file:
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@@
     (links 359)
     (no_connects 359)
-    (area 25.959599 35.408399 171.754001 149.300401)
+    (area 23.419599 22.454399 169.214001 136.346401)
     (thickness 1.6)
-    (drawings 56)
+    (drawings 63)
     (tracks 0)
     (zones 0)
@@
   )
   (module Pin_Headers:Pin_Header_Straight_2x10_Pitch2.54mm (layer F.Cu)
-    (at 53.34 108.966 90)
+    (at 75.438 130.048 180)
     (descr "Through hole straight pin header, 2x10, 2.54mm pitch, double rows")
     (tags "Through hole pin header THT 2x10 2.54mm double row")
-    (fp_text reference J1 (at 1.27 -2.33 90) (layer F.SilkS)
+    (fp_text reference J1 (at 1.27 -2.33 180) (layer F.SilkS)
       (effects (font (size 1 1) (thickness 0.15)))
     )
-    (fp_text value DUT (at 1.27 25.19 90) (layer F.Fab)
+    (fp_text value DUT (at 1.27 25.19 180) (layer F.Fab)
       (effects (font (size 1 1) (thickness 0.15)))
     )
@@
     (fp_line (start 4.35 24.65) (end 4.35 -1.8) (layer F.CrtYd) (width 0.05))
     (fp_line (start 4.35 -1.8) (end -1.8 -1.8) (layer F.CrtYd) (width 0.05))
-    (fp_text user %R (at 1.27 11.43 180) (layer F.Fab)
+    (fp_text user %R (at 1.27 11.43 270) (layer F.Fab)
       (effects (font (size 1 1) (thickness 0.15)))
     )
-    (pad 1 thru_hole rect (at 0 0 90) (size 1.7 1.7) (drill 1) (layers *.Cu *.Mask)
+    (pad 1 thru_hole rect (at 0 0 180) (size 1.7 1.7) (drill 1) (layers *.Cu *.Mask)
       (net 43 /AIN0))
-    (pad 2 thru_hole oval (at 2.54 0 90) (size 1.7 1.7) (drill 1) (layers *.Cu *.Mask)
+    (pad 2 thru_hole oval (at 2.54 0 180) (size 1.7 1.7) (drill 1) (layers *.Cu *.Mask)
       (net 44 /AIN1))
-    (pad 3 thru_hole oval (at 0 2.54 90) (size 1.7 1.7) (drill 1) (layers *.Cu *.Mask)
+    (pad 3 thru_hole oval (at 0 2.54 180) (size 1.7 1.7) (drill 1) (layers *.Cu *.Mask)
       (net 45 /AIN2))
-    (pad 4 thru_hole oval (at 2.54 2.54 90) (size 1.7 1.7) (drill 1) (layers *.Cu *.Mask)
+    (pad 4 thru_hole oval (at 2.54 2.54 180) (size 1.7 1.7) (drill 1) (layers *.Cu *.Mask)
       (net 46 /AIN3))
-    (pad 5 thru_hole oval (at 0 5.08 90) (size 1.7 1.7) (drill 1) (layers *.Cu *.Mask)
+    (pad 5 thru_hole oval (at 0 5.08 180) (size 1.7 1.7) (drill 1) (layers *.Cu *.Mask)
       (net 47 /INA40_V-))
-    (pad 6 thru_hole oval (at 2.54 5.08 90) (size 1.7 1.7) (drill 1) (layers *.Cu *.Mask)
+    (pad 6 thru_hole oval (at 2.54 5.08 180) (size 1.7 1.7) (drill 1) (layers *.Cu *.Mask)
       (net 48 /INA41_V-))
-    (pad 7 thru_hole oval (at 0 7.62 90) (size 1.7 1.7) (drill 1) (layers *.Cu *.Mask)
+    (pad 7 thru_hole oval (at 0 7.62 180) (size 1.7 1.7) (drill 1) (layers *.Cu *.Mask)
       (net 49 /INA42_V-))
-    (pad 8 thru_hole oval (at 2.54 7.62 90) (size 1.7 1.7) (drill 1) (layers *.Cu *.Mask)
+    (pad 8 thru_hole oval (at 2.54 7.62 180) (size 1.7 1.7) (drill 1) (layers *.Cu *.Mask)
       (net 50 /INA43_V-))
-    (pad 9 thru_hole oval (at 0 10.16 90) (size 1.7 1.7) (drill 1) (layers *.Cu *.Mask)
+    (pad 9 thru_hole oval (at 0 10.16 180) (size 1.7 1.7) (drill 1) (layers *.Cu *.Mask)
       (net 51 /I2C-SDA))
-    (pad 10 thru_hole oval (at 2.54 10.16 90) (size 1.7 1.7) (drill 1) (layers *.Cu *.Mask)
+    (pad 10 thru_hole oval (at 2.54 10.16 180) (size 1.7 1.7) (drill 1) (layers *.Cu *.Mask)
       (net 52 /I2C-SCK))
-    (pad 11 thru_hole oval (at 0 12.7 90) (size 1.7 1.7) (drill 1) (layers *.Cu *.Mask)
+    (pad 11 thru_hole oval (at 0 12.7 180) (size 1.7 1.7) (drill 1) (layers *.Cu *.Mask)
       (net 2 GND))
-    (pad 12 thru_hole oval (at 2.54 12.7 90) (size 1.7 1.7) (drill 1) (layers *.Cu *.Mask)
+    (pad 12 thru_hole oval (at 2.54 12.7 180) (size 1.7 1.7) (drill 1) (layers *.Cu *.Mask)
       (net 2 GND))
-    (pad 13 thru_hole oval (at 0 15.24 90) (size 1.7 1.7) (drill 1) (layers *.Cu *.Mask)
+    (pad 13 thru_hole oval (at 0 15.24 180) (size 1.7 1.7) (drill 1) (layers *.Cu *.Mask)
       (net 2 GND))
-    (pad 14 thru_hole oval (at 2.54 15.24 90) (size 1.7 1.7) (drill 1) (layers *.Cu *.Mask)
+    (pad 14 thru_hole oval (at 2.54 15.24 180) (size 1.7 1.7) (drill 1) (layers *.Cu *.Mask)
       (net 2 GND))
-    (pad 15 thru_hole oval (at 0 17.78 90) (size 1.7 1.7) (drill 1) (layers *.Cu *.Mask)
+    (pad 15 thru_hole oval (at 0 17.78 180) (size 1.7 1.7) (drill 1) (layers *.Cu *.Mask)
       (net 2 GND))
-    (pad 16 thru_hole oval (at 2.54 17.78 90) (size 1.7 1.7) (drill 1) (layers *.Cu *.Mask)
+    (pad 16 thru_hole oval (at 2.54 17.78 180) (size 1.7 1.7) (drill 1) (layers *.Cu *.Mask)
       (net 2 GND))
-    (pad 17 thru_hole oval (at 0 20.32 90) (size 1.7 1.7) (drill 1) (layers *.Cu *.Mask)
+    (pad 17 thru_hole oval (at 0 20.32 180) (size 1.7 1.7) (drill 1) (layers *.Cu *.Mask)
       (net 2 GND))
-    (pad 18 thru_hole oval (at 2.54 20.32 90) (size 1.7 1.7) (drill 1) (layers *.Cu *.Mask)
+    (pad 18 thru_hole oval (at 2.54 20.32 180) (size 1.7 1.7) (drill 1) (layers *.Cu *.Mask)
       (net 53 /UART-RX))
-    (pad 19 thru_hole oval (at 0 22.86 90) (size 1.7 1.7) (drill 1) (layers *.Cu *.Mask)
+    (pad 19 thru_hole oval (at 0 22.86 180) (size 1.7 1.7) (drill 1) (layers *.Cu *.Mask)
       (net 54 /UART-TX))
-    (pad 20 thru_hole oval (at 2.54 22.86 90) (size 1.7 1.7) (drill 1) (layers *.Cu *.Mask)
+    (pad 20 thru_hole oval (at 2.54 22.86 180) (size 1.7 1.7) (drill 1) (layers *.Cu *.Mask)
       (net 55 /ADAPTER_ID))
     (model ${KISYS3DMOD}/Pin_Headers.3dshapes/Pin_Header_Straight_2x10_Pitch2.54mm.wrl
@@
   )
   (module INA219BIDCNR:SOT65P280X145-8N (layer F.Cu)
-    (at 90.678 40.386)
+    (at 90.932 40.386)
     (attr smd)
     (fp_text reference U4 (at 0.712769 -4.22571) (layer F.SilkS)
@@
     )
   )
+  (gr_line (start 26.416 134.366) (end 26.416 134.62) (angle 90) (layer F.SilkS) (width 0.2))
+  (gr_line (start 66.548 134.366) (end 26.416 134.366) (angle 90) (layer F.SilkS) (width 0.2))
+  (gr_line (start 66.548 103.378) (end 66.548 134.366) (angle 90) (layer F.SilkS) (width 0.2))
+  (gr_line (start 26.416 103.378) (end 66.548 103.378) (angle 90) (layer F.SilkS) (width 0.2))
+  (gr_line (start 67.818 134.62) (end 72.644 134.62) (angle 90) (layer F.SilkS) (width 0.2))
+  (gr_line (start 67.818 134.112) (end 67.818 134.62) (angle 90) (layer F.SilkS) (width 0.2))
+  (gr_line (start 67.818 103.378) (end 67.818 134.112) (angle 90) (layer F.SilkS) (width 0.2))
+  (gr_line (start 71.882 103.378) (end 67.818 103.378) (angle 90) (layer F.SilkS) (width 0.2))
+  (gr_line (start 80.01 134.62) (end 71.882 134.62) (angle 90) (layer F.SilkS) (width 0.2))
+  (gr_line (start 80.01 103.378) (end 80.01 134.62) (angle 90) (layer F.SilkS) (width 0.2))
+  (gr_line (start 71.628 103.378) (end 80.01 103.378) (angle 90) (layer F.SilkS) (width 0.2))
+  (gr_line (start 26.416 134.366) (end 26.416 103.378) (angle 90) (layer F.SilkS) (width 0.2))
   (gr_line (start 23.4696 22.5044) (end 24.2824 22.5044) (angle 90) (layer Edge.Cuts) (width 0.1))
   (gr_line (start 23.4696 136.2964) (end 23.4696 22.5044) (angle 90) (layer Edge.Cuts) (width 0.1))
@@
     (effects (font (size 1.5 1.5) (thickness 0.3)))
   )
-  (gr_text "PROTO Area" (at 35.0012 115.5192) (layer F.SilkS)
+  (gr_text "PROTO Area" (at 33.528 105.41) (layer F.SilkS)
     (effects (font (size 1.5 1.5) (thickness 0.3)))
   )
   (gr_line (start 28.1432 113.284) (end 28.1432 113.4872) (angle 90) (layer F.SilkS) (width 0.2))
-  (gr_line (start 26.7208 113.284) (end 28.1432 113.284) (angle 90) (layer F.SilkS) (width 0.2))
-  (gr_line (start 26.7208 134.1628) (end 26.7208 113.284) (angle 90) (layer F.SilkS) (width 0.2))
-  (gr_line (start 76.7588 134.1628) (end 26.7208 134.1628) (angle 90) (layer F.SilkS) (width 0.2))
-  (gr_line (start 76.7588 113.1824) (end 76.7588 134.1628) (angle 90) (layer F.SilkS) (width 0.2))
-  (gr_line (start 27.2288 113.1824) (end 76.7588 113.1824) (angle 90) (layer F.SilkS) (width 0.2))
   (gr_line (start 145.7452 113.6396) (end 82.6516 113.6396) (angle 90) (layer F.SilkS) (width 0.2))
   (gr_line (start 145.7452 134.62) (end 145.7452 113.6396) (angle 90) (layer F.SilkS) (width 0.2))
