File: HARDWARE/v0.01/KiCad/FixtureDevKit-ADS.sch (KiCad schematic (older format))
At the start: 54 parts, among them J16 ADS_48, J17 ADS_48, J18 ADS_4A, J19 ADS_4A, J20 ADS_48, J21 ADS_4A, J22 ADS, J23 ADS, J24 ADS_49, J25 ADS_49, J26 ADS_49, J27 ADS_4B, J28 ADS_4B, J29 ADS_4B, U1 ADS1015IDGST, U2 ADS1015IDGST, U3 ADS1015IDGST, U4 ADS1015IDGST

Commit message: beginning pcb layout
Connections:
- net C4-VCC-3V3: now also J18.1 (Pin_1), J19.1 (Pin_1), J24.1 (Pin_1), J25.1 (Pin_1), J27.1 (Pin_1), J28.1 (Pin_1); no longer J18.4 (Pin_4), J19.4 (Pin_4), J24.4 (Pin_4), J25.4 (Pin_4), J27.4 (Pin_4), J28.4 (Pin_4)
- net GND: now also J18.2 (Pin_2), J19.2 (Pin_2), J24.2 (Pin_2), J25.2 (Pin_2), J27.2 (Pin_2), J28.2 (Pin_2); no longer J18.3 (Pin_3), J19.3 (Pin_3), J24.3 (Pin_3), J25.3 (Pin_3), J27.3 (Pin_3), J28.3 (Pin_3)
- net I2C-SCK: now also J18.4 (Pin_4), J19.4 (Pin_4), J24.4 (Pin_4), J25.4 (Pin_4), J27.4 (Pin_4), J28.4 (Pin_4); no longer J18.1 (Pin_1), J19.1 (Pin_1), J24.1 (Pin_1), J25.1 (Pin_1), J27.1 (Pin_1), J28.1 (Pin_1)
- net I2C-SDA: now also J18.3 (Pin_3), J19.3 (Pin_3), J24.3 (Pin_3), J25.3 (Pin_3), J27.3 (Pin_3), J28.3 (Pin_3); no longer J18.2 (Pin_2), J19.2 (Pin_2), J24.2 (Pin_2), J25.2 (Pin_2), J27.2 (Pin_2), J28.2 (Pin_2)
Changed lines of the file:
@@
 $EndComp
 $Comp
-L GND #PWR020
+L GND #PWR024
 U 1 1 59F13B4C
 P 3100 3200
-F 0 "#PWR020" H 3100 2950 50  0001 C CNN
+F 0 "#PWR024" H 3100 2950 50  0001 C CNN
 F 1 "GND" H 3100 3050 50  0000 C CNN
 F 2 "" H 3100 3200 50  0001 C CNN
@@
 $EndComp
 $Comp
-L GND #PWR021
+L GND #PWR025
 U 1 1 59F13B6F
 P 1900 4000
-F 0 "#PWR021" H 1900 3750 50  0001 C CNN
+F 0 "#PWR025" H 1900 3750 50  0001 C CNN
 F 1 "GND" H 1900 3850 50  0000 C CNN
 F 2 "" H 1900 4000 50  0001 C CNN
@@
 	1900 3950 1900 4000
 $Comp
-L GND #PWR022
+L GND #PWR026
 U 1 1 59F13B77
 P 700 3750
-F 0 "#PWR022" H 700 3500 50  0001 C CNN
+F 0 "#PWR026" H 700 3500 50  0001 C CNN
 F 1 "GND" H 700 3600 50  0000 C CNN
 F 2 "" H 700 3750 50  0001 C CNN
@@
 SCL
 $Comp
-L GND #PWR023
+L GND #PWR027
 U 1 1 59F17684
 P 1250 3200
-F 0 "#PWR023" H 1250 2950 50  0001 C CNN
+F 0 "#PWR027" H 1250 2950 50  0001 C CNN
 F 1 "GND" H 1250 3050 50  0000 C CNN
 F 2 "" H 1250 3200 50  0001 C CNN
@@
 SCL
 $Comp
-L GND #PWR024
+L GND #PWR028
 U 1 1 59F183D4
 P 1250 4450
-F 0 "#PWR024" H 1250 4200 50  0001 C CNN
+F 0 "#PWR028" H 1250 4200 50  0001 C CNN
 F 1 "GND" H 1250 4300 50  0000 C CNN
 F 2 "" H 1250 4450 50  0001 C CNN
@@
 $EndComp
 $Comp
-L GND #PWR025
+L GND #PWR029
 U 1 1 59F1A7E1
 P 6350 3200
-F 0 "#PWR025" H 6350 2950 50  0001 C CNN
+F 0 "#PWR029" H 6350 2950 50  0001 C CNN
 F 1 "GND" H 6350 3050 50  0000 C CNN
 F 2 "" H 6350 3200 50  0001 C CNN
@@
 $EndComp
 $Comp
-L GND #PWR026
+L GND #PWR030
 U 1 1 59F1A7ED
 P 5150 4000
-F 0 "#PWR026" H 5150 3750 50  0001 C CNN
+F 0 "#PWR030" H 5150 3750 50  0001 C CNN
 F 1 "GND" H 5150 3850 50  0000 C CNN
 F 2 "" H 5150 4000 50  0001 C CNN
@@
 L Conn_01x04 J24
 U 1 1 59F1A814
-P 4600 2800
-F 0 "J24" H 4600 3000 50  0000 C CNN
-F 1 "ADS_49" H 4600 2500 50  0000 C CNN
-F 2 "Pin_Headers:Pin_Header_Straight_1x04_Pitch2.54mm" H 4600 2800 50  0001 C CNN
-F 3 "" H 4600 2800 50  0001 C CNN
-	1    4600 2800
-	0    1    -1   0
+P 4500 2800
+F 0 "J24" H 4500 3000 50  0000 C CNN
+F 1 "ADS_49" H 4500 2500 50  0000 C CNN
+F 2 "Pin_Headers:Pin_Header_Straight_1x04_Pitch2.54mm" H 4500 2800 50  0001 C CNN
+F 3 "" H 4500 2800 50  0001 C CNN
+	1    4500 2800
+	0    -1   -1   0
 $EndComp
 Text Label 4400 3050 3    60   ~ 0
@@
 SCL
 $Comp
-L GND #PWR027
+L GND #PWR031
 U 1 1 59F1A81D
 P 4500 3200
-F 0 "#PWR027" H 4500 2950 50  0001 C CNN
+F 0 "#PWR031" H 4500 2950 50  0001 C CNN
 F 1 "GND" H 4500 3050 50  0000 C CNN
 F 2 "" H 4500 3200 50  0001 C CNN
@@
 L Conn_01x04 J25
 U 1 1 59F1A827
-P 4600 4850
-F 0 "J25" H 4600 5050 50  0000 C CNN
-F 1 "ADS_49" H 4600 4550 50  0000 C CNN
-F 2 "Pin_Headers:Pin_Header_Straight_1x04_Pitch2.54mm" H 4600 4850 50  0001 C CNN
-F 3 "" H 4600 4850 50  0001 C CNN
-	1    4600 4850
-	0    1    1    0
+P 4500 4850
+F 0 "J25" H 4500 5050 50  0000 C CNN
+F 1 "ADS_49" H 4500 4550 50  0000 C CNN
+F 2 "Pin_Headers:Pin_Header_Straight_1x04_Pitch2.54mm" H 4500 4850 50  0001 C CNN
+F 3 "" H 4500 4850 50  0001 C CNN
+	1    4500 4850
+	0    -1   1    0
 $EndComp
 Text Label 4400 4600 1    60   ~ 0
@@
 SCL
 $Comp
-L GND #PWR028
+L GND #PWR032
 U 1 1 59F1A830
 P 4500 4450
-F 0 "#PWR028" H 4500 4200 50  0001 C CNN
+F 0 "#PWR032" H 4500 4200 50  0001 C CNN
 F 1 "GND" H 4500 4300 50  0000 C CNN
 F 2 "" H 4500 4450 50  0001 C CNN
@@
 $EndComp
 $Comp
-L GND #PWR029
+L GND #PWR033
 U 1 1 59F1B4EE
 P 3100 5900
-F 0 "#PWR029" H 3100 5650 50  0001 C CNN
+F 0 "#PWR033" H 3100 5650 50  0001 C CNN
 F 1 "GND" H 3100 5750 50  0000 C CNN
 F 2 "" H 3100 5900 50  0001 C CNN
@@
 $EndComp
 $Comp
-L GND #PWR030
+L GND #PWR034
 U 1 1 59F1B4FA
 P 1900 6700
-F 0 "#PWR030" H 1900 6450 50  0001 C CNN
+F 0 "#PWR034" H 1900 6450 50  0001 C CNN
 F 1 "GND" H 1900 6550 50  0000 C CNN
 F 2 "" H 1900 6700 50  0001 C CNN
@@
 L Conn_01x04 J18
 U 1 1 59F1B521
-P 1350 5500
-F 0 "J18" H 1350 5700 50  0000 C CNN
-F 1 "ADS_4A" H 1350 5200 50  0000 C CNN
-F 2 "Pin_Headers:Pin_Header_Straight_1x04_Pitch2.54mm" H 1350 5500 50  0001 C CNN
-F 3 "" H 1350 5500 50  0001 C CNN
-	1    1350 5500
-	0    1    -1   0
+P 1250 5500
+F 0 "J18" H 1250 5700 50  0000 C CNN
+F 1 "ADS_4A" H 1250 5200 50  0000 C CNN
+F 2 "Pin_Headers:Pin_Header_Straight_1x04_Pitch2.54mm" H 1250 5500 50  0001 C CNN
+F 3 "" H 1250 5500 50  0001 C CNN
+	1    1250 5500
+	0    -1   -1   0
 $EndComp
 Text Label 1150 5750 3    60   ~ 0
@@
 SCL
 $Comp
-L GND #PWR031
+L GND #PWR035
 U 1 1 59F1B52A
 P 1250 5900
-F 0 "#PWR031" H 1250 5650 50  0001 C CNN
+F 0 "#PWR035" H 1250 5650 50  0001 C CNN
 F 1 "GND" H 1250 5750 50  0000 C CNN
 F 2 "" H 1250 5900 50  0001 C CNN
@@
 L Conn_01x04 J19
 U 1 1 59F1B534
-P 1350 7550
-F 0 "J19" H 1350 7750 50  0000 C CNN
-F 1 "ADS_4A" H 1350 7250 50  0000 C CNN
-F 2 "Pin_Headers:Pin_Header_Straight_1x04_Pitch2.54mm" H 1350 7550 50  0001 C CNN
-F 3 "" H 1350 7550 50  0001 C CNN
-	1    1350 7550
-	0    1    1    0
+P 1250 7550
+F 0 "J19" H 1250 7750 50  0000 C CNN
+F 1 "ADS_4A" H 1250 7250 50  0000 C CNN
+F 2 "Pin_Headers:Pin_Header_Straight_1x04_Pitch2.54mm" H 1250 7550 50  0001 C CNN
+F 3 "" H 1250 7550 50  0001 C CNN
+	1    1250 7550
+	0    -1   1    0
 $EndComp
 Text Label 1150 7300 1    60   ~ 0
@@
 SCL
 $Comp
-L GND #PWR032
+L GND #PWR036
 U 1 1 59F1B53D
 P 1250 7150
-F 0 "#PWR032" H 1250 6900 50  0001 C CNN
+F 0 "#PWR036" H 1250 6900 50  0001 C CNN
 F 1 "GND" H 1250 7000 50  0000 C CNN
 F 2 "" H 1250 7150 50  0001 C CNN
@@
 $EndComp
 $Comp
-L GND #PWR033
+L GND #PWR037
 U 1 1 59F1B587
 P 9600 3200
-F 0 "#PWR033" H 9600 2950 50  0001 C CNN
+F 0 "#PWR037" H 9600 2950 50  0001 C CNN
 F 1 "GND" H 9600 3050 50  0000 C CNN
 F 2 "" H 9600 3200 50  0001 C CNN
@@
 $EndComp
 $Comp
-L GND #PWR034
+L GND #PWR038
 U 1 1 59F1B593
 P 8400 4000
-F 0 "#PWR034" H 8400 3750 50  0001 C CNN
+F 0 "#PWR038" H 8400 3750 50  0001 C CNN
 F 1 "GND" H 8400 3850 50  0000 C CNN
 F 2 "" H 8400 4000 50  0001 C CNN
@@
 L Conn_01x04 J27
 U 1 1 59F1B5BA
-P 7850 2800
-F 0 "J27" H 7850 3000 50  0000 C CNN
-F 1 "ADS_4B" H 7850 2500 50  0000 C CNN
-F 2 "Pin_Headers:Pin_Header_Straight_1x04_Pitch2.54mm" H 7850 2800 50  0001 C CNN
-F 3 "" H 7850 2800 50  0001 C CNN
-	1    7850 2800
-	0    1    -1   0
+P 7750 2800
+F 0 "J27" H 7750 3000 50  0000 C CNN
+F 1 "ADS_4B" H 7750 2500 50  0000 C CNN
+F 2 "Pin_Headers:Pin_Header_Straight_1x04_Pitch2.54mm" H 7750 2800 50  0001 C CNN
+F 3 "" H 7750 2800 50  0001 C CNN
+	1    7750 2800
+	0    -1   -1   0
 $EndComp
 Text Label 7650 3050 3    60   ~ 0
@@
 SCL
 $Comp
-L GND #PWR035
+L GND #PWR039
 U 1 1 59F1B5C3
 P 7750 3200
-F 0 "#PWR035" H 7750 2950 50  0001 C CNN
+F 0 "#PWR039" H 7750 2950 50  0001 C CNN
 F 1 "GND" H 7750 3050 50  0000 C CNN
 F 2 "" H 7750 3200 50  0001 C CNN
@@
 L Conn_01x04 J28
 U 1 1 59F1B5CD
-P 7850 4850
-F 0 "J28" H 7850 5050 50  0000 C CNN
-F 1 "ADS_4B" H 7850 4550 50  0000 C CNN
-F 2 "Pin_Headers:Pin_Header_Straight_1x04_Pitch2.54mm" H 7850 4850 50  0001 C CNN
-F 3 "" H 7850 4850 50  0001 C CNN
-	1    7850 4850
-	0    1    1    0
+P 7750 4850
+F 0 "J28" H 7750 5050 50  0000 C CNN
+F 1 "ADS_4B" H 7750 4550 50  0000 C CNN
+F 2 "Pin_Headers:Pin_Header_Straight_1x04_Pitch2.54mm" H 7750 4850 50  0001 C CNN
+F 3 "" H 7750 4850 50  0001 C CNN
+	1    7750 4850
+	0    -1   1    0
 $EndComp
 Text Label 7650 4600 1    60   ~ 0
@@
 SCL
 $Comp
-L GND #PWR036
+L GND #PWR040
 U 1 1 59F1B5D6
 P 7750 4450
-F 0 "#PWR036" H 7750 4200 50  0001 C CNN
+F 0 "#PWR040" H 7750 4200 50  0001 C CNN
 F 1 "GND" H 7750 4300 50  0000 C CNN
 F 2 "" H 7750 4450 50  0001 C CNN
@@
 SCL
 $Comp
-L GND #PWR037
+L GND #PWR041
 U 1 1 59F24258
 P 4250 6150
-F 0 "#PWR037" H 4250 5900 50  0001 C CNN
+F 0 "#PWR041" H 4250 5900 50  0001 C CNN
 F 1 "GND" H 4250 6000 50  0000 C CNN
 F 2 "" H 4250 6150 50  0001 C CNN
@@
 SCL
 $Comp
-L GND #PWR038
+L GND #PWR042
 U 1 1 59F2434D
 P 4250 6900
-F 0 "#PWR038" H 4250 6650 50  0001 C CNN
+F 0 "#PWR042" H 4250 6650 50  0001 C CNN
 F 1 "GND" H 4250 6750 50  0000 C CNN
 F 2 "" H 4250 6900 50  0001 C CNN
@@
 $EndComp
 $Comp
-L GND #PWR039
+L GND #PWR043
 U 1 1 59EFF3E5
 P 750 4350
-F 0 "#PWR039" H 750 4100 50  0001 C CNN
+F 0 "#PWR043" H 750 4100 50  0001 C CNN
 F 1 "GND" H 750 4200 50  0000 C CNN
 F 2 "" H 750 4350 50  0001 C CNN
@@
 $EndComp
 $Comp
-L GND #PWR040
+L GND #PWR044
 U 1 1 59F0004D
 P 4000 4350
-F 0 "#PWR040" H 4000 4100 50  0001 C CNN
+F 0 "#PWR044" H 4000 4100 50  0001 C CNN
 F 1 "GND" H 4000 4200 50  0000 C CNN
 F 2 "" H 4000 4350 50  0001 C CNN
@@
 $EndComp
 $Comp
-L GND #PWR041
+L GND #PWR045
 U 1 1 59F00AA9
 P 750 7050
-F 0 "#PWR041" H 750 6800 50  0001 C CNN
+F 0 "#PWR045" H 750 6800 50  0001 C CNN
 F 1 "GND" H 750 6900 50  0000 C CNN
 F 2 "" H 750 7050 50  0001 C CNN
@@
 $EndComp
 $Comp
-L GND #PWR042
+L GND #PWR046
 U 1 1 59F00E3C
 P 7250 4350
-F 0 "#PWR042" H 7250 4100 50  0001 C CNN
+F 0 "#PWR046" H 7250 4100 50  0001 C CNN
 F 1 "GND" H 7250 4200 50  0000 C CNN
 F 2 "" H 7250 4350 50  0001 C CNN
