File: HARDWARE/v0.01/KiCad/FixtureDevKit-INA.sch (KiCad schematic (older format))
At the start: 42 parts, among them J100 INA_43, J101 INA_43, J102 INA_41, J103 INA_43, J104 INA, J105 INA, J92 INA_40, J93 INA_40, J94 INA_42, J95 INA_42, J96 INA_40, J97 INA_42, J98 INA_41, J99 INA_41, U10 INA219BIDCNT, U7 INA219BIDCNT, U8 INA219BIDCNT, U9 INA219BIDCNT

Commit message: adding footprints
Parts:
- C10, C11, C12, C9: footprint (none) -> Capacitors_SMD:C_0805_HandSoldering
- J100, J101, J104, J105, J92, J93, J94, J95, J98, J99: footprint (none) -> Pin_Headers:Pin_Header_Straight_1x04_Pitch2.54mm
- J102, J103, J96, J97, JP2, JP3, JP4, JP5: footprint (none) -> Pin_Headers:Pin_Header_Straight_1x02_Pitch2.54mm
- R86, R87, R88, R89, R90, R91, R92, R93: footprint (none) -> Resistors_SMD:R_0805_HandSoldering
Changed lines of the file:
@@
 F 0 "C9" H 1325 2750 50  0000 L CNN
 F 1 "0.1uF" H 1325 2550 50  0000 L CNN
-F 2 "" H 1338 2500 50  0001 C CNN
+F 2 "Capacitors_SMD:C_0805_HandSoldering" H 1338 2500 50  0001 C CNN
 F 3 "" H 1300 2650 50  0001 C CNN
 	1    1300 2650
@@
 F 0 "R88" V 1380 3150 50  0000 C CNN
 F 1 "1K" V 1300 3150 50  0000 C CNN
-F 2 "" V 1230 3150 50  0001 C CNN
+F 2 "Resistors_SMD:R_0805_HandSoldering" V 1230 3150 50  0001 C CNN
 F 3 "" H 1300 3150 50  0001 C CNN
 	1    1300 3150
@@
 F 0 "R86" V 1130 3250 50  0000 C CNN
 F 1 "1K" V 1050 3250 50  0000 C CNN
-F 2 "" V 980 3250 50  0001 C CNN
+F 2 "Resistors_SMD:R_0805_HandSoldering" V 980 3250 50  0001 C CNN
 F 3 "" H 1050 3250 50  0001 C CNN
 	1    1050 3250
@@
 F 0 "J96" H 2900 3150 50  0000 C CNN
 F 1 "INA_40" H 2900 2850 50  0000 C CNN
-F 2 "" H 2900 3050 50  0001 C CNN
+F 2 "Pin_Headers:Pin_Header_Straight_1x02_Pitch2.54mm" H 2900 3050 50  0001 C CNN
 F 3 "" H 2900 3050 50  0001 C CNN
 	1    2900 3050
@@
 F 0 "JP2" H 1050 2930 50  0000 C CNN
 F 1 "Jumper_NO" H 1060 2790 50  0000 C CNN
-F 2 "" H 1050 2850 50  0001 C CNN
+F 2 "Pin_Headers:Pin_Header_Straight_1x02_Pitch2.54mm" H 1050 2850 50  0001 C CNN
 F 3 "" H 1050 2850 50  0001 C CNN
 	1    1050 2850
@@
 F 0 "J92" H 2000 2200 50  0000 C CNN
 F 1 "INA_40" H 2000 1700 50  0000 C CNN
-F 2 "" H 2000 2000 50  0001 C CNN
+F 2 "Pin_Headers:Pin_Header_Straight_1x04_Pitch2.54mm" H 2000 2000 50  0001 C CNN
 F 3 "" H 2000 2000 50  0001 C CNN
 	1    2000 2000
@@
 F 0 "J93" H 2000 4550 50  0000 C CNN
 F 1 "INA_40" H 2000 4050 50  0000 C CNN
-F 2 "" H 2000 4350 50  0001 C CNN
+F 2 "Pin_Headers:Pin_Header_Straight_1x04_Pitch2.54mm" H 2000 4350 50  0001 C CNN
 F 3 "" H 2000 4350 50  0001 C CNN
 	1    2000 4350
@@
 F 0 "C11" H 4175 2750 50  0000 L CNN
 F 1 "0.1uF" H 4175 2550 50  0000 L CNN
-F 2 "" H 4188 2500 50  0001 C CNN
+F 2 "Capacitors_SMD:C_0805_HandSoldering" H 4188 2500 50  0001 C CNN
 F 3 "" H 4150 2650 50  0001 C CNN
 	1    4150 2650
@@
 F 0 "R92" V 4230 3150 50  0000 C CNN
 F 1 "1K" V 4150 3150 50  0000 C CNN
-F 2 "" V 4080 3150 50  0001 C CNN
+F 2 "Resistors_SMD:R_0805_HandSoldering" V 4080 3150 50  0001 C CNN
 F 3 "" H 4150 3150 50  0001 C CNN
 	1    4150 3150
@@
 F 0 "R90" V 3980 3250 50  0000 C CNN
 F 1 "1K" V 3900 3250 50  0000 C CNN
-F 2 "" V 3830 3250 50  0001 C CNN
+F 2 "Resistors_SMD:R_0805_HandSoldering" V 3830 3250 50  0001 C CNN
 F 3 "" H 3900 3250 50  0001 C CNN
 	1    3900 3250
@@
 F 0 "J102" H 5750 3150 50  0000 C CNN
 F 1 "INA_41" H 5750 2850 50  0000 C CNN
-F 2 "" H 5750 3050 50  0001 C CNN
+F 2 "Pin_Headers:Pin_Header_Straight_1x02_Pitch2.54mm" H 5750 3050 50  0001 C CNN
 F 3 "" H 5750 3050 50  0001 C CNN
 	1    5750 3050
@@
 F 0 "JP4" H 3900 2930 50  0000 C CNN
 F 1 "Jumper_NO" H 3910 2790 50  0000 C CNN
-F 2 "" H 3900 2850 50  0001 C CNN
+F 2 "Pin_Headers:Pin_Header_Straight_1x02_Pitch2.54mm" H 3900 2850 50  0001 C CNN
 F 3 "" H 3900 2850 50  0001 C CNN
 	1    3900 2850
@@
 F 0 "J98" H 4850 2200 50  0000 C CNN
 F 1 "INA_41" H 4850 1700 50  0000 C CNN
-F 2 "" H 4850 2000 50  0001 C CNN
+F 2 "Pin_Headers:Pin_Header_Straight_1x04_Pitch2.54mm" H 4850 2000 50  0001 C CNN
 F 3 "" H 4850 2000 50  0001 C CNN
 	1    4850 2000
@@
 F 0 "J99" H 4850 4550 50  0000 C CNN
 F 1 "INA_41" H 4850 4050 50  0000 C CNN
-F 2 "" H 4850 4350 50  0001 C CNN
+F 2 "Pin_Headers:Pin_Header_Straight_1x04_Pitch2.54mm" H 4850 4350 50  0001 C CNN
 F 3 "" H 4850 4350 50  0001 C CNN
 	1    4850 4350
@@
 F 0 "C10" H 1325 5850 50  0000 L CNN
 F 1 "0.1uF" H 1325 5650 50  0000 L CNN
-F 2 "" H 1338 5600 50  0001 C CNN
+F 2 "Capacitors_SMD:C_0805_HandSoldering" H 1338 5600 50  0001 C CNN
 F 3 "" H 1300 5750 50  0001 C CNN
 	1    1300 5750
@@
 F 0 "R89" V 1380 6250 50  0000 C CNN
 F 1 "1K" V 1300 6250 50  0000 C CNN
-F 2 "" V 1230 6250 50  0001 C CNN
+F 2 "Resistors_SMD:R_0805_HandSoldering" V 1230 6250 50  0001 C CNN
 F 3 "" H 1300 6250 50  0001 C CNN
 	1    1300 6250
@@
 F 0 "R87" V 1130 6350 50  0000 C CNN
 F 1 "1K" V 1050 6350 50  0000 C CNN
-F 2 "" V 980 6350 50  0001 C CNN
+F 2 "Resistors_SMD:R_0805_HandSoldering" V 980 6350 50  0001 C CNN
 F 3 "" H 1050 6350 50  0001 C CNN
 	1    1050 6350
@@
 F 0 "J97" H 2900 6250 50  0000 C CNN
 F 1 "INA_42" H 2900 5950 50  0000 C CNN
-F 2 "" H 2900 6150 50  0001 C CNN
+F 2 "Pin_Headers:Pin_Header_Straight_1x02_Pitch2.54mm" H 2900 6150 50  0001 C CNN
 F 3 "" H 2900 6150 50  0001 C CNN
 	1    2900 6150
@@
 F 0 "JP3" H 1050 6030 50  0000 C CNN
 F 1 "Jumper_NO" H 1060 5890 50  0000 C CNN
-F 2 "" H 1050 5950 50  0001 C CNN
+F 2 "Pin_Headers:Pin_Header_Straight_1x02_Pitch2.54mm" H 1050 5950 50  0001 C CNN
 F 3 "" H 1050 5950 50  0001 C CNN
 	1    1050 5950
@@
 F 0 "J94" H 2000 5300 50  0000 C CNN
 F 1 "INA_42" H 2000 4800 50  0000 C CNN
-F 2 "" H 2000 5100 50  0001 C CNN
+F 2 "Pin_Headers:Pin_Header_Straight_1x04_Pitch2.54mm" H 2000 5100 50  0001 C CNN
 F 3 "" H 2000 5100 50  0001 C CNN
 	1    2000 5100
@@
 F 0 "J95" H 2000 7650 50  0000 C CNN
 F 1 "INA_42" H 2000 7150 50  0000 C CNN
-F 2 "" H 2000 7450 50  0001 C CNN
+F 2 "Pin_Headers:Pin_Header_Straight_1x04_Pitch2.54mm" H 2000 7450 50  0001 C CNN
 F 3 "" H 2000 7450 50  0001 C CNN
 	1    2000 7450
@@
 F 0 "C12" H 4175 5850 50  0000 L CNN
 F 1 "0.1uF" H 4175 5650 50  0000 L CNN
-F 2 "" H 4188 5600 50  0001 C CNN
+F 2 "Capacitors_SMD:C_0805_HandSoldering" H 4188 5600 50  0001 C CNN
 F 3 "" H 4150 5750 50  0001 C CNN
 	1    4150 5750
@@
 F 0 "R93" V 4230 6250 50  0000 C CNN
 F 1 "1K" V 4150 6250 50  0000 C CNN
-F 2 "" V 4080 6250 50  0001 C CNN
+F 2 "Resistors_SMD:R_0805_HandSoldering" V 4080 6250 50  0001 C CNN
 F 3 "" H 4150 6250 50  0001 C CNN
 	1    4150 6250
@@
 F 0 "R91" V 3980 6350 50  0000 C CNN
 F 1 "1K" V 3900 6350 50  0000 C CNN
-F 2 "" V 3830 6350 50  0001 C CNN
+F 2 "Resistors_SMD:R_0805_HandSoldering" V 3830 6350 50  0001 C CNN
 F 3 "" H 3900 6350 50  0001 C CNN
 	1    3900 6350
@@
 F 0 "J103" H 5750 6250 50  0000 C CNN
 F 1 "INA_43" H 5750 5950 50  0000 C CNN
-F 2 "" H 5750 6150 50  0001 C CNN
+F 2 "Pin_Headers:Pin_Header_Straight_1x02_Pitch2.54mm" H 5750 6150 50  0001 C CNN
 F 3 "" H 5750 6150 50  0001 C CNN
 	1    5750 6150
@@
 F 0 "JP5" H 3900 6030 50  0000 C CNN
 F 1 "Jumper_NO" H 3910 5890 50  0000 C CNN
-F 2 "" H 3900 5950 50  0001 C CNN
+F 2 "Pin_Headers:Pin_Header_Straight_1x02_Pitch2.54mm" H 3900 5950 50  0001 C CNN
 F 3 "" H 3900 5950 50  0001 C CNN
 	1    3900 5950
@@
 F 0 "J100" H 4850 5300 50  0000 C CNN
 F 1 "INA_43" H 4850 4800 50  0000 C CNN
-F 2 "" H 4850 5100 50  0001 C CNN
+F 2 "Pin_Headers:Pin_Header_Straight_1x04_Pitch2.54mm" H 4850 5100 50  0001 C CNN
 F 3 "" H 4850 5100 50  0001 C CNN
 	1    4850 5100
@@
 F 0 "J101" H 4850 7650 50  0000 C CNN
 F 1 "INA_43" H 4850 7150 50  0000 C CNN
-F 2 "" H 4850 7450 50  0001 C CNN
+F 2 "Pin_Headers:Pin_Header_Straight_1x04_Pitch2.54mm" H 4850 7450 50  0001 C CNN
 F 3 "" H 4850 7450 50  0001 C CNN
 	1    4850 7450
@@
 F 0 "J104" H 6800 2400 50  0000 C CNN
 F 1 "INA" H 6800 1900 50  0000 C CNN
-F 2 "" H 6800 2200 50  0001 C CNN
+F 2 "Pin_Headers:Pin_Header_Straight_1x04_Pitch2.54mm" H 6800 2200 50  0001 C CNN
 F 3 "" H 6800 2200 50  0001 C CNN
 	1    6800 2200
@@
 F 0 "J105" H 6800 3250 50  0000 C CNN
 F 1 "INA" H 6800 2750 50  0000 C CNN
-F 2 "" H 6800 3050 50  0001 C CNN
+F 2 "Pin_Headers:Pin_Header_Straight_1x04_Pitch2.54mm" H 6800 3050 50  0001 C CNN
 F 3 "" H 6800 3050 50  0001 C CNN
 	1    6800 3050

Commit message: adding footprints, starting layout
Parts:
- TP105, TP106, TP107, TP108, TP109, TP110, TP111, TP112: footprint (none) -> TestPoint:TestPoint
- U10, U7, U8, U9: footprint (none) -> INA219BIDCNR:SOT65P280X145-8N
Changed lines of the file:
@@
 LIBS:contrib
 LIBS:valves
-LIBS:FDN337N
+LIBS:TCA6424ARGJR
 LIBS:Fixture-Dev-Kit-cache
 EELAYER 25 0
@@
 F 0 "U7" H 1700 4650 60  0000 C CNN
 F 1 "INA219BIDCNT" H 2000 3600 60  0000 C CNN
-F 2 "" H 2000 3600 60  0001 C CNN
+F 2 "INA219BIDCNR:SOT65P280X145-8N" H 2000 3600 60  0001 C CNN
 F 3 "" H 2000 3600 60  0001 C CNN
 	1    2000 3600
@@
 F 0 "U9" H 4550 4650 60  0000 C CNN
 F 1 "INA219BIDCNT" H 4850 3600 60  0000 C CNN
-F 2 "" H 4850 3600 60  0001 C CNN
+F 2 "INA219BIDCNR:SOT65P280X145-8N" H 4850 3600 60  0001 C CNN
 F 3 "" H 4850 3600 60  0001 C CNN
 	1    4850 3600
@@
 F 0 "U8" H 1700 7750 60  0000 C CNN
 F 1 "INA219BIDCNT" H 2000 6700 60  0000 C CNN
-F 2 "" H 2000 6700 60  0001 C CNN
+F 2 "INA219BIDCNR:SOT65P280X145-8N" H 2000 6700 60  0001 C CNN
 F 3 "" H 2000 6700 60  0001 C CNN
 	1    2000 6700
@@
 F 0 "U10" H 4550 7750 60  0000 C CNN
 F 1 "INA219BIDCNT" H 4850 6700 60  0000 C CNN
-F 2 "" H 4850 6700 60  0001 C CNN
+F 2 "INA219BIDCNR:SOT65P280X145-8N" H 4850 6700 60  0001 C CNN
 F 3 "" H 4850 6700 60  0001 C CNN
 	1    4850 6700
@@
 F 0 "TP105" H 2600 3300 50  0000 C BNN
 F 1 "V+" H 2600 3250 50  0000 C CNN
-F 2 "" H 2600 3000 50  0001 C CNN
+F 2 "TestPoint:TestPoint" H 2600 3000 50  0001 C CNN
 F 3 "" H 2600 3000 50  0001 C CNN
 	1    2600 3000
@@
 F 0 "TP106" H 2600 3500 50  0000 C BNN
 F 1 "V-" H 2600 3450 50  0000 C CNN
-F 2 "" H 2600 3200 50  0001 C CNN
+F 2 "TestPoint:TestPoint" H 2600 3200 50  0001 C CNN
 F 3 "" H 2600 3200 50  0001 C CNN
 	1    2600 3200
@@
 F 0 "TP109" H 5450 3300 50  0000 C BNN
 F 1 "V+" H 5450 3250 50  0000 C CNN
-F 2 "" H 5450 3000 50  0001 C CNN
+F 2 "TestPoint:TestPoint" H 5450 3000 50  0001 C CNN
 F 3 "" H 5450 3000 50  0001 C CNN
 	1    5450 3000
@@
 F 0 "TP110" H 5450 3500 50  0000 C BNN
 F 1 "V-" H 5450 3450 50  0000 C CNN
-F 2 "" H 5450 3200 50  0001 C CNN
+F 2 "TestPoint:TestPoint" H 5450 3200 50  0001 C CNN
 F 3 "" H 5450 3200 50  0001 C CNN
 	1    5450 3200
@@
 F 0 "TP112" H 5450 6600 50  0000 C BNN
 F 1 "V-" H 5450 6550 50  0000 C CNN
-F 2 "" H 5450 6300 50  0001 C CNN
+F 2 "TestPoint:TestPoint" H 5450 6300 50  0001 C CNN
 F 3 "" H 5450 6300 50  0001 C CNN
 	1    5450 6300
@@
 F 0 "TP108" H 2600 6600 50  0000 C BNN
 F 1 "V-" H 2600 6550 50  0000 C CNN
-F 2 "" H 2600 6300 50  0001 C CNN
+F 2 "TestPoint:TestPoint" H 2600 6300 50  0001 C CNN
 F 3 "" H 2600 6300 50  0001 C CNN
 	1    2600 6300
@@
 F 0 "TP107" H 2600 6400 50  0000 C BNN
 F 1 "V+" H 2600 6350 50  0000 C CNN
-F 2 "" H 2600 6100 50  0001 C CNN
+F 2 "TestPoint:TestPoint" H 2600 6100 50  0001 C CNN
 F 3 "" H 2600 6100 50  0001 C CNN
 	1    2600 6100
@@
 F 0 "TP111" H 5450 6400 50  0000 C BNN
 F 1 "V+" H 5450 6350 50  0000 C CNN
-F 2 "" H 5450 6100 50  0001 C CNN
+F 2 "TestPoint:TestPoint" H 5450 6100 50  0001 C CNN
 F 3 "" H 5450 6100 50  0001 C CNN
 	1    5450 6100

Commit message: beginning pcb layout
Parts:
- removed J104, J105: INA, Pin_Headers:Pin_Header_Straight_1x04_Pitch2.54mm, symbol Conn_01x04
Connections:
- net C4-VCC-3V3: now also J100.1 (Pin_1), J101.1 (Pin_1), J92.1 (Pin_1), J93.1 (Pin_1), J94.1 (Pin_1), J95.1 (Pin_1), J98.1 (Pin_1), J99.1 (Pin_1); no longer J100.4 (Pin_4), J101.4 (Pin_4), J92.4 (Pin_4), J93.4 (Pin_4), J94.4 (Pin_4), J95.4 (Pin_4), J98.4 (Pin_4), J99.4 (Pin_4)
- net GND: now also J100.2 (Pin_2), J101.2 (Pin_2), J92.2 (Pin_2), J93.2 (Pin_2), J94.2 (Pin_2), J95.2 (Pin_2), J98.2 (Pin_2), J99.2 (Pin_2); no longer J100.3 (Pin_3), J101.3 (Pin_3), J92.3 (Pin_3), J93.3 (Pin_3), J94.3 (Pin_3), J95.3 (Pin_3), J98.3 (Pin_3), J99.3 (Pin_3)
- net I2C-SCK: now also J100.4 (Pin_4), J101.4 (Pin_4), J92.4 (Pin_4), J93.4 (Pin_4), J94.4 (Pin_4), J95.4 (Pin_4), J98.4 (Pin_4), J99.4 (Pin_4); no longer J100.1 (Pin_1), J101.1 (Pin_1), J92.1 (Pin_1), J93.1 (Pin_1), J94.1 (Pin_1), J95.1 (Pin_1), J98.1 (Pin_1), J99.1 (Pin_1)
- net I2C-SDA: now also J100.3 (Pin_3), J101.3 (Pin_3), J92.3 (Pin_3), J93.3 (Pin_3), J94.3 (Pin_3), J95.3 (Pin_3), J98.3 (Pin_3), J99.3 (Pin_3); no longer J100.2 (Pin_2), J101.2 (Pin_2), J92.2 (Pin_2), J93.2 (Pin_2), J94.2 (Pin_2), J95.2 (Pin_2), J98.2 (Pin_2), J99.2 (Pin_2)
Other:
- note removed: "Main Circuit \nHeaders\n"
