File: HARDWARE/v0.01/KiCad/_autosave-Fixture-Dev-Kit.kicad_pcb (KiCad board)
At the start: 2 copper layers, 379 parts, among them J1 POWER, J10 LED_3, J100 INA_43, J101 INA_43, J102 INA_41, J103 INA_43, J104 INA, J105 INA, J106 LED_6, J107 LED_7, J11 SW_5, J12 LED_4, J13 SW_6, J14 LED_5, J15 SW_7, J16 ADS_48, J17 ADS_48, J18 ADS_4A, J19 ADS_4A, J2 LED_0, J20 ADS_48, J21 ADS_4A, J22 ADS, J23 ADS, J24 ADS_49, J25 ADS_49, J26 ADS_49, J27 ADS_4B, J28 ADS_4B, J29 ADS_4B, J3 SW_0, J30 LOAD_0, J31 LOAD_1, J32 LOAD_2, J33 LOAD_3, J34 Conn_01x20, J35 BAT, J36 CHIP4LH, J38 Conn_01x20, J39 VBUS, J4 SW_1, J40 VBUS, J41 B_D+, J42 D-TP's, J43 B_D-, J44 USB_ID, J45 UPDATE, J46 ANT--SELECT, J47 Conn_01x20, J49 VBUS, J5 LED_1, J50 A_D+, J51 A_D-, J52 CHIP4RH, J53 Conn_01x20, J54 Conn_01x35, J56 Conn_01x35, J57 IOExp_0, J58 IOExp_0, J59 Conn_01x24, J6 SW_2, J60 IOExp_0, J61 IOExp_0, J62 Conn_01x24, J63 FET_0, J64 FET_0, J65 FET_0, J66 FET_0, J67 FET_0, J68 FET_0, J69 FET_0, J7 LED_2, J70 FET_0, J71 NFET_0, J72 NFET_4, J73 NFET_1, J74 NFET_5, J75 NFET_2, J76 NFET_6, J77 NFET_3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

Commit message: updaing PCB layout
Parts:
- moved J20 190.7 mm to (189.5, 32.6)
- moved U1 0.25 mm to (186.4, 38.7)
Changed lines of the file:
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@@
   )
   (module Pin_Headers:Pin_Header_Straight_1x04_Pitch2.54mm (layer F.Cu)
-    (at 293.028095 192.775)
+    (at 189.492 32.62)
     (descr "Through hole straight pin header, 1x04, 2.54mm pitch, single row")
     (tags "Through hole pin header THT 1x04 2.54mm single row")
@@
   )
   (module ADS1015IDGST:SOP50P490X110-10N (layer F.Cu)
-    (at 186.3551 38.94968 90)
+    (at 186.444 38.716 90)
     (attr smd)
     (fp_text reference U1 (at 0.711301 -3.58191 90) (layer F.SilkS)
