File: HARDWARE/v0.01/KiCad/FixtureDevKit-NMosfets.sch (KiCad schematic (older format))
At the start: 32 parts, among them J71 NFET_0, J72 NFET_4, J73 NFET_1, J74 NFET_5, J75 NFET_2, J76 NFET_6, J77 NFET_3, J78 NFET_7, Q13 FDN337N, Q14 FDN337N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

Commit message: adding footprints
Parts:
- J71, J72, J73, J74, J75, J76, J77, J78: footprint (none) -> Pin_Headers:Pin_Header_Straight_2x03_Pitch2.54mm
- Q13, Q14, Q15, Q16, Q17, Q18, Q19, Q20: footprint SSOT-3 -> (none)
- R68, R69, R70, R71, R72, R73, R74, R75, R76, R77, R78, R79, R80, R81, R82, R83: footprint (none) -> Resistors_SMD:R_0805_HandSoldering
Changed lines of the file:
@@
 F 0 "J71" H 2550 1750 50  0000 C CNN
 F 1 "NFET_0" H 2550 1350 50  0000 C CNN
-F 2 "" H 2500 1550 50  0001 C CNN
+F 2 "Pin_Headers:Pin_Header_Straight_2x03_Pitch2.54mm" H 2500 1550 50  0001 C CNN
 F 3 "" H 2500 1550 50  0001 C CNN
 	1    2500 1550
@@
 F 0 "Q13" H 2700 2950 50  0000 L BNN
 F 1 "FDN337N" H 2700 2850 50  0000 L BNN
-F 2 "SSOT-3" H 2600 2950 50  0001 L BNN
+F 2 "" H 2600 2950 50  0001 L BNN
 F 3 "ON Semiconductor" H 2600 2950 50  0001 L BNN
 F 4 "None" H 2600 2950 50  0001 L BNN "Package"
@@
 F 0 "R68" V 2430 2700 50  0000 C CNN
 F 1 "DNP" V 2350 2700 50  0000 C CNN
-F 2 "" V 2280 2700 50  0001 C CNN
+F 2 "Resistors_SMD:R_0805_HandSoldering" V 2280 2700 50  0001 C CNN
 F 3 "" H 2350 2700 50  0001 C CNN
 	1    2350 2700
@@
 F 0 "R70" V 2730 2700 50  0000 C CNN
 F 1 "DNP" V 2650 2700 50  0000 C CNN
-F 2 "" V 2580 2700 50  0001 C CNN
+F 2 "Resistors_SMD:R_0805_HandSoldering" V 2580 2700 50  0001 C CNN
 F 3 "" H 2650 2700 50  0001 C CNN
 	1    2650 2700
@@
 F 0 "R69" V 2430 5350 50  0000 C CNN
 F 1 "DNP" V 2350 5350 50  0000 C CNN
-F 2 "" V 2280 5350 50  0001 C CNN
+F 2 "Resistors_SMD:R_0805_HandSoldering" V 2280 5350 50  0001 C CNN
 F 3 "" H 2350 5350 50  0001 C CNN
 	1    2350 5350
@@
 F 0 "R71" V 2730 5350 50  0000 C CNN
 F 1 "DNP" V 2650 5350 50  0000 C CNN
-F 2 "" V 2580 5350 50  0001 C CNN
+F 2 "Resistors_SMD:R_0805_HandSoldering" V 2580 5350 50  0001 C CNN
 F 3 "" H 2650 5350 50  0001 C CNN
 	1    2650 5350
@@
 F 0 "J72" H 2550 4400 50  0000 C CNN
 F 1 "NFET_4" H 2550 4000 50  0000 C CNN
-F 2 "" H 2500 4200 50  0001 C CNN
+F 2 "Pin_Headers:Pin_Header_Straight_2x03_Pitch2.54mm" H 2500 4200 50  0001 C CNN
 F 3 "" H 2500 4200 50  0001 C CNN
 	1    2500 4200
@@
 F 0 "Q14" H 2700 5600 50  0000 L BNN
 F 1 "FDN337N" H 2700 5500 50  0000 L BNN
-F 2 "SSOT-3" H 2600 5600 50  0001 L BNN
+F 2 "" H 2600 5600 50  0001 L BNN
 F 3 "ON Semiconductor" H 2600 5600 50  0001 L BNN
 F 4 "None" H 2600 5600 50  0001 L BNN "Package"
@@
 F 0 "R81" V 8130 5350 50  0000 C CNN
 F 1 "DNP" V 8050 5350 50  0000 C CNN
-F 2 "" V 7980 5350 50  0001 C CNN
+F 2 "Resistors_SMD:R_0805_HandSoldering" V 7980 5350 50  0001 C CNN
 F 3 "" H 8050 5350 50  0001 C CNN
 	1    8050 5350
@@
 F 0 "R83" V 8430 5350 50  0000 C CNN
 F 1 "DNP" V 8350 5350 50  0000 C CNN
-F 2 "" V 8280 5350 50  0001 C CNN
+F 2 "Resistors_SMD:R_0805_HandSoldering" V 8280 5350 50  0001 C CNN
 F 3 "" H 8350 5350 50  0001 C CNN
 	1    8350 5350
@@
 F 0 "J78" H 8250 4400 50  0000 C CNN
 F 1 "NFET_7" H 8250 4000 50  0000 C CNN
-F 2 "" H 8200 4200 50  0001 C CNN
+F 2 "Pin_Headers:Pin_Header_Straight_2x03_Pitch2.54mm" H 8200 4200 50  0001 C CNN
 F 3 "" H 8200 4200 50  0001 C CNN
 	1    8200 4200
@@
 F 0 "Q20" H 8400 5600 50  0000 L BNN
 F 1 "FDN337N" H 8400 5500 50  0000 L BNN
-F 2 "SSOT-3" H 8300 5600 50  0001 L BNN
+F 2 "" H 8300 5600 50  0001 L BNN
 F 3 "ON Semiconductor" H 8300 5600 50  0001 L BNN
 F 4 "None" H 8300 5600 50  0001 L BNN "Package"
@@
 F 0 "R77" V 6230 5350 50  0000 C CNN
 F 1 "DNP" V 6150 5350 50  0000 C CNN
-F 2 "" V 6080 5350 50  0001 C CNN
+F 2 "Resistors_SMD:R_0805_HandSoldering" V 6080 5350 50  0001 C CNN
 F 3 "" H 6150 5350 50  0001 C CNN
 	1    6150 5350
@@
 F 0 "R79" V 6530 5350 50  0000 C CNN
 F 1 "DNP" V 6450 5350 50  0000 C CNN
-F 2 "" V 6380 5350 50  0001 C CNN
+F 2 "Resistors_SMD:R_0805_HandSoldering" V 6380 5350 50  0001 C CNN
 F 3 "" H 6450 5350 50  0001 C CNN
 	1    6450 5350
@@
 F 0 "J76" H 6350 4400 50  0000 C CNN
 F 1 "NFET_6" H 6350 4000 50  0000 C CNN
-F 2 "" H 6300 4200 50  0001 C CNN
+F 2 "Pin_Headers:Pin_Header_Straight_2x03_Pitch2.54mm" H 6300 4200 50  0001 C CNN
 F 3 "" H 6300 4200 50  0001 C CNN
 	1    6300 4200
@@
 F 0 "Q18" H 6500 5600 50  0000 L BNN
 F 1 "FDN337N" H 6500 5500 50  0000 L BNN
-F 2 "SSOT-3" H 6400 5600 50  0001 L BNN
+F 2 "" H 6400 5600 50  0001 L BNN
 F 3 "ON Semiconductor" H 6400 5600 50  0001 L BNN
 F 4 "None" H 6400 5600 50  0001 L BNN "Package"
@@
 F 0 "R73" V 4330 5350 50  0000 C CNN
 F 1 "DNP" V 4250 5350 50  0000 C CNN
-F 2 "" V 4180 5350 50  0001 C CNN
+F 2 "Resistors_SMD:R_0805_HandSoldering" V 4180 5350 50  0001 C CNN
 F 3 "" H 4250 5350 50  0001 C CNN
 	1    4250 5350
@@
 F 0 "R75" V 4630 5350 50  0000 C CNN
 F 1 "DNP" V 4550 5350 50  0000 C CNN
-F 2 "" V 4480 5350 50  0001 C CNN
+F 2 "Resistors_SMD:R_0805_HandSoldering" V 4480 5350 50  0001 C CNN
 F 3 "" H 4550 5350 50  0001 C CNN
 	1    4550 5350
@@
 F 0 "J74" H 4450 4400 50  0000 C CNN
 F 1 "NFET_5" H 4450 4000 50  0000 C CNN
-F 2 "" H 4400 4200 50  0001 C CNN
+F 2 "Pin_Headers:Pin_Header_Straight_2x03_Pitch2.54mm" H 4400 4200 50  0001 C CNN
 F 3 "" H 4400 4200 50  0001 C CNN
 	1    4400 4200
@@
 F 0 "Q16" H 4600 5600 50  0000 L BNN
 F 1 "FDN337N" H 4600 5500 50  0000 L BNN
-F 2 "SSOT-3" H 4500 5600 50  0001 L BNN
+F 2 "" H 4500 5600 50  0001 L BNN
 F 3 "ON Semiconductor" H 4500 5600 50  0001 L BNN
 F 4 "None" H 4500 5600 50  0001 L BNN "Package"
@@
 F 0 "R80" V 8130 2700 50  0000 C CNN
 F 1 "DNP" V 8050 2700 50  0000 C CNN
-F 2 "" V 7980 2700 50  0001 C CNN
+F 2 "Resistors_SMD:R_0805_HandSoldering" V 7980 2700 50  0001 C CNN
 F 3 "" H 8050 2700 50  0001 C CNN
 	1    8050 2700
@@
 F 0 "R82" V 8430 2700 50  0000 C CNN
 F 1 "DNP" V 8350 2700 50  0000 C CNN
-F 2 "" V 8280 2700 50  0001 C CNN
+F 2 "Resistors_SMD:R_0805_HandSoldering" V 8280 2700 50  0001 C CNN
 F 3 "" H 8350 2700 50  0001 C CNN
 	1    8350 2700
@@
 F 0 "J77" H 8250 1750 50  0000 C CNN
 F 1 "NFET_3" H 8250 1350 50  0000 C CNN
-F 2 "" H 8200 1550 50  0001 C CNN
+F 2 "Pin_Headers:Pin_Header_Straight_2x03_Pitch2.54mm" H 8200 1550 50  0001 C CNN
 F 3 "" H 8200 1550 50  0001 C CNN
 	1    8200 1550
@@
 F 0 "Q19" H 8400 2950 50  0000 L BNN
 F 1 "FDN337N" H 8400 2850 50  0000 L BNN
-F 2 "SSOT-3" H 8300 2950 50  0001 L BNN
+F 2 "" H 8300 2950 50  0001 L BNN
 F 3 "ON Semiconductor" H 8300 2950 50  0001 L BNN
 F 4 "None" H 8300 2950 50  0001 L BNN "Package"
@@
 F 0 "R76" V 6230 2700 50  0000 C CNN
 F 1 "DNP" V 6150 2700 50  0000 C CNN
-F 2 "" V 6080 2700 50  0001 C CNN
+F 2 "Resistors_SMD:R_0805_HandSoldering" V 6080 2700 50  0001 C CNN
 F 3 "" H 6150 2700 50  0001 C CNN
 	1    6150 2700
@@
 F 0 "R78" V 6530 2700 50  0000 C CNN
 F 1 "DNP" V 6450 2700 50  0000 C CNN
-F 2 "" V 6380 2700 50  0001 C CNN
+F 2 "Resistors_SMD:R_0805_HandSoldering" V 6380 2700 50  0001 C CNN
 F 3 "" H 6450 2700 50  0001 C CNN
 	1    6450 2700
@@
 F 0 "J75" H 6350 1750 50  0000 C CNN
 F 1 "NFET_2" H 6350 1350 50  0000 C CNN
-F 2 "" H 6300 1550 50  0001 C CNN
+F 2 "Pin_Headers:Pin_Header_Straight_2x03_Pitch2.54mm" H 6300 1550 50  0001 C CNN
 F 3 "" H 6300 1550 50  0001 C CNN
 	1    6300 1550
@@
 F 0 "Q17" H 6500 2950 50  0000 L BNN
 F 1 "FDN337N" H 6500 2850 50  0000 L BNN
-F 2 "SSOT-3" H 6400 2950 50  0001 L BNN
+F 2 "" H 6400 2950 50  0001 L BNN
 F 3 "ON Semiconductor" H 6400 2950 50  0001 L BNN
 F 4 "None" H 6400 2950 50  0001 L BNN "Package"
@@
 F 0 "R72" V 4330 2700 50  0000 C CNN
 F 1 "DNP" V 4250 2700 50  0000 C CNN
-F 2 "" V 4180 2700 50  0001 C CNN
+F 2 "Resistors_SMD:R_0805_HandSoldering" V 4180 2700 50  0001 C CNN
 F 3 "" H 4250 2700 50  0001 C CNN
 	1    4250 2700
@@
 F 0 "R74" V 4630 2700 50  0000 C CNN
 F 1 "DNP" V 4550 2700 50  0000 C CNN
-F 2 "" V 4480 2700 50  0001 C CNN
+F 2 "Resistors_SMD:R_0805_HandSoldering" V 4480 2700 50  0001 C CNN
 F 3 "" H 4550 2700 50  0001 C CNN
 	1    4550 2700
@@
 F 0 "J73" H 4450 1750 50  0000 C CNN
 F 1 "NFET_1" H 4450 1350 50  0000 C CNN
-F 2 "" H 4400 1550 50  0001 C CNN
+F 2 "Pin_Headers:Pin_Header_Straight_2x03_Pitch2.54mm" H 4400 1550 50  0001 C CNN
 F 3 "" H 4400 1550 50  0001 C CNN
 	1    4400 1550
@@
 F 0 "Q15" H 4600 2950 50  0000 L BNN
 F 1 "FDN337N" H 4600 2850 50  0000 L BNN
-F 2 "SSOT-3" H 4500 2950 50  0001 L BNN
+F 2 "" H 4500 2950 50  0001 L BNN
 F 3 "ON Semiconductor" H 4500 2950 50  0001 L BNN
 F 4 "None" H 4500 2950 50  0001 L BNN "Package"

Commit message: adding footprints, starting layout
Parts:
- Q13, Q14, Q15, Q16, Q17, Q18, Q19, Q20: footprint (none) -> FDN337N:SSOT-3
Changed lines of the file:
@@
 LIBS:contrib
 LIBS:valves
-LIBS:FDN337N
+LIBS:TCA6424ARGJR
 LIBS:Fixture-Dev-Kit-cache
 EELAYER 25 0
@@
 F 0 "Q13" H 2700 2950 50  0000 L BNN
 F 1 "FDN337N" H 2700 2850 50  0000 L BNN
-F 2 "" H 2600 2950 50  0001 L BNN
+F 2 "FDN337N:SSOT-3" H 2600 2950 50  0001 L BNN
 F 3 "ON Semiconductor" H 2600 2950 50  0001 L BNN
 F 4 "None" H 2600 2950 50  0001 L BNN "Package"
@@
 F 0 "Q14" H 2700 5600 50  0000 L BNN
 F 1 "FDN337N" H 2700 5500 50  0000 L BNN
-F 2 "" H 2600 5600 50  0001 L BNN
+F 2 "FDN337N:SSOT-3" H 2600 5600 50  0001 L BNN
 F 3 "ON Semiconductor" H 2600 5600 50  0001 L BNN
 F 4 "None" H 2600 5600 50  0001 L BNN "Package"
@@
 F 0 "Q20" H 8400 5600 50  0000 L BNN
 F 1 "FDN337N" H 8400 5500 50  0000 L BNN
-F 2 "" H 8300 5600 50  0001 L BNN
+F 2 "FDN337N:SSOT-3" H 8300 5600 50  0001 L BNN
 F 3 "ON Semiconductor" H 8300 5600 50  0001 L BNN
 F 4 "None" H 8300 5600 50  0001 L BNN "Package"
@@
 F 0 "Q18" H 6500 5600 50  0000 L BNN
 F 1 "FDN337N" H 6500 5500 50  0000 L BNN
-F 2 "" H 6400 5600 50  0001 L BNN
+F 2 "FDN337N:SSOT-3" H 6400 5600 50  0001 L BNN
 F 3 "ON Semiconductor" H 6400 5600 50  0001 L BNN
 F 4 "None" H 6400 5600 50  0001 L BNN "Package"
@@
 F 0 "Q16" H 4600 5600 50  0000 L BNN
 F 1 "FDN337N" H 4600 5500 50  0000 L BNN
-F 2 "" H 4500 5600 50  0001 L BNN
+F 2 "FDN337N:SSOT-3" H 4500 5600 50  0001 L BNN
 F 3 "ON Semiconductor" H 4500 5600 50  0001 L BNN
 F 4 "None" H 4500 5600 50  0001 L BNN "Package"
@@
 F 0 "Q19" H 8400 2950 50  0000 L BNN
 F 1 "FDN337N" H 8400 2850 50  0000 L BNN
-F 2 "" H 8300 2950 50  0001 L BNN
+F 2 "FDN337N:SSOT-3" H 8300 2950 50  0001 L BNN
 F 3 "ON Semiconductor" H 8300 2950 50  0001 L BNN
 F 4 "None" H 8300 2950 50  0001 L BNN "Package"
@@
 F 0 "Q17" H 6500 2950 50  0000 L BNN
 F 1 "FDN337N" H 6500 2850 50  0000 L BNN
-F 2 "" H 6400 2950 50  0001 L BNN
+F 2 "FDN337N:SSOT-3" H 6400 2950 50  0001 L BNN
 F 3 "ON Semiconductor" H 6400 2950 50  0001 L BNN
 F 4 "None" H 6400 2950 50  0001 L BNN "Package"
@@
 F 0 "Q15" H 4600 2950 50  0000 L BNN
 F 1 "FDN337N" H 4600 2850 50  0000 L BNN
-F 2 "" H 4500 2950 50  0001 L BNN
+F 2 "FDN337N:SSOT-3" H 4500 2950 50  0001 L BNN
 F 3 "ON Semiconductor" H 4500 2950 50  0001 L BNN
 F 4 "None" H 4500 2950 50  0001 L BNN "Package"

Commit message: updating pcb layout
Connections:
- net Source_2 is gone; now on net Drain_2: J75.1 (Pin_1), J75.6 (Pin_6), Q17.2 (S), R76.2
- net Source_3 is gone; now on net Drain_3: J77.1 (Pin_1), J77.6 (Pin_6), Q19.2 (S), R80.2
- net Source_4 is gone; now on net Drain_4: J72.1 (Pin_1), J72.6 (Pin_6), Q14.2 (S), R69.2
- net Source_5 is gone; now on net Drain_5: J74.1 (Pin_1), J74.6 (Pin_6), Q16.2 (S), R73.2
- net Source_6 is gone; now on net Drain_6: J76.1 (Pin_1), J76.6 (Pin_6), Q18.2 (S), R77.2
- net Source_7 is gone; now on net Drain_7: J78.1 (Pin_1), J78.6 (Pin_6), Q20.2 (S), R81.2
- net Drain_0: now also J71.5 (Pin_5), J71.6 (Pin_6); no longer J71.3 (Pin_3), J71.4 (Pin_4)
- net Drain_1: now also J73.5 (Pin_5), J73.6 (Pin_6); no longer J73.3 (Pin_3), J73.4 (Pin_4)
- net Drain_2: now also J75.2 (Pin_2), J75.5 (Pin_5); no longer J75.3 (Pin_3), J75.4 (Pin_4)
- net Drain_3: now also J77.2 (Pin_2), J77.5 (Pin_5); no longer J77.3 (Pin_3), J77.4 (Pin_4)
- net Drain_4: now also J72.2 (Pin_2), J72.5 (Pin_5); no longer J72.3 (Pin_3), J72.4 (Pin_4)
- net Drain_5: now also J74.2 (Pin_2), J74.5 (Pin_5); no longer J74.3 (Pin_3), J74.4 (Pin_4)
- net Drain_6: now also J76.2 (Pin_2), J76.5 (Pin_5); no longer J76.3 (Pin_3), J76.4 (Pin_4)
- net Drain_7: now also J78.2 (Pin_2), J78.5 (Pin_5); no longer J78.3 (Pin_3), J78.4 (Pin_4)
- net Gate_0: now also J71.3 (Pin_3), J71.4 (Pin_4); no longer J71.2 (Pin_2), J71.5 (Pin_5)
- net Gate_1: now also J73.3 (Pin_3), J73.4 (Pin_4); no longer J73.2 (Pin_2), J73.5 (Pin_5)
- net Gate_2: now also J75.3 (Pin_3), J75.4 (Pin_4); no longer J75.2 (Pin_2), J75.5 (Pin_5)
- net Gate_3: now also J77.3 (Pin_3), J77.4 (Pin_4); no longer J77.2 (Pin_2), J77.5 (Pin_5)
- net Gate_4: now also J72.3 (Pin_3), J72.4 (Pin_4); no longer J72.2 (Pin_2), J72.5 (Pin_5)
- net Gate_5: now also J74.3 (Pin_3), J74.4 (Pin_4); no longer J74.2 (Pin_2), J74.5 (Pin_5)
- net Gate_6: now also J76.3 (Pin_3), J76.4 (Pin_4); no longer J76.2 (Pin_2), J76.5 (Pin_5)
- net Gate_7: now also J78.3 (Pin_3), J78.4 (Pin_4); no longer J78.2 (Pin_2), J78.5 (Pin_5)
- net Source_0: now also J71.2 (Pin_2); no longer J71.6 (Pin_6)
- net Source_1: now also J73.2 (Pin_2); no longer J73.6 (Pin_6)
Changed lines of the file:
@@
 Text Label 2400 1800 3    60   ~ 0
 Source_0
-Text Label 2500 1800 3    60   ~ 0
+Text Label 2600 1800 3    60   ~ 0
 Gate_0
-Text Label 2600 1800 3    60   ~ 0
+Text Label 2400 1200 1    60   ~ 0
 Drain_0
 Text Label 2500 2600 1    60   ~ 0
@@
 Wire Wire Line
 	2200 2950 2400 2950
-Wire Wire Line
-	2600 1250 2600 1800
-Wire Wire Line
-	2500 1250 2500 1800
-Wire Wire Line
-	2400 1250 2400 1800
 Connection ~ 2400 1750
 Connection ~ 2500 1750
@@
 Wire Wire Line
 	2800 5600 3050 5600
-Connection ~ 2600 4400
-Connection ~ 2500 4400
 Connection ~ 2400 4400
 Wire Wire Line
-	2400 3900 2400 4450
-Wire Wire Line
-	2500 3900 2500 4450
-Wire Wire Line
-	2600 3900 2600 4450
+	2400 3850 2400 4450
 Wire Wire Line
 	2200 5600 2400 5600
@@
 Text Label 2500 5250 1    60   ~ 0
 Gate_4
+Text Label 2400 3850 1    60   ~ 0
+Drain_4
 Text Label 2600 4450 3    60   ~ 0
-Drain_4
-Text Label 2500 4450 3    60   ~ 0
 Gate_4
 Text Label 2400 4450 3    60   ~ 0
@@
 Wire Wire Line
 	4700 5600 4950 5600
-Connection ~ 8300 4400
-Connection ~ 8200 4400
 Connection ~ 8100 4400
 Wire Wire Line
-	8100 3900 8100 4450
-Wire Wire Line
-	8200 3900 8200 4450
-Wire Wire Line
-	8300 3900 8300 4450
+	8100 3850 8100 4450
 Wire Wire Line
 	7900 5600 8100 5600
@@
 Text Label 8200 5250 1    60   ~ 0
 Gate_7
+Text Label 8100 3850 1    60   ~ 0
+Drain_7
 Text Label 8300 4450 3    60   ~ 0
-Drain_7
-Text Label 8200 4450 3    60   ~ 0
 Gate_7
 Text Label 8100 4450 3    60   ~ 0
@@
 	0    1    1    0
 $EndComp
-Connection ~ 6400 4400
-Connection ~ 6300 4400
 Connection ~ 6200 4400
 Wire Wire Line
-	6200 3900 6200 4450
-Wire Wire Line
-	6300 3900 6300 4450
-Wire Wire Line
-	6400 3900 6400 4450
+	6200 3850 6200 4450
 Wire Wire Line
 	6000 5600 6200 5600
@@
 Text Label 6300 5250 1    60   ~ 0
 Gate_6
+Text Label 6200 3850 1    60   ~ 0
+Drain_6
 Text Label 6400 4450 3    60   ~ 0
-Drain_6
-Text Label 6300 4450 3    60   ~ 0
 Gate_6
 Text Label 6200 4450 3    60   ~ 0
@@
 	0    1    1    0
 $EndComp
-Connection ~ 4500 4400
-Connection ~ 4400 4400
 Connection ~ 4300 4400
 Wire Wire Line
-	4300 3900 4300 4450
-Wire Wire Line
-	4400 3900 4400 4450
-Wire Wire Line
-	4500 3900 4500 4450
+	4300 3850 4300 4450
 Wire Wire Line
 	4100 5600 4300 5600
@@
 Text Label 4400 5250 1    60   ~ 0
 Gate_5
+Text Label 4300 3850 1    60   ~ 0
+Drain_5
 Text Label 4500 4450 3    60   ~ 0
-Drain_5
-Text Label 4400 4450 3    60   ~ 0
 Gate_5
 Text Label 4300 4450 3    60   ~ 0
@@
 Wire Wire Line
 	4700 2950 4950 2950
-Connection ~ 8300 1750
-Connection ~ 8200 1750
 Connection ~ 8100 1750
 Wire Wire Line
-	8100 1250 8100 1800
-Wire Wire Line
-	8200 1250 8200 1800
-Wire Wire Line
-	8300 1250 8300 1800
+	8100 1200 8100 1800
 Wire Wire Line
 	7900 2950 8100 2950
@@
 Text Label 8200 2600 1    60   ~ 0
 Gate_3
+Text Label 8100 1200 1    60   ~ 0
+Drain_3
 Text Label 8300 1800 3    60   ~ 0
-Drain_3
-Text Label 8200 1800 3    60   ~ 0
 Gate_3
 Text Label 8100 1800 3    60   ~ 0
@@
 	0    1    1    0
 $EndComp
-Connection ~ 6400 1750
-Connection ~ 6300 1750
 Connection ~ 6200 1750
 Wire Wire Line
-	6200 1250 6200 1800
-Wire Wire Line
-	6300 1250 6300 1800
-Wire Wire Line
-	6400 1250 6400 1800
+	6200 1200 6200 1800
 Wire Wire Line
 	6000 2950 6200 2950
@@
 Text Label 6300 2600 1    60   ~ 0
 Gate_2
+Text Label 6200 1200 1    60   ~ 0
+Drain_2
 Text Label 6400 1800 3    60   ~ 0
-Drain_2
-Text Label 6300 1800 3    60   ~ 0
 Gate_2
 Text Label 6200 1800 3    60   ~ 0
@@
 	0    1    1    0
 $EndComp
-Connection ~ 4500 1750
-Connection ~ 4400 1750
-Connection ~ 4300 1750
-Wire Wire Line
-	4300 1250 4300 1800
-Wire Wire Line
-	4400 1250 4400 1800
-Wire Wire Line
-	4500 1250 4500 1800
 Wire Wire Line
 	4100 2950 4300 2950
@@
 Text Label 4400 2600 1    60   ~ 0
 Gate_1
+Text Label 4300 1200 1    60   ~ 0
+Drain_1
 Text Label 4500 1800 3    60   ~ 0
-Drain_1
-Text Label 4400 1800 3    60   ~ 0
 Gate_1
 Text Label 4300 1800 3    60   ~ 0
@@
 	0    1    1    0
 $EndComp
+Wire Wire Line
+	2500 1750 2400 1750
+Wire Wire Line
+	2400 1750 2400 1800
+Wire Wire Line
+	2600 1250 2600 1800
+Wire Wire Line
+	2500 1250 2400 1250
+Wire Wire Line
+	2400 1250 2400 1200
+Wire Wire Line
+	4300 1800 4300 1750
+Wire Wire Line
+	4300 1750 4400 1750
+Wire Wire Line
+	4500 1250 4500 1800
+Connection ~ 4500 1750
+Wire Wire Line
+	4400 1250 4300 1250
+Wire Wire Line
+	4300 1250 4300 1200
+Wire Wire Line
+	6200 1750 6300 1750
+Wire Wire Line
+	6400 1250 6400 1800
+Connection ~ 6400 1750
+Wire Wire Line
+	6300 1250 6200 1250
+Connection ~ 6200 1250
+Wire Wire Line
+	8100 1750 8200 1750
+Wire Wire Line
+	8300 1250 8300 1800
+Connection ~ 8300 1750
+Wire Wire Line
+	8200 1250 8100 1250
+Connection ~ 8100 1250
+Wire Wire Line
+	2400 4400 2500 4400
+Wire Wire Line
+	2600 3900 2600 4450
+Connection ~ 2600 4400
+Wire Wire Line
+	2500 3900 2400 3900
+Connection ~ 2400 3900
+Wire Wire Line
+	4300 4400 4400 4400
+Wire Wire Line
+	4500 3900 4500 4450
+Connection ~ 4500 4400
+Wire Wire Line
+	4400 3900 4300 3900
+Connection ~ 4300 3900
+Wire Wire Line
+	6200 4400 6300 4400
+Wire Wire Line
+	6400 3900 6400 4450
+Connection ~ 6400 4400
+Wire Wire Line
+	6300 3900 6200 3900
+Connection ~ 6200 3900
+Wire Wire Line
+	8100 4400 8200 4400
+Wire Wire Line
+	8300 3900 8300 4450
+Connection ~ 8300 4400
+Wire Wire Line
+	8200 3900 8100 3900
+Connection ~ 8100 3900
 $EndSCHEMATC
