File: HARDWARE/v0.02/KiCad/Fixture-Dev-Kit.sch (KiCad schematic (older format))
At the start: 4 parts, among them J1 DUT, J2 POWER, J39 DUT BAT, J40 DUT BAT

Commit message: adding 3v3 line up to DUT header
Parts:
- added F6, F?: Fuse, 1206:1206, symbol Fuse
Connections:
- wire segments 47 -> 50
Changed lines of the file:
@@
 $EndSheet
 $Comp
-L PWR_FLAG #FLG01
+L PWR_FLAG #FLG1
 U 1 1 59EFDEB7
 P 1200 5000
-F 0 "#FLG01" H 1200 5075 50  0001 C CNN
+F 0 "#FLG1" H 1200 5075 50  0001 C CNN
 F 1 "PWR_FLAG" H 1200 5150 50  0000 C CNN
 F 2 "" H 1200 5000 50  0001 C CNN
@@
 $EndComp
 $Comp
-L PWR_FLAG #FLG02
+L PWR_FLAG #FLG2
 U 1 1 59EFDEC9
 P 1700 5000
-F 0 "#FLG02" H 1700 5075 50  0001 C CNN
+F 0 "#FLG2" H 1700 5075 50  0001 C CNN
 F 1 "PWR_FLAG" H 1700 5150 50  0000 C CNN
 F 2 "" H 1700 5000 50  0001 C CNN
@@
 $EndComp
 $Comp
-L GND #PWR03
+L GND #PWR9
 U 1 1 59EFDED6
 P 1700 5100
-F 0 "#PWR03" H 1700 4850 50  0001 C CNN
+F 0 "#PWR9" H 1700 4850 50  0001 C CNN
 F 1 "GND" H 1700 4950 50  0000 C CNN
 F 2 "" H 1700 5100 50  0001 C CNN
@@
 	1550 4350 1800 4350
 $Comp
-L GND #PWR04
+L GND #PWR7
 U 1 1 59F1B0B1
 P 1800 4450
-F 0 "#PWR04" H 1800 4200 50  0001 C CNN
+F 0 "#PWR7" H 1800 4200 50  0001 C CNN
 F 1 "GND" H 1800 4300 50  0000 C CNN
 F 2 "" H 1800 4450 50  0001 C CNN
@@
 	850  4000 2550 4000
 $Comp
-L +5V #PWR05
+L +5V #PWR8
 U 1 1 59F1DD6A
 P 1200 5100
-F 0 "#PWR05" H 1200 4950 50  0001 C CNN
+F 0 "#PWR8" H 1200 4950 50  0001 C CNN
 F 1 "+5V" H 1200 5240 50  0000 C CNN
 F 2 "" H 1200 5100 50  0001 C CNN
@@
 $EndComp
 $Comp
-L +5V #PWR06
+L +5V #PWR6
 U 1 1 59F1DD81
 P 1800 4350
-F 0 "#PWR06" H 1800 4200 50  0001 C CNN
+F 0 "#PWR6" H 1800 4200 50  0001 C CNN
 F 1 "+5V" H 1800 4490 50  0000 C CNN
 F 2 "" H 1800 4350 50  0001 C CNN
@@
 $EndSheet
 $Comp
-L GND #PWR07
+L GND #PWR5
 U 1 1 59FA7F5A
 P 9250 4050
-F 0 "#PWR07" H 9250 3800 50  0001 C CNN
+F 0 "#PWR5" H 9250 3800 50  0001 C CNN
 F 1 "GND" H 9250 3900 50  0000 C CNN
 F 2 "" H 9250 4050 50  0001 C CNN
@@
 	2650 1600 2500 1600
 $Comp
-L +5V #PWR08
+L +5V #PWR1
 U 1 1 59FB980B
 P 2650 1950
-F 0 "#PWR08" H 2650 1800 50  0001 C CNN
+F 0 "#PWR1" H 2650 1800 50  0001 C CNN
 F 1 "+5V" H 2650 2090 50  0000 C CNN
 F 2 "" H 2650 1950 50  0001 C CNN
@@
 	6850 3200 6700 3200
 $Comp
-L +5V #PWR09
+L +5V #PWR3
 U 1 1 59FC47B7
 P 4500 3050
-F 0 "#PWR09" H 4500 2900 50  0001 C CNN
+F 0 "#PWR3" H 4500 2900 50  0001 C CNN
 F 1 "+5V" H 4500 3190 50  0000 C CNN
 F 2 "" H 4500 3050 50  0001 C CNN
@@
 $EndComp
 $Comp
-L +5V #PWR010
+L +5V #PWR4
 U 1 1 59FC49D9
 P 6900 3100
-F 0 "#PWR010" H 6900 2950 50  0001 C CNN
+F 0 "#PWR4" H 6900 2950 50  0001 C CNN
 F 1 "+5V" H 6900 3240 50  0000 C CNN
 F 2 "" H 6900 3100 50  0001 C CNN
@@
 	9250 3550 9200 3550
 Connection ~ 9250 3750
-Wire Wire Line
-	8700 3050 8700 4050
-Connection ~ 8700 3250
 Connection ~ 8700 3450
 Connection ~ 8700 3650
 Wire Wire Line
-	8700 4050 9250 4050
+	9250 4050 8700 4050
 Connection ~ 8700 3850
+$Comp
+L +5V #PWR2
+U 1 1 5A01083F
+P 8050 2750
+F 0 "#PWR2" H 8050 2600 50  0001 C CNN
+F 1 "+5V" H 8050 2890 50  0000 C CNN
+F 2 "" H 8050 2750 50  0001 C CNN
+F 3 "" H 8050 2750 50  0001 C CNN
+	1    8050 2750
+	1    0    0    -1
+$EndComp
+$Comp
+L Fuse F6
+U 1 1 5A0109B9
+P 8050 2900
+F 0 "F6" V 8130 2900 50  0000 C CNN
+F 1 "Fuse" V 7975 2900 50  0000 C CNN
+F 2 "1206:1206" V 7980 2900 50  0001 C CNN
+F 3 "" H 8050 2900 50  0001 C CNN
+	1    8050 2900
+	1    0    0    -1
+$EndComp
+Wire Wire Line
+	8050 3050 8700 3050
+Text Label 7850 2750 1    60   ~ 0
+C4-VCC-3V3
+Wire Wire Line
+	8700 4050 8700 3450
+Wire Wire Line
+	7850 3250 8700 3250
+$Comp
+L Fuse F?
+U 1 1 5A01306A
+P 7850 2900
+F 0 "F?" V 7930 2900 50  0000 C CNN
+F 1 "Fuse" V 7775 2900 50  0000 C CNN
+F 2 "1206:1206" V 7780 2900 50  0001 C CNN
+F 3 "" H 7850 2900 50  0001 C CNN
+	1    7850 2900
+	1    0    0    -1
+$EndComp
+Wire Wire Line
+	7850 3050 7850 3250
 $EndSCHEMATC

Commit message: updating project name
Parts:
- gave numbers to parts that had none: 1
Changed lines of the file:
@@
 encoding utf-8
 Sheet 1 7
-Title "CHIP4 Fixture Dev Kit"
+Title "Ms. Smith's 7th Period Science Class Project"
 Date "2017-10-25"
 Rev "v0.01"
-Comp "Next Thing Co"
-Comment1 "Havin' a Blast!"
+Comp ""
+Comment1 ""
 Comment2 ""
 Comment3 ""
@@
 	7850 3250 8700 3250
 $Comp
-L Fuse F?
+L Fuse F7
 U 1 1 5A01306A
 P 7850 2900
-F 0 "F?" V 7930 2900 50  0000 C CNN
+F 0 "F7" V 7930 2900 50  0000 C CNN
 F 1 "Fuse" V 7775 2900 50  0000 C CNN
 F 2 "1206:1206" V 7780 2900 50  0001 C CNN
