File: HARDWARE/v0.02/KiCad/FixtureDevKit-INA.sch (KiCad schematic (older format))
At the start: 68 parts, among them J27 INA_40, J28 INA_40, J29 INA_40, J30 INA_40, J35 40 V+, J36 41 V+, J37 42 V+, J38 43 V+, Q10 NTF2955-D, Q11 NTF2955-D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

Commit message: adding latest updates from pcb layout designed 11/8/2017
Changed lines of the file:
@@
 LIBS:TCA6424ARGJR
 LIBS:USB-A1HSW6
+LIBS:jumper
 LIBS:Fixture-Dev-Kit-cache
 EELAYER 25 0
@@
 $EndComp
 $Comp
-L GND #PWR30
+L GND #PWR31
 U 1 1 59F0363E
 P 2050 2450
-F 0 "#PWR30" H 2050 2200 50  0001 C CNN
+F 0 "#PWR31" H 2050 2200 50  0001 C CNN
 F 1 "GND" H 2050 2300 50  0000 C CNN
 F 2 "" H 2050 2450 50  0001 C CNN
@@
 SDA
 $Comp
-L GND #PWR32
+L GND #PWR29
 U 1 1 59F06DD3
 P 1500 3400
-F 0 "#PWR32" H 1500 3150 50  0001 C CNN
+F 0 "#PWR29" H 1500 3150 50  0001 C CNN
 F 1 "GND" H 1500 3250 50  0000 C CNN
 F 2 "" H 1500 3400 50  0001 C CNN
@@
 $EndComp
 $Comp
-L GND #PWR28
+L GND #PWR33
 U 1 1 59F80F3B
 P 3250 2150
-F 0 "#PWR28" H 3250 1900 50  0001 C CNN
+F 0 "#PWR33" H 3250 1900 50  0001 C CNN
 F 1 "GND" H 3250 2000 50  0000 C CNN
 F 2 "" H 3250 2150 50  0001 C CNN
@@
 $EndComp
 $Comp
-L GND #PWR31
+L GND #PWR37
 U 1 1 59FAD47F
 P 5850 2450
-F 0 "#PWR31" H 5850 2200 50  0001 C CNN
+F 0 "#PWR37" H 5850 2200 50  0001 C CNN
 F 1 "GND" H 5850 2300 50  0000 C CNN
 F 2 "" H 5850 2450 50  0001 C CNN
@@
 SDA
 $Comp
-L GND #PWR33
+L GND #PWR35
 U 1 1 59FAD4A2
 P 5300 3400
-F 0 "#PWR33" H 5300 3150 50  0001 C CNN
+F 0 "#PWR35" H 5300 3150 50  0001 C CNN
 F 1 "GND" H 5300 3250 50  0000 C CNN
 F 2 "" H 5300 3400 50  0001 C CNN
@@
 $EndComp
 $Comp
-L GND #PWR29
+L GND #PWR39
 U 1 1 59FAD4ED
 P 7050 2150
-F 0 "#PWR29" H 7050 1900 50  0001 C CNN
+F 0 "#PWR39" H 7050 1900 50  0001 C CNN
 F 1 "GND" H 7050 2000 50  0000 C CNN
 F 2 "" H 7050 2150 50  0001 C CNN
@@
 $EndComp
 $Comp
-L GND #PWR36
+L GND #PWR32
 U 1 1 59FAE04E
 P 2050 5650
-F 0 "#PWR36" H 2050 5400 50  0001 C CNN
+F 0 "#PWR32" H 2050 5400 50  0001 C CNN
 F 1 "GND" H 2050 5500 50  0000 C CNN
 F 2 "" H 2050 5650 50  0001 C CNN
@@
 SDA
 $Comp
-L GND #PWR38
+L GND #PWR30
 U 1 1 59FAE071
 P 1500 6600
-F 0 "#PWR38" H 1500 6350 50  0001 C CNN
+F 0 "#PWR30" H 1500 6350 50  0001 C CNN
 F 1 "GND" H 1500 6450 50  0000 C CNN
 F 2 "" H 1500 6600 50  0001 C CNN
@@
 $EndComp
 $Comp
-L GND #PWR37
+L GND #PWR38
 U 1 1 59FAE0E9
 P 5850 5650
-F 0 "#PWR37" H 5850 5400 50  0001 C CNN
+F 0 "#PWR38" H 5850 5400 50  0001 C CNN
 F 1 "GND" H 5850 5500 50  0000 C CNN
 F 2 "" H 5850 5650 50  0001 C CNN
@@
 SDA
 $Comp
-L GND #PWR39
+L GND #PWR36
 U 1 1 59FAE10C
 P 5300 6600
-F 0 "#PWR39" H 5300 6350 50  0001 C CNN
+F 0 "#PWR36" H 5300 6350 50  0001 C CNN
 F 1 "GND" H 5300 6450 50  0000 C CNN
 F 2 "" H 5300 6600 50  0001 C CNN
@@
 $EndComp
 $Comp
-L GND #PWR35
+L GND #PWR40
 U 1 1 59FAE157
 P 7050 5350
-F 0 "#PWR35" H 7050 5100 50  0001 C CNN
+F 0 "#PWR40" H 7050 5100 50  0001 C CNN
 F 1 "GND" H 7050 5200 50  0000 C CNN
 F 2 "" H 7050 5350 50  0001 C CNN
@@
 	1    0    0    -1
 $EndComp
+Text HLabel 5300 1650 2    60   Output ~ 0
+JUMP
+Text Label 5200 1650 2    60   ~ 0
+JUMP
+Wire Wire Line
+	5200 1650 5300 1650
 $EndSCHEMATC
