File: HARDWARE/v0.05/KiCad/FixtureDevKit-INA.sch (KiCad schematic (older format))
At the start: 68 parts, among them J27 INA_40, J28 INA_40, J29 INA_40, J30 INA_40, J35 40 V+, J36 41 V+, J37 42 V+, J38 43 V+, Q10 NTF2955-D, Q11 NTF2955-D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

Commit message: adding files ffor the C4 adapter board dev kit
updating N-Channel labeling on INA circuits
Parts:
- Q10, Q5, Q6, Q9: value NTF2955-D -> ZXMN4A06GT
Changed lines of the file:
@@
 P 3150 2350
 F 0 "Q5" H 3350 2400 50  0000 L CNN
-F 1 "NTF2955-D" H 3350 2300 50  0000 L CNN
+F 1 "ZXMN4A06GT" H 3350 2300 50  0000 L CNN
 F 2 "NTF2955T1G:SOT230P700X180-4N" H 3350 2450 50  0001 C CNN
 F 3 "" H 3150 2350 50  0001 C CNN
@@
 P 6950 2350
 F 0 "Q6" H 7150 2400 50  0000 L CNN
-F 1 "NTF2955-D" H 7150 2300 50  0000 L CNN
+F 1 "ZXMN4A06GT" H 7150 2300 50  0000 L CNN
 F 2 "NTF2955T1G:SOT230P700X180-4N" H 7150 2450 50  0001 C CNN
 F 3 "" H 6950 2350 50  0001 C CNN
@@
 P 3150 5550
 F 0 "Q9" H 3350 5600 50  0000 L CNN
-F 1 "NTF2955-D" H 3350 5500 50  0000 L CNN
+F 1 "ZXMN4A06GT" H 3350 5500 50  0000 L CNN
 F 2 "NTF2955T1G:SOT230P700X180-4N" H 3350 5650 50  0001 C CNN
 F 3 "" H 3150 5550 50  0001 C CNN
@@
 P 6950 5550
 F 0 "Q10" H 7150 5600 50  0000 L CNN
-F 1 "NTF2955-D" H 7150 5500 50  0000 L CNN
+F 1 "ZXMN4A06GT" H 7150 5500 50  0000 L CNN
 F 2 "NTF2955T1G:SOT230P700X180-4N" H 7150 5650 50  0001 C CNN
 F 3 "" H 6950 5550 50  0001 C CNN
